File: 3PDT/pcb/3PDT.sch (EAGLE design)
At the start: 4 parts, among them SW1 3PDT, X1 2510-

Commit message: 20170914
Connections:
- net N$6 renamed GND
Changed lines of the file:
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@@
 <part name="R1" library="pedals-resistors" deviceset="R_" device=".3B"/>
 <part name="D1" library="pedals-diodes" deviceset="LED" device=""/>
+<part name="GND1" library="pedals-supply" deviceset="GND" device=""/>
+<part name="GND2" library="pedals-supply" deviceset="GND" device=""/>
 </parts>
 <sheets>
@@
 <instance part="R1" gate="G$1" x="33.02" y="88.9"/>
 <instance part="D1" gate="G$1" x="33.02" y="83.82"/>
+<instance part="GND1" gate="GND" x="-12.7" y="78.74" rot="R90"/>
+<instance part="GND2" gate="GND" x="2.54" y="81.28" rot="R270"/>
 </instances>
 <busses>
@@
 </segment>
 </net>
-<net name="N$6" class="0">
-<segment>
-<pinref part="X1" gate="-6" pin="KL"/>
-<wire x1="-17.78" y1="78.74" x2="0" y2="78.74" width="0.1524" layer="91"/>
-<wire x1="0" y1="78.74" x2="0" y2="81.28" width="0.1524" layer="91"/>
-<pinref part="SW1" gate="B" pin="2"/>
-<wire x1="0" y1="81.28" x2="7.62" y2="81.28" width="0.1524" layer="91"/>
-</segment>
-</net>
 <net name="N$7" class="0">
 <segment>
@@
 </segment>
 </net>
+<net name="GND" class="0">
+<segment>
+<pinref part="X1" gate="-6" pin="KL"/>
+<pinref part="GND1" gate="GND" pin="GND"/>
+<wire x1="-17.78" y1="78.74" x2="-15.24" y2="78.74" width="0.1524" layer="91"/>
+</segment>
+<segment>
+<pinref part="GND2" gate="GND" pin="GND"/>
+<pinref part="SW1" gate="B" pin="2"/>
+<wire x1="5.08" y1="81.28" x2="7.62" y2="81.28" width="0.1524" layer="91"/>
+</segment>
+</net>
