File: MXR Dynacomp/pcb/dynacomp.brd (EAGLE design)
At the start: 59 x 71.3 mm, 50 parts, among them IC1 CA3080E, J1 POWER_JACK, Q1 2N3904, Q2 2N3904, Q3 2N3904, Q4 2N3904, Q5 2N3904, X1 2510-

Commit message: 20170902
Parts:
- removed C14: 10u, pedals-capacitors-elec:040_020
- added C2: 100n, pedals-capacitors-film:050X030_025_2
- C1: value 47n -> 100u; device pedals-capacitors-film:BOX_SMALL -> pedals-capacitors-elec:040_020
- C10: value 1u -> 10n; device pedals-capacitors-elec:040_020 -> pedals-capacitors-film:BOX_SMALL
- C11: value 1n -> 10u; device pedals-capacitors-film:BOX_SMALL -> pedals-capacitors-elec:040_020
- C13: value 10n -> 47n
- C3: value 100u -> 47u
- C4: value 100n -> 150p; device pedals-capacitors-film:BOX_SMALL -> pedals-capacitors-film:050X030_025_2
- C5: value 47u -> 10n; device pedals-capacitors-elec:040_020 -> pedals-capacitors-film:BOX_SMALL
- C6: value 10n -> 1u; device pedals-capacitors-film:BOX_SMALL -> pedals-capacitors-film:BOX_BIG
- C7: value 150p -> 10n; device pedals-capacitors-film:050X030_025_2 -> pedals-capacitors-film:BOX_SMALL
- C8: device pedals-capacitors-film:BOX_BIG -> pedals-capacitors-elec:040_020
- C9: value 10n -> 1n
- moved Q4 100.8 mm to (54.0, 27.9), turned to 90 degrees
- moved D3 99.7 mm to (54.0, 20.3), turned to 270 degrees
- moved R21 98.7 mm to (46.4, 36.8), turned to 270 degrees
- moved Q5 91.9 mm to (40.0, 39.4), turned to 180 degrees
- moved C12 91.3 mm to (43.8, 17.8), turned to 90 degrees
- moved R19 88.2 mm to (40.0, 35.6), turned to 180 degrees
- moved R16 85.8 mm to (41.3, 19.1), turned to 90 degrees
- moved C1 85.1 mm to (30.9, 37.8)
- moved R17 80.7 mm to (46.4, 19.1), turned to 270 degrees
- moved C13 79.7 mm to (41.3, 27.9), turned to 270 degrees
- moved R20 78.8 mm to (23.5, 43.2)
- moved R18 75.7 mm to (51.4, 19.1), turned to 90 degrees
- moved R11 73.5 mm to (23.5, 40.6)
- moved D1 70.8 mm to (32.4, 45.7), turned to 270 degrees
- moved R4 69.9 mm to (23.5, 14.0), turned to 180 degrees
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Connections:
- removed net N$7: C1.1, R21.2
- new net C40: C13.1, R21.2
- net C10: now also C7.2, C8.+; no longer C10.+, C9.2
- net C8: now also C6.1; no longer C8.1
- net GND: now also C1.-, C11.-, C2.1, C4.2, C8.-; no longer C10.-, C14.-, C4.1, C5.-, C7.2
- net IN: now also C4.1, C5.2; no longer C6.2, C7.1
- net N$1: now also C12.2; no longer C1.2
- net N$10: now also C7.1; no longer C9.1
- net N$14: now also C10.2; no longer C12.2
- net N$15: now also C9.2; no longer C11.2
- net N$17: now also C10.1; no longer C12.1
- net N$19: now also C12.1; no longer C13.1
- net N$3: now also C5.1; no longer C6.1
- net N$8: now also C11.+; no longer C14.+
- net N$9: now also C6.2; no longer C8.2
- net VB: now also C3.+, C9.1; no longer C11.1, C5.+
- net VR: now also C1.+, C2.2; no longer C3.+, C4.2
Routing:
- net +9V: track 0.00 -> 67.0 mm
- net VR: track 0.00 -> 42.4 mm
- net N$13: track 0.00 -> 41.2 mm
- net N$19: track 0.00 -> 26.4 mm
- net N$15: track 0.00 -> 22.3 mm
- net VB: track 0.00 -> 21.7 mm
- net N$8: track 0.00 -> 21.4 mm
- net C8: track 0.00 -> 19.1 mm
- net IN: track 0.00 -> 18.7 mm
- net N$6: track 0.00 -> 16.4 mm
- net N$11: track 0.00 -> 12.9 mm
- net N$9: track 0.00 -> 12.5 mm
- net N$10: track 0.00 -> 12.2 mm
- net C10: track 0.00 -> 11.9 mm
- net N$1: track 0.00 -> 11.7 mm
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- added copper zone on layer 1, net GND

Commit message: 20170914
Routing:
- net N$15: track 22.3 -> 22.8 mm
Changed lines of the file:
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@@
 <contactref element="OUTPUT" pad="S"/>
 <contactref element="INPUT" pad="S"/>
-<polygon width="0.4064" layer="16" isolate="0.254">
+<polygon width="0.3048" layer="16" isolate="0.254">
 <vertex x="0" y="72.39"/>
 <vertex x="58.42" y="72.39"/>
@@
 <contactref element="C11" pad="-"/>
 <contactref element="VOLUME" pad="1"/>
-<polygon width="0.4064" layer="1" isolate="0.254">
+<polygon width="0.3048" layer="1" isolate="0.254">
 <vertex x="59.055" y="1.905"/>
 <vertex x="59.055" y="73.025"/>
@@
 <via x="35.7505" y="20.955" extent="1-16" drill="0.5" diameter="0.85"/>
 <via x="33.02" y="20.955" extent="1-16" drill="0.5" diameter="0.85"/>
-<via x="35.7505" y="27.94" extent="1-16" drill="0.5" diameter="0.85"/>
-<via x="33.02" y="27.94" extent="1-16" drill="0.5" diameter="0.85"/>
+<via x="36.5125" y="29.21" extent="1-16" drill="0.5" diameter="0.85"/>
+<via x="33.02" y="29.21" extent="1-16" drill="0.5" diameter="0.85"/>
 <via x="22.987" y="6.5405" extent="1-16" drill="0.5" diameter="0.85"/>
-<via x="22.987" y="9.0805" extent="1-16" drill="0.5" diameter="0.85"/>
+<via x="22.987" y="10.6045" extent="1-16" drill="0.5" diameter="0.85"/>
 <via x="39.37" y="6.35" extent="1-16" drill="0.5" diameter="0.85"/>
 <via x="48.26" y="6.35" extent="1-16" drill="0.5" diameter="0.85"/>
 <via x="53.1495" y="10.7315" extent="1-16" drill="0.5" diameter="0.85"/>
-<via x="18.415" y="8.6995" extent="1-16" drill="0.5" diameter="0.85"/>
+<via x="18.415" y="10.6045" extent="1-16" drill="0.5" diameter="0.85"/>
 <via x="9.525" y="9.9695" extent="1-16" drill="0.5" diameter="0.85"/>
 <via x="4.0005" y="15.875" extent="1-16" drill="0.5" diameter="0.85"/>
@@
 <via x="26.67" y="39.37" extent="1-16" drill="0.5" diameter="0.85"/>
 <via x="24.13" y="39.37" extent="1-16" drill="0.5" diameter="0.85"/>
+<via x="48.26" y="12.065" extent="1-16" drill="0.5" diameter="0.85"/>
+<via x="43.815" y="23.495" extent="1-16" drill="0.5" diameter="0.85"/>
+<via x="39.37" y="34.925" extent="1-16" drill="0.5" diameter="0.85"/>
+<via x="11.43" y="23.9395" extent="1-16" drill="0.5" diameter="0.85"/>
 </signal>
 <signal name="VR">
@@
 <contactref element="R7" pad="2"/>
 <contactref element="C6" pad="2"/>
-<wire x1="9.525" y1="21.59" x2="10.16" y2="22.225" width="0.254" layer="16"/>
-<wire x1="10.16" y1="22.225" x2="16.51" y2="22.225" width="0.254" layer="16"/>
-<wire x1="16.51" y1="22.225" x2="17.145" y2="21.59" width="0.254" layer="16"/>
 <wire x1="5.715" y1="20.32" x2="6.985" y2="21.59" width="0.254" layer="16"/>
 <wire x1="6.985" y1="21.59" x2="9.525" y2="21.59" width="0.254" layer="16"/>
+<wire x1="9.525" y1="21.59" x2="10.795" y2="21.59" width="0.254" layer="16"/>
+<wire x1="10.795" y1="21.59" x2="11.43" y2="22.225" width="0.254" layer="16"/>
+<wire x1="11.43" y1="22.225" x2="15.24" y2="22.225" width="0.254" layer="16"/>
+<wire x1="15.24" y1="22.225" x2="15.875" y2="21.59" width="0.254" layer="16"/>
+<wire x1="15.875" y1="21.59" x2="17.145" y2="21.59" width="0.254" layer="16"/>
 </signal>
 <signal name="C8">
@@
 <wire x1="17.145" y1="39.37" x2="17.145" y2="39.4335" width="0.254" layer="16"/>
 <wire x1="17.145" y1="39.4335" x2="15.621" y2="41.021" width="0.254" layer="16"/>
-<wire x1="15.621" y1="41.021" x2="10.4775" y2="41.021" width="0.254" layer="16"/>
 <wire x1="10.4775" y1="41.021" x2="9.525" y2="40.005" width="0.254" layer="16"/>
 <wire x1="9.525" y1="40.005" x2="9.525" y2="39.37" width="0.254" layer="16"/>
+<wire x1="15.621" y1="41.021" x2="10.4775" y2="41.021" width="0.254" layer="16"/>
 </signal>
 <signal name="N$10">
@@
 <contactref element="R14" pad="1"/>
 <contactref element="Q2" pad="2"/>
-<wire x1="37.465" y1="27.94" x2="33.02" y2="32.385" width="0.254" layer="16"/>
-<wire x1="33.02" y1="32.385" x2="27.305" y2="32.385" width="0.254" layer="16"/>
-<wire x1="36.195" y1="22.86" x2="34.925" y2="24.13" width="0.254" layer="16"/>
-<wire x1="34.925" y1="24.13" x2="34.925" y2="25.4" width="0.254" layer="16"/>
-<wire x1="34.925" y1="25.4" x2="37.465" y2="27.94" width="0.254" layer="16"/>
+<wire x1="34.29" y1="32.385" x2="27.305" y2="32.385" width="0.254" layer="16"/>
+<wire x1="36.195" y1="22.86" x2="35.56" y2="23.495" width="0.254" layer="16"/>
 <wire x1="36.195" y1="22.86" x2="38.735" y2="20.32" width="0.254" layer="16"/>
+<wire x1="35.56" y1="23.495" x2="35.56" y2="27.94" width="0.254" layer="16"/>
+<wire x1="35.56" y1="27.94" x2="35.56" y2="31.115" width="0.254" layer="16"/>
+<wire x1="35.56" y1="31.115" x2="34.29" y2="32.385" width="0.254" layer="16"/>
+<wire x1="37.465" y1="27.94" x2="35.56" y2="27.94" width="0.254" layer="16"/>
 </signal>
 <signal name="N$14">
