File: Vemuran Jan Ray/pcb/jan_ray.brd (EAGLE design)
At the start: 58.9 x 72.4 mm, 39 parts, among them J1 POWER_JACK, X1 2510-

Commit message: 20170505
Parts:
- removed C3: 100n, pedals-capacitors-film:BOX_SMALL
- removed TRIM: 10k, pedals-potentiometers:2262_TRIM
- added R12: 3.9k, pedals-resistors:R0207/3
- C1: device pedals-capacitors-film:BOX_SMALL -> pedals-capacitors-film:050X030_025_2
- C11, C6, C7: device pedals-capacitors-film:050X030_025 -> pedals-capacitors-film:050X030_025_2
- C2: value 47u -> 100u
- IC1: value (none) -> LM4558
- J1: value POWER_JACK -> (none)
- R1: value 100 -> 47
- R3: value 1.5k -> 7.5k
- moved C11 114.9 mm to (45.7, 29.8), turned to 270 degrees
- moved C10 112.3 mm to (47.0, 37.5), turned to 90 degrees
- moved C9 111.7 mm to (29.2, 18.4)
- moved R11 110.3 mm to (43.2, 28.6), turned to 90 degrees
- moved R1 107.8 mm to (35.6, 43.2)
- moved R10 106.1 mm to (48.3, 28.6), turned to 90 degrees
- moved R7 102.5 mm to (13.3, 26.0), turned to 90 degrees
- moved D1 101.7 mm to (34.3, 45.7)
- moved R9 100.0 mm to (50.8, 28.6), turned to 90 degrees
- moved R5 99.8 mm to (29.2, 24.8), turned to 180 degrees
- moved D3 99.7 mm to (8.89, 32.4), turned to 180 degrees
- moved C8 98.2 mm to (29.2, 22.2)
- moved C4 95.3 mm to (37.5, 21.0)
- moved D2 92.1 mm to (8.89, 34.9)
- moved R3 89.5 mm to (39.4, 28.6), turned to 270 degrees
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Connections:
- net +9V: now also X1.5; no longer X1.3
- net GND: now also X1.3; no longer C3.2, X1.5
- net N$10: now also R12.1; no longer TRIM.1
- net N$5: now also R12.2; no longer TRIM.2, TRIM.3
- net VR: no longer C3.1
Routing:
- net N$4: track 0.00 -> 78.0 mm
- net N$6: track 0.00 -> 77.9 mm
- net +9V: track 0.00 -> 67.1 mm, vias 0 -> 1
- net N$2: track 0.00 -> 64.6 mm
- net OUT: track 0.00 -> 62.2 mm
- net GND: track 0.00 -> 36.8 mm
- net N$11: track 0.00 -> 27.6 mm
- net N$14: track 0.00 -> 27.4 mm
- net N$5: track 0.00 -> 26.9 mm
- net N$15: track 0.00 -> 23.2 mm
- net VB: track 0.00 -> 21.2 mm
- net VR: track 0.00 -> 21.2 mm
- net N$16: track 0.00 -> 21.2 mm
- net N$13: track 0.00 -> 16.9 mm
- net IN: track 0.00 -> 15.8 mm
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- added copper zone on layer 1, net GND
Other:
- board size 58.9 x 72.4 mm -> 58.9 x 67.3 mm

Commit message: 20170712
Parts:
- C12, C9: device pedals-capacitors-film:BOX_MED -> pedals-capacitors-film:BOX_BIG
- J1: value (none) -> POWER_JACK
- R12: value 3.9k -> (none); device pedals-resistors:R0207/3 -> pedals-potentiometers:RTRIM3296W
- U$1: device pedals-enclosures:125B -> pedals-pcb:125B_PCB
- moved U$1 32.2 mm to (-0.32, 2.92)
- moved R7 5.39 mm to (17.1, 22.2)
- moved R8 4.02 mm to (9.53, 22.2)
- moved X1 3.81 mm to (29.2, 6.35)
- moved R12 3.59 mm to (13.3, 23.5), turned to 0 degrees
- moved BASS 3.49 mm to (10.8, 13.7)
- moved TREBLE 3.49 mm to (47.6, 13.7)
- moved INPUT 2.98 mm to (15.4, 61.0)
- moved OUTPUT 2.98 mm to (43.1, 61.0)
- moved GAIN 1.02 mm to (10.8, 44.2)
- moved VOLUME 1.02 mm to (47.6, 44.2)
- moved C5 0.64 mm to (22.2, 22.2)
- moved C7 0.64 mm to (22.2, 33.7)
- moved C10 0.63 mm to (47.6, 37.5)
- moved C6 0.63 mm to (19.7, 28.6)
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Connections:
- net N$5: now also R12.3
Routing:
- net N$5: track 26.9 -> 35.4 mm
- net N$2: track 64.6 -> 72.5 mm
- net N$4: track 78.0 -> 85.0 mm
- net N$6: track 77.9 -> 82.8 mm
- net N$12: track 15.1 -> 19.6 mm
- net OUT: track 62.2 -> 66.0 mm
- net +9V: track 67.1 -> 70.7 mm
- net IN: track 15.8 -> 19.4 mm
- net N$13: track 16.9 -> 19.9 mm
- net N$3: track 12.0 -> 10.7 mm
- net N$14: track 27.4 -> 26.3 mm
- net N$16: track 21.2 -> 20.3 mm
- net N$10: track 8.51 -> 7.77 mm
- net VB: track 21.2 -> 21.9 mm
Other:
- board size 58.9 x 67.3 mm -> 59 x 71.3 mm

Commit message: 20170726
Parts:
- moved R6 4.58 mm to (14.6, 33.7), turned to 90 degrees
- moved D4 3.42 mm to (19.7, 33.7), turned to 270 degrees
- moved D2 3.42 mm to (12.1, 33.7), turned to 90 degrees
- moved D3 1.42 mm to (9.53, 33.7), turned to 90 degrees
- moved D5 1.42 mm to (17.1, 33.7), turned to 270 degrees
- moved C2 0.19 mm to (31.9, 39.4)
- moved R1 0.13 mm to (35.7, 43.2)
Routing:
- net N$5: track 35.4 -> 29.4 mm
- net N$8: track 2.54 -> 6.88 mm
- net N$9: track 2.54 -> 6.88 mm
- net N$6: track 82.8 -> 80.2 mm
- net N$11: track 27.2 -> 27.9 mm
- net N$4: track 85.0 -> 84.3 mm
- net N$7: track 5.73 -> 6.26 mm

Commit message: 20170821
Parts:
- R12: value (none) -> 10k
Changed lines of the file:
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@@
 </element>
 <element name="U$1" library="pedals-pcb" package="125B_PCB" value="" x="-0.3175" y="2.921"/>
-<element name="R12" library="pedals-potentiometers" package="RTRIM3296W" value="" x="13.335" y="23.495"/>
+<element name="R12" library="pedals-potentiometers" package="RTRIM3296W" value="10k" x="13.335" y="23.495"/>
 </elements>
 <signals>

Commit message: 20170824
Changed lines of the file:
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@@
 <plain>
 <circle x="25.4" y="27.305" radius="0.547034375" width="0.4064" layer="41"/>
-<wire x1="30.353" y1="36.5125" x2="34.671" y2="36.5125" width="0" layer="41"/>
-<wire x1="34.671" y1="36.5125" x2="37.7825" y2="36.5125" width="0" layer="41"/>
+<wire x1="30.353" y1="36.5125" x2="34.6075" y2="36.5125" width="0" layer="41"/>
+<wire x1="34.6075" y1="36.5125" x2="37.7825" y2="36.5125" width="0" layer="41"/>
 <wire x1="37.7825" y1="36.5125" x2="37.7825" y2="41.275" width="0" layer="41"/>
 <wire x1="30.353" y1="36.5125" x2="30.353" y2="53.34" width="0" layer="41"/>
 <wire x1="37.7825" y1="41.275" x2="34.925" y2="44.45" width="0" layer="41"/>
 <wire x1="34.925" y1="44.45" x2="34.925" y2="46.99" width="0" layer="41"/>
-<wire x1="34.671" y1="36.5125" x2="34.671" y2="19.05" width="0" layer="41"/>
-<wire x1="34.671" y1="19.05" x2="41.275" y2="19.05" width="0" layer="41"/>
+<wire x1="34.6075" y1="36.5125" x2="34.6075" y2="19.05" width="0" layer="41"/>
+<wire x1="34.6075" y1="19.05" x2="41.275" y2="19.05" width="0" layer="41"/>
 <wire x1="41.275" y1="19.05" x2="41.275" y2="44.45" width="0" layer="41"/>
 <wire x1="0" y1="57.15" x2="20.955" y2="57.15" width="0" layer="41"/>

Commit message: 20170914
Parts:
- removed C4: 47u, pedals-capacitors-elec:050_020_1
- added C3: 47u, pedals-capacitors-elec:050_020
- C2: device pedals-capacitors-elec:050_020_1 -> pedals-capacitors-elec:050_020
- D1: device pedals-diodes:DO35-2 -> pedals-diodes:DO41-2
- moved D1 7.43 mm to (27.9, 43.2)
- moved R1 6.96 mm to (29.2, 40.6)
- moved C2 5.97 mm to (36.8, 35.9)
- moved C1 5.75 mm to (30.5, 38.1), turned to 180 degrees
- moved R4 1.42 mm to (20.3, 21.0)
- moved R7 1.42 mm to (17.8, 21.0)
- moved R8 1.42 mm to (10.2, 21.0)
- moved C6 1.42 mm to (20.3, 27.3)
- moved R12 1.42 mm to (14.0, 22.2)
- moved R3 1.27 mm to (38.1, 28.6)
- moved R6 0.90 mm to (15.2, 33.0)
- moved D4 0.64 mm to (20.3, 33.7)
- moved D5 0.64 mm to (17.8, 33.7), turned to 90 degrees
- moved D2 0.63 mm to (12.7, 33.7)
- moved D3 0.63 mm to (10.2, 33.7)
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Connections:
- net GND: now also C3.-; no longer C4.-
- net VB: now also C3.+; no longer C4.+
Routing:
- net GND: track 36.9 -> 0.00 mm
- net +9V: track 70.7 -> 61.6 mm, vias 1 -> 0
- net VR: track 21.1 -> 12.1 mm
- net N$12: track 19.6 -> 15.3 mm
- net N$9: track 6.88 -> 2.54 mm
- net OUT: track 66.0 -> 62.7 mm
- net N$5: track 29.4 -> 27.2 mm
- net N$14: track 26.3 -> 24.3 mm
- net N$13: track 19.9 -> 18.0 mm
- net N$11: track 27.9 -> 26.1 mm
- net N$3: track 10.7 -> 9.42 mm
- net N$16: track 20.3 -> 21.3 mm
- net IN: track 19.4 -> 18.5 mm
- net N$15: track 23.2 -> 22.3 mm
- net N$2: track 72.5 -> 71.8 mm
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- added copper zone on layer 16, net GND

Commit message: 20171003
Parts:
- moved D1 0.32 mm to (27.6, 43.2)
Changed lines of the file:
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@@
 <element name="C8" library="pedals-capacitors-film" package="BOX_SMALL" value="39n" x="29.21" y="22.225"/>
 <element name="C9" library="pedals-capacitors-film" package="BOX_BIG" value="1u" x="29.21" y="17.78"/>
-<element name="D1" library="pedals-diodes" package="DO41-2" value="1N4148" x="27.94" y="43.18"/>
+<element name="D1" library="pedals-diodes" package="DO41-2" value="1N4148" x="27.6225" y="43.18"/>
 <element name="D2" library="pedals-diodes" package="DO35-2" value="1N4148" x="12.7" y="33.655" rot="R90"/>
 <element name="D3" library="pedals-diodes" package="DO35-2" value="1N4148" x="10.16" y="33.655" rot="R90"/>
@@
 <wire x1="32.385" y1="63.5" x2="32.385" y2="46.99" width="0.8128" layer="16"/>
 <wire x1="32.385" y1="46.99" x2="30.48" y2="45.085" width="0.8128" layer="16"/>
-<wire x1="30.48" y1="45.085" x2="30.48" y2="43.18" width="0.8128" layer="16"/>
+<wire x1="30.48" y1="45.085" x2="30.4165" y2="43.18" width="0.8128" layer="16"/>
 <wire x1="27.94" y1="7.62" x2="27.8765" y2="12.7635" width="0.8128" layer="1"/>
 <wire x1="27.8765" y1="12.7635" x2="29.718" y2="14.605" width="0.8128" layer="1"/>
 <wire x1="29.718" y1="14.605" x2="29.718" y2="35.56" width="0.8128" layer="1"/>
 <wire x1="29.718" y1="35.56" x2="30.4165" y2="36.2585" width="0.8128" layer="1"/>
-<wire x1="30.4165" y1="36.2585" x2="30.48" y2="43.18" width="0.8128" layer="1"/>
+<wire x1="30.4165" y1="36.2585" x2="30.4165" y2="43.18" width="0.8128" layer="1"/>
 </signal>
 <signal name="GND">
@@
 </polygon>
 <contactref element="C3" pad="-"/>
+<via x="57.5945" y="61.595" extent="1-16" drill="0.5" diameter="0.85"/>
+<via x="57.5945" y="51.435" extent="1-16" drill="0.5" diameter="0.85"/>
+<via x="10.6045" y="71.3105" extent="1-16" drill="0.5" diameter="0.85"/>
+<via x="21.3995" y="71.3105" extent="1-16" drill="0.5" diameter="0.85"/>
+<via x="30.2895" y="71.3105" extent="1-16" drill="0.5" diameter="0.85"/>
+<via x="0.8255" y="51.435" extent="1-16" drill="0.5" diameter="0.85"/>
+<via x="10.6045" y="61.595" extent="1-16" drill="0.5" diameter="0.85"/>
+<via x="10.6045" y="51.435" extent="1-16" drill="0.5" diameter="0.85"/>
+<via x="21.3995" y="51.435" extent="1-16" drill="0.5" diameter="0.85"/>
+<via x="30.2895" y="62.23" extent="1-16" drill="0.5" diameter="0.85"/>
+<via x="30.2895" y="51.435" extent="1-16" drill="0.5" diameter="0.85"/>
+<via x="37.2745" y="71.3105" extent="1-16" drill="0.5" diameter="0.85"/>
+<via x="46.7995" y="71.3105" extent="1-16" drill="0.5" diameter="0.85"/>
+<via x="37.2745" y="61.595" extent="1-16" drill="0.5" diameter="0.85"/>
+<via x="37.2745" y="51.435" extent="1-16" drill="0.5" diameter="0.85"/>
+<via x="46.7995" y="61.595" extent="1-16" drill="0.5" diameter="0.85"/>
+<via x="46.7995" y="51.435" extent="1-16" drill="0.5" diameter="0.85"/>
+<via x="57.5945" y="41.275" extent="1-16" drill="0.5" diameter="0.85"/>
+<via x="57.5945" y="31.115" extent="1-16" drill="0.5" diameter="0.85"/>
+<via x="57.5945" y="20.955" extent="1-16" drill="0.5" diameter="0.85"/>
+<via x="57.5945" y="10.795" extent="1-16" drill="0.5" diameter="0.85"/>
+<via x="57.5945" y="2.9845" extent="1-16" drill="0.5" diameter="0.85"/>
+<via x="49.53" y="2.9845" extent="1-16" drill="0.5" diameter="0.85"/>
+<via x="39.37" y="2.9845" extent="1-16" drill="0.5" diameter="0.85"/>
+<via x="29.21" y="2.9845" extent="1-16" drill="0.5" diameter="0.85"/>
+<via x="19.05" y="2.9845" extent="1-16" drill="0.5" diameter="0.85"/>
+<via x="8.89" y="2.9845" extent="1-16" drill="0.5" diameter="0.85"/>
+<via x="0.8255" y="2.9845" extent="1-16" drill="0.5" diameter="0.85"/>
+<via x="0.8255" y="61.595" extent="1-16" drill="0.5" diameter="0.85"/>
+<via x="0.8255" y="41.275" extent="1-16" drill="0.5" diameter="0.85"/>
+<via x="0.8255" y="31.115" extent="1-16" drill="0.5" diameter="0.85"/>
+<via x="0.8255" y="20.955" extent="1-16" drill="0.5" diameter="0.85"/>
+<via x="0.8255" y="10.795" extent="1-16" drill="0.5" diameter="0.85"/>
+<via x="39.37" y="6.1595" extent="1-16" drill="0.5" diameter="0.85"/>
+<via x="49.53" y="6.1595" extent="1-16" drill="0.5" diameter="0.85"/>
+<via x="39.37" y="9.3345" extent="1-16" drill="0.5" diameter="0.85"/>
+<via x="49.53" y="9.3345" extent="1-16" drill="0.5" diameter="0.85"/>
+<via x="19.05" y="9.3345" extent="1-16" drill="0.5" diameter="0.85"/>
+<via x="21.59" y="9.3345" extent="1-16" drill="0.5" diameter="0.85"/>
+<via x="8.89" y="8.6995" extent="1-16" drill="0.5" diameter="0.85"/>
+<via x="13.335" y="11.2395" extent="1-16" drill="0.5" diameter="0.85"/>
+<via x="13.335" y="13.7795" extent="1-16" drill="0.5" diameter="0.85"/>
+<via x="53.7845" y="10.795" extent="1-16" drill="0.5" diameter="0.85"/>
+<via x="53.7845" y="20.955" extent="1-16" drill="0.5" diameter="0.85"/>
+<via x="53.7845" y="31.115" extent="1-16" drill="0.5" diameter="0.85"/>
+<via x="49.3395" y="41.275" extent="1-16" drill="0.5" diameter="0.85"/>
+<via x="26.543" y="11.2395" extent="1-16" drill="0.5" diameter="0.85"/>
+<via x="29.21" y="11.2395" extent="1-16" drill="0.5" diameter="0.85"/>
+<via x="33.655" y="20.1295" extent="1-16" drill="0.5" diameter="0.85"/>
+<via x="27.305" y="20.1295" extent="1-16" drill="0.5" diameter="0.85"/>
+<via x="31.115" y="31.115" extent="1-16" drill="0.5" diameter="0.85"/>
+<via x="27.3685" y="31.115" extent="1-16" drill="0.5" diameter="0.85"/>
+<via x="50.165" y="13.7795" extent="1-16" drill="0.5" diameter="0.85"/>
+<via x="39.37" y="14.4145" extent="1-16" drill="0.5" diameter="0.85"/>
+<via x="16.51" y="19.4945" extent="1-16" drill="0.5" diameter="0.85"/>
+<via x="8.3185" y="41.91" extent="1-16" drill="0.5" diameter="0.85"/>
+<via x="8.3185" y="44.45" extent="1-16" drill="0.5" diameter="0.85"/>
+<via x="14.0335" y="38.735" extent="1-16" drill="0.5" diameter="0.85"/>
+<via x="14.6685" y="31.115" extent="1-16" drill="0.5" diameter="0.85"/>
+<via x="12.7635" y="27.305" extent="1-16" drill="0.5" diameter="0.85"/>
+<via x="3.3655" y="51.435" extent="1-16" drill="0.5" diameter="0.85"/>
+<via x="2.921" y="41.275" extent="1-16" drill="0.5" diameter="0.85"/>
+<via x="2.921" y="31.115" extent="1-16" drill="0.5" diameter="0.85"/>
+<via x="2.921" y="20.955" extent="1-16" drill="0.5" diameter="0.85"/>
+<via x="40.64" y="26.2255" extent="1-16" drill="0.5" diameter="0.85"/>
+<via x="45.085" y="30.48" extent="1-16" drill="0.5" diameter="0.85"/>
+<via x="42.545" y="29.21" extent="1-16" drill="0.5" diameter="0.85"/>
+<via x="31.75" y="41.91" extent="1-16" drill="0.5" diameter="0.85"/>
+<via x="29.1465" y="41.91" extent="1-16" drill="0.5" diameter="0.85"/>
+<via x="19.05" y="15.6845" extent="1-16" drill="0.5" diameter="0.85"/>
+<via x="22.86" y="15.0495" extent="1-16" drill="0.5" diameter="0.85"/>
+<via x="21.3995" y="61.595" extent="1-16" drill="0.5" diameter="0.85"/>
+<via x="16.5735" y="33.655" extent="1-16" drill="0.5" diameter="0.85"/>
+<via x="22.2885" y="33.02" extent="1-16" drill="0.5" diameter="0.85"/>
 </signal>
 <signal name="N$1">
 <contactref element="D1" pad="C"/>
 <contactref element="R1" pad="1"/>
-<wire x1="25.4" y1="43.18" x2="25.4" y2="40.64" width="0.8128" layer="16"/>
+<wire x1="24.892" y1="43.18" x2="24.892" y2="41.148" width="0.8128" layer="16"/>
+<wire x1="24.892" y1="41.148" x2="25.4" y2="40.64" width="0.8128" layer="16"/>
 </signal>
 <signal name="VR">
