File: Vemuran Jan Ray/pcb/jan_ray.sch (EAGLE design)
At the start: 37 parts, among them IC1 LM4558, J1 POWER_JACK, X1 2510-

Commit message: 20170712
Parts:
- C12, C9: device pedals-capacitors-film:CER/FILMBOX.2 -> pedals-capacitors-film:CER/FILMBOX.3
- R12: value 3.9k -> (none); device pedals-resistors:R_.3B -> pedals-potentiometers:R-TRIMM3296W
Connections:
- net N$10: now also R12.A; no longer R12.1
- net N$5: now also R12.E, R12.S; no longer R12.2

Commit message: 20170821
Parts:
- R12: value (none) -> 10k
Changed lines of the file:
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@@
 <part name="GND9" library="pedals-supply" deviceset="GND" device=""/>
 <part name="V3" library="pedals-supply" deviceset="+9V" device=""/>
-<part name="R12" library="pedals-potentiometers" deviceset="R-TRIMM" device="3296W"/>
+<part name="R12" library="pedals-potentiometers" deviceset="R-TRIMM" device="3296W" value="10k"/>
 </parts>
 <sheets>

Commit message: 20170914
Parts:
- removed C4: 47u, pedals-capacitors-elec:0501
- added C3: 47u, pedals-capacitors-elec:0500
- C2: device pedals-capacitors-elec:0501 -> pedals-capacitors-elec:0500
- D1: device pedals-diodes:DO35.2 -> pedals-diodes:DO41.2
Connections:
- net GND: now also C3.-; no longer C4.-
- net VB: now also C3.+; no longer C4.+

Commit message: 20171009
Parts:
- D1: value 1N4148 -> 1N4002
Connections:
- removed net N$1: D1.C, R1.1
- net +9V: now also D1.C, R1.1; no longer D1.A
- net GND: now also D1.A
Other:
- moved on the sheet: D1
Changed lines of the file:
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@@
 <setting verticaltext="up"/>
 </settings>
-<grid distance="0.1" unitdist="inch" unit="inch" style="lines" multiple="1" display="no" altdistance="0.01" altunitdist="inch" altunit="inch"/>
+<grid distance="0.1" unitdist="inch" unit="inch" style="lines" multiple="1" display="yes" altdistance="0.01" altunitdist="inch" altunit="inch"/>
 <layers>
 <layer number="1" name="Top" color="4" fill="1" visible="no" active="no"/>
@@
 <part name="GND1" library="pedals-supply" deviceset="GND" device=""/>
 <part name="V2" library="pedals-supply" deviceset="+9V" device=""/>
-<part name="D1" library="pedals-diodes" deviceset="DO41" device=".2" value="1N4148"/>
+<part name="D1" library="pedals-diodes" deviceset="DO41" device=".2" value="1N4002"/>
 <part name="R1" library="pedals-resistors" deviceset="R_" device=".3B" value="47"/>
 <part name="C1" library="pedals-capacitors-film" deviceset="CER/FILM" device="2" value="100n"/>
@@
 <part name="R12" library="pedals-potentiometers" deviceset="R-TRIMM" device="3296W" value="10k"/>
 <part name="C3" library="pedals-capacitors-elec" deviceset="050" device="0" value="47u"/>
+<part name="GND4" library="pedals-supply" deviceset="GND" device=""/>
 </parts>
 <sheets>
@@
 <instance part="V1" gate="+9V" x="-35.56" y="78.74" rot="R180"/>
 <instance part="GND1" gate="GND" x="-30.48" y="78.74"/>
-<instance part="V2" gate="+9V" x="-12.7" y="93.98" rot="R90"/>
-<instance part="D1" gate="G$1" x="-2.54" y="93.98"/>
+<instance part="V2" gate="+9V" x="-5.08" y="93.98" rot="R90"/>
+<instance part="D1" gate="G$1" x="0" y="88.9" rot="R90"/>
 <instance part="R1" gate="G$1" x="7.62" y="93.98"/>
 <instance part="C1" gate="G$1" x="15.24" y="86.36" rot="R90"/>
@@
 <instance part="R12" gate="G$1" x="38.1" y="20.32" rot="R270"/>
 <instance part="C3" gate="1" x="58.42" y="88.9" rot="R270"/>
+<instance part="GND4" gate="GND" x="0" y="76.2"/>
 </instances>
 <busses>
@@
 </segment>
 <segment>
-<pinref part="V2" gate="+9V" pin="+9V"/>
-<pinref part="D1" gate="G$1" pin="A"/>
-<wire x1="-10.16" y1="93.98" x2="-7.62" y2="93.98" width="0.1524" layer="91"/>
-</segment>
-<segment>
 <pinref part="X1" gate="-5" pin="KL"/>
 <wire x1="-27.94" y1="53.34" x2="-22.86" y2="53.34" width="0.1524" layer="91"/>
 <pinref part="V3" gate="+9V" pin="+9V"/>
+</segment>
+<segment>
+<pinref part="V2" gate="+9V" pin="+9V"/>
+<pinref part="R1" gate="G$1" pin="1"/>
+<wire x1="-2.54" y1="93.98" x2="0" y2="93.98" width="0.1524" layer="91"/>
+<pinref part="D1" gate="G$1" pin="C"/>
+<wire x1="0" y1="93.98" x2="2.54" y2="93.98" width="0.1524" layer="91"/>
+<wire x1="0" y1="91.44" x2="0" y2="93.98" width="0.1524" layer="91"/>
+<junction x="0" y="93.98"/>
 </segment>
 </net>
@@
 <pinref part="GND9" gate="GND" pin="GND"/>
 </segment>
+<segment>
+<pinref part="GND4" gate="GND" pin="GND"/>
+<pinref part="D1" gate="G$1" pin="A"/>
+<wire x1="0" y1="78.74" x2="0" y2="83.82" width="0.1524" layer="91"/>
+</segment>
 </net>
-<net name="N$1" class="0">
-<segment>
-<pinref part="D1" gate="G$1" pin="C"/>
-<pinref part="R1" gate="G$1" pin="1"/>
-<wire x1="0" y1="93.98" x2="2.54" y2="93.98" width="0.1524" layer="91"/>
-</segment>
-</net>
