File: Klon Centaur/pcb/klon.sch (EAGLE design)
At the start: 50 parts, among them IC1 ICL7660CPA, IC2 TL072, J1 POWER_JACK, X1 2510-

Commit message: 20171102
Parts:
- removed GAIN: 250kB, pedals-potentiometers:POTS16MM
- removed PRESENCE: 50kB, pedals-potentiometers:POTS16MM
- removed TONE: 25kB, pedals-potentiometers:POTS16MM
- removed X1: 2510-, pedals-headers:2510-
- added C19: 2.2n, pedals-capacitors-film:CER/FILMBOX.1
- added C20: 27n, pedals-capacitors-film:CER/FILMBOX.1
- added C21: 820p, pedals-capacitors-film:CER/FILM2
- added C22: 3.9n, pedals-capacitors-film:CER/FILMBOX.1
- added C23, C24: 4.7u, pedals-capacitors-elec:0500
- added D8: LEDA, pedals-diodes:LEDA
- added GAIN1, GAIN2: 100kB, pedals-potentiometers:POTS16MM
- added IC3: TL072, pedals-integrated circuits:DUALTH
- added R15: 1.5k, pedals-resistors:R_.3B
- added R16: 1k, pedals-resistors:R_.3B
- added R17: 22k, pedals-resistors:R_.3B
- added R18: 27k, pedals-resistors:R_.3B
- added R19: 12k, pedals-resistors:R_.3B
- added R20: 392k, pedals-resistors:R_.3B
- added R21: 1.8k, pedals-resistors:R_.3B
- added R22, R23, R26, R29: 100k, pedals-resistors:R_.3B
- added R24, R28: 4.7k, pedals-resistors:R_.3B
- added R25, R27: 560, pedals-resistors:R_.3B
- added R30, R31: 68k, pedals-resistors:R_.3B
- added SW2: (no value), pedals-switches:DPDTPADS
- added TREBLE: 10kB, pedals-potentiometers:POTS16MM
- C11: value 10u -> 68n; device pedals-capacitors-elec:0500 -> pedals-capacitors-film:CER/FILMBOX.1
- C12: value 68n -> 82n
- C13: value 82n -> 390p; device pedals-capacitors-film:CER/FILMBOX.1 -> pedals-capacitors-film:CER/FILM2
- C14: value 390p -> 1u; device pedals-capacitors-film:CER/FILM2 -> pedals-capacitors-elec:0400
- C17: value 1u -> 68n; device pedals-capacitors-elec:0400 -> pedals-capacitors-film:CER/FILMBOX.1
- C18: value 68n -> 390n; device pedals-capacitors-film:CER/FILMBOX.1 -> pedals-capacitors-film:CER/FILMBOX.2
- VOLUME: value 100kA -> 10kB
Connections:
- removed net N$2: INPUT.T, X1-7.KL
- removed net N$4: OUTPUT.T, X1-1.KL
- new net N$23: GAIN1.3, R15.1, R16.1
- new net N$24: C18.2, R16.2
- new net N$25: GAIN1.2, R17.1, R18.1, R19.1
- new net N$26: C19.2, R17.2
- new net N$27: C20.1, C21.2, IC3_A.-IN, R11.2, R13.2, R18.2, R20.1
- new net N$28: C20.2, R19.2
- new net N$29: R21.2, TREBLE.1
- new net N$30: R24.1, TREBLE.3
- new net N$31: C22.1, IC3_B.-IN, R22.2, R23.1
- new net N$32: C22.2, TREBLE.2
- new net N$33: C23.+, IC3_B.OUT, R23.2, R24.2
- new net N$34: C24.-, R26.2, R27.1
- new net N$35: R27.2, R31.1, SW2_A.3
- new net N$36: D8.C, SW2_B.1
- new net N$37: D8.A, R28.2
- new net N$40: C23.-, R25.1
- new net N$41: R25.2, VOLUME.3
- new net N$42: R30.1, SW2_A.1, VOLUME.2
- net +9V: now also R28.1; no longer X1-5.KL
- net -VC: now also IC3_PWR.V-
- net GND: now also C16.-, R26.1, R29.1, SW2_B.2, VOLUME.1; no longer C17.-, X1-3.KL
- net IN: now also INPUT.T; no longer X1-8.KL
- net N$10: now also C11.1, GAIN2.1; no longer C12.1, TONE.1
- net N$12: now also GAIN2.3; no longer TONE.3
- net N$13: now also C12.2; no longer C13.2
- net N$14: now also C12.1, C13.2; no longer C13.1, C14.2
- net N$16: now also C13.1, C14.+; no longer C14.1, C15.+
- net N$17: now also C15.+, C19.1; no longer C16.-
- net N$18: now also C14.-; no longer C15.-
- net N$19: now also C15.-, SW2_B.3; no longer C16.+
- net N$20: now also C16.+; no longer C17.+
- net N$21: now also C21.1, IC3_A.OUT, R20.2, R21.1, R22.1; no longer R11.2, R13.2
- net N$22: now also C17.2, C18.1, GAIN1.1, R15.2; no longer C18.2
- net N$8: now also C17.1, C24.+; no longer C18.1
- net N$9: now also C11.2; no longer C12.2
- net OUT: now also OUTPUT.T, R29.2, R30.2, R31.2, SW2_A.2; no longer X1-2.KL
- net VB: now also GAIN2.2, IC3_A.+IN, IC3_B.+IN; no longer TONE.2
- net VC: now also IC3_PWR.V+
Other:
- moved on the sheet: C10, C12, C13, C15, C16, C18, C9, D4, D5, D6, D7, IC2_A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
