File: Mad Professor Deep Blue Delay/pcb/deepblue.sch (EAGLE design)
At the start: 55 parts, among them IC1 TL072, IC2 PT2399, J2 POWER_JACK, X1 2510-

Commit message: 20170914
Parts:
- added C26: 100n, pedals-capacitors-film:CER/FILM2
- C2, C3: device pedals-capacitors-elec:0400 -> pedals-capacitors-elec:0500
- C5: value 100n -> 10u; device pedals-capacitors-film:CER/FILM2 -> pedals-capacitors-elec:0500
- C6: device pedals-capacitors-elec:0400 -> pedals-capacitors-film:CER/FILM1
Connections:
- net GND: now also C26.1, C5.-, C6.1; no longer C5.1, C6.-
- net VC: now also C26.2, C5.+, C6.2; no longer C5.2, C6.+
Other:
- moved on the sheet: C1, C10, C11, C12, C13, C14, C15, C16, C17, C18, C19, C2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

Commit message: 20171216
Parts:
- removed TONE: 100kB, pedals-potentiometers:POTS16MM
- added DELAY: 50kB, pedals-potentiometers:POTS16MM
- added R20: 1.5k, pedals-resistors:R_.3B
- C10, C11, C12, C13, C14, C16, C17, C18, C19, C20, C22, C7: device pedals-capacitors-film:CER/FILM2 -> pedals-capacitors-film:CER/FILMBOX.1
- C15: device pedals-capacitors-elec:0631 -> pedals-capacitors-elec:0500
- C4: device pedals-capacitors-elec:0400 -> pedals-capacitors-elec:0500
- R14: value 5k -> 5.1k
Connections:
- removed net DGND: IC2.DGND
- new net N$28: DELAY.1, IC2.DGND
- new net N$29: DELAY.2, DELAY.3, R20.1
- new net N$30: IC2.VCO, R20.2
