File: #Misc/BBE Green Screamer/greenscreamer_redraw.sch (EAGLE design)
At the start: 27 parts, among them U1 TL072

Commit message: 20180125
Other:
- note added: "GAIN"
- note added: "TONE"
- note added: "VOLUME"
Changed lines of the file:
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@@
 <?xml version="1.0" encoding="utf-8"?>
 <!DOCTYPE eagle SYSTEM "eagle.dtd">
-<eagle version="8.2.0">
+<eagle version="8.5.1">
 <drawing>
 <settings>
 <setting alwaysvectorfont="no"/>
+<setting keepoldvectorfont="yes"/>
 <setting verticaltext="up"/>
 </settings>
-<grid distance="0.1" unitdist="inch" unit="inch" style="lines" multiple="1" display="yes" altdistance="0.01" altunitdist="inch" altunit="inch"/>
+<grid distance="0.1" unitdist="inch" unit="inch" style="lines" multiple="1" display="no" altdistance="0.01" altunitdist="inch" altunit="inch"/>
 <layers>
 <layer number="1" name="Top" color="4" fill="1" visible="no" active="no"/>
@@
 <sheet>
 <plain>
+<text x="91.44" y="99.06" size="1.778" layer="95">GAIN</text>
+<text x="127" y="91.44" size="1.778" layer="95">TONE</text>
+<text x="172.72" y="48.26" size="1.778" layer="95">VOLUME</text>
 </plain>
 <instances>
