File: #Misc/DOD Supra Distortion/supra_redraw.sch (EAGLE design)
At the start: 66 parts, among them Q1 J113, Q2 J113, Q3 2N3904, U1 MC1458, U2 LF353, U3 CD4007

Commit message: 20180125
Parts:
- removed 1101: BATTERY, pedals-jacks:BATTERY
- removed DCJACK: (no value), pedals-jacks:DC_KOBICONN
- removed IN: (no value), pedals-jacks:STEREO
- removed OUT: (no value), pedals-jacks:MONO
Connections:
- removed net N$1: 1101.P$1, DCJACK.R
- removed net N$10: C14.-, OUT.TIP, R11.2
- removed net N$2: C15.+, D7.C, DCJACK.S, R12.1
- removed net N$3: 1101.P$2, IN.R
- removed net N$4: C1.2, IN.T
- new net +9V: C15.+, D7.C, R12.1
- new net IN: C1.2
- new net OUT: C14.-, R11.2
- net GND: no longer DCJACK.T, IN.S, OUT.SLEEVE
Changed lines of the file:
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@@
 <?xml version="1.0" encoding="utf-8"?>
 <!DOCTYPE eagle SYSTEM "eagle.dtd">
-<eagle version="8.2.0">
+<eagle version="8.5.1">
 <drawing>
 <settings>
 <setting alwaysvectorfont="no"/>
+<setting keepoldvectorfont="yes"/>
 <setting verticaltext="up"/>
 </settings>
-<grid distance="0.1" unitdist="inch" unit="inch" style="lines" multiple="1" display="yes" altdistance="0.01" altunitdist="inch" altunit="inch"/>
+<grid distance="0.1" unitdist="inch" unit="inch" style="lines" multiple="1" display="no" altdistance="0.01" altunitdist="inch" altunit="inch"/>
 <layers>
 <layer number="1" name="Top" color="4" fill="1" visible="no" active="no"/>
@@
 <layer number="59" name="tCarbon" color="7" fill="1" visible="no" active="no"/>
 <layer number="60" name="bCarbon" color="7" fill="1" visible="no" active="no"/>
+<layer number="88" name="SimResults" color="9" fill="1" visible="yes" active="yes"/>
+<layer number="89" name="SimProbes" color="9" fill="1" visible="yes" active="yes"/>
 <layer number="90" name="Modules" color="5" fill="1" visible="yes" active="yes"/>
 <layer number="91" name="Nets" color="2" fill="1" visible="yes" active="yes"/>
@@
 </classes>
 <parts>
-<part name="DCJACK" library="pedals-jacks" deviceset="DC_KOBICONN" device=""/>
-<part name="GND102" library="gm-supply" deviceset="GND" device=""/>
-<part name="1101" library="pedals-jacks" deviceset="BATTERY" device=""/>
 <part name="R12" library="pedals-resistors" deviceset="R_" device=".3B" value="100R"/>
 <part name="D7" library="pedals-diodes" deviceset="DO35" device=".2" value="1N4148"/>
@@
 <part name="VR101" library="gm-supply" deviceset="VR" device=""/>
 <part name="VB102" library="gm-supply" deviceset="VB" device=""/>
-<part name="IN" library="pedals-jacks" deviceset="STEREO" device=""/>
-<part name="GND101" library="gm-supply" deviceset="GND" device=""/>
 <part name="C1" library="pedals-capacitors-film" deviceset="CER/FILM" device="BOX.1" value="10n"/>
 <part name="C21" library="pedals-capacitors-film" deviceset="CER/FILM" device="BOX.1" value="120p"/>
@@
 <part name="R11" library="pedals-resistors" deviceset="R_" device=".3B" value="100k"/>
 <part name="GND105" library="gm-supply" deviceset="GND" device=""/>
-<part name="OUT" library="pedals-jacks" deviceset="MONO" device=""/>
-<part name="GND103" library="gm-supply" deviceset="GND" device=""/>
 <part name="U2" library="pedals-integrated circuits" deviceset="DUAL" device="TH" value="LF353"/>
 <part name="C3" library="pedals-capacitors-film" deviceset="CER/FILM" device="BOX.1" value="120p"/>
@@
 <part name="R24" library="pedals-resistors" deviceset="R_" device=".3B" value="100k"/>
 <part name="GND1" library="gm-supply" deviceset="GND" device=""/>
+<part name="IN" library="pedals-supply" deviceset="IN" device=""/>
+<part name="OUT" library="pedals-supply" deviceset="OUT" device=""/>
+<part name="V1" library="pedals-supply" deviceset="+9V" device=""/>
 </parts>
 <sheets>
@@
 </plain>
 <instances>
-<instance part="DCJACK" gate="G$1" x="-33.02" y="53.34" rot="MR180"/>
-<instance part="GND102" gate="GND" x="-20.32" y="45.72"/>
-<instance part="1101" gate="G$1" x="-15.24" y="66.04" rot="R180"/>
 <instance part="R12" gate="G$1" x="7.62" y="55.88"/>
 <instance part="D7" gate="G$1" x="-10.16" y="50.8" rot="R90"/>
@@
 <instance part="VR101" gate="G$1" x="30.48" y="55.88" rot="R270"/>
 <instance part="VB102" gate="G$1" x="30.48" y="35.56" rot="R270"/>
-<instance part="IN" gate="G$1" x="-35.56" y="86.36" rot="MR180"/>
-<instance part="GND101" gate="GND" x="-20.32" y="76.2"/>
 <instance part="C1" gate="G$1" x="-1.27" y="86.36"/>
 <instance part="C21" gate="G$1" x="5.08" y="80.01" rot="R90"/>
@@
 <instance part="R11" gate="G$1" x="254" y="50.8" rot="MR90"/>
 <instance part="GND105" gate="GND" x="254" y="40.64" rot="MR0"/>
-<instance part="OUT" gate="G$1" x="276.86" y="55.88" rot="MR0"/>
-<instance part="GND103" gate="GND" x="269.24" y="48.26" rot="MR0"/>
 <instance part="U2" gate="_A" x="83.82" y="63.5" rot="MR180"/>
 <instance part="U2" gate="_B" x="182.88" y="55.88" rot="MR180"/>
@@
 <instance part="R24" gate="G$1" x="68.58" y="-15.24" rot="MR270"/>
 <instance part="GND1" gate="GND" x="111.76" y="-15.24" rot="R90"/>
+<instance part="IN" gate="G$1" x="-10.16" y="86.36"/>
+<instance part="OUT" gate="G$1" x="259.08" y="58.42"/>
+<instance part="V1" gate="+9V" x="-10.16" y="60.96"/>
 </instances>
 <busses>
@@
 <net name="GND" class="0">
 <segment>
-<pinref part="DCJACK" gate="G$1" pin="T"/>
-<pinref part="GND102" gate="GND" pin="GND"/>
-<wire x1="-22.86" y1="50.8" x2="-20.32" y2="50.8" width="0.1524" layer="91"/>
-<wire x1="-20.32" y1="50.8" x2="-20.32" y2="48.26" width="0.1524" layer="91"/>
-</segment>
-<segment>
 <pinref part="GND104" gate="GND" pin="GND"/>
 <pinref part="D7" gate="G$1" pin="A"/>
@@
 </segment>
 <segment>
-<pinref part="IN" gate="G$1" pin="S"/>
-<pinref part="GND101" gate="GND" pin="GND"/>
-<wire x1="-22.86" y1="81.28" x2="-20.32" y2="81.28" width="0.1524" layer="91"/>
-<wire x1="-20.32" y1="81.28" x2="-20.32" y2="78.74" width="0.1524" layer="91"/>
-</segment>
-<segment>
 <pinref part="U1" gate="_PWR" pin="V-"/>
 <pinref part="GND111" gate="GND" pin="GND"/>
@@
 <pinref part="C21" gate="G$1" pin="2"/>
 <wire x1="5.08" y1="71.12" x2="5.08" y2="76.2" width="0.1524" layer="91"/>
-</segment>
-<segment>
-<pinref part="OUT" gate="G$1" pin="SLEEVE"/>
-<pinref part="GND103" gate="GND" pin="GND"/>
-<wire x1="271.78" y1="53.34" x2="269.24" y2="53.34" width="0.1524" layer="91"/>
-<wire x1="269.24" y1="53.34" x2="269.24" y2="50.8" width="0.1524" layer="91"/>
 </segment>
 <segment>
@@
 </segment>
 </net>
-<net name="N$1" class="0">
-<segment>
-<pinref part="DCJACK" gate="G$1" pin="R"/>
-<pinref part="1101" gate="G$1" pin="P$1"/>
-<wire x1="-22.86" y1="53.34" x2="-15.24" y2="53.34" width="0.1524" layer="91"/>
-<wire x1="-15.24" y1="53.34" x2="-15.24" y2="60.96" width="0.1524" layer="91"/>
-</segment>
-</net>
-<net name="N$2" class="0">
-<segment>
-<pinref part="DCJACK" gate="G$1" pin="S"/>
-<pinref part="R12" gate="G$1" pin="1"/>
-<wire x1="-22.86" y1="55.88" x2="-10.16" y2="55.88" width="0.1524" layer="91"/>
-<pinref part="D7" gate="G$1" pin="C"/>
-<wire x1="-10.16" y1="55.88" x2="0" y2="55.88" width="0.1524" layer="91"/>
-<wire x1="0" y1="55.88" x2="2.54" y2="55.88" width="0.1524" layer="91"/>
-<wire x1="-10.16" y1="53.34" x2="-10.16" y2="55.88" width="0.1524" layer="91"/>
-<pinref part="C15" gate="1" pin="+"/>
-<wire x1="0" y1="53.34" x2="0" y2="55.88" width="0.1524" layer="91"/>
-<junction x="-10.16" y="55.88"/>
-<junction x="0" y="55.88"/>
-</segment>
-</net>
 <net name="VB" class="0">
 <segment>
@@
 <pinref part="R17" gate="G$1" pin="2"/>
 <wire x1="96.52" y1="0" x2="96.52" y2="-2.54" width="0.1524" layer="91"/>
-</segment>
-</net>
-<net name="N$3" class="0">
-<segment>
-<pinref part="1101" gate="G$1" pin="P$2"/>
-<wire x1="-15.24" y1="71.12" x2="-15.24" y2="83.82" width="0.1524" layer="91"/>
-<pinref part="IN" gate="G$1" pin="R"/>
-<wire x1="-22.86" y1="83.82" x2="-15.24" y2="83.82" width="0.1524" layer="91"/>
-</segment>
-</net>
-<net name="N$4" class="0">
-<segment>
-<pinref part="IN" gate="G$1" pin="T"/>
-<pinref part="C1" gate="G$1" pin="2"/>
-<wire x1="-22.86" y1="86.36" x2="-5.08" y2="86.36" width="0.1524" layer="91"/>
 </segment>
 </net>
@@
 <pinref part="C10" gate="1" pin="+"/>
 <wire x1="58.42" y1="30.48" x2="58.42" y2="33.02" width="0.1524" layer="91"/>
-</segment>
-</net>
-<net name="N$10" class="0">
-<segment>
-<pinref part="OUT" gate="G$1" pin="TIP"/>
-<pinref part="C14" gate="1" pin="-"/>
-<wire x1="271.78" y1="58.42" x2="254" y2="58.42" width="0.1524" layer="91"/>
-<pinref part="R11" gate="G$1" pin="2"/>
-<wire x1="254" y1="58.42" x2="251.46" y2="58.42" width="0.1524" layer="91"/>
-<wire x1="254" y1="55.88" x2="254" y2="58.42" width="0.1524" layer="91"/>
-<junction x="254" y="58.42"/>
 </segment>
 </net>
@@
 </segment>
 </net>
+<net name="IN" class="0">
+<segment>
+<pinref part="C1" gate="G$1" pin="2"/>
+<pinref part="IN" gate="G$1" pin="IN"/>
+<wire x1="-7.62" y1="86.36" x2="-5.08" y2="86.36" width="0.1524" layer="91"/>
+</segment>
+</net>
+<net name="OUT" class="0">
+<segment>
+<pinref part="C14" gate="1" pin="-"/>
+<pinref part="R11" gate="G$1" pin="2"/>
+<wire x1="254" y1="58.42" x2="251.46" y2="58.42" width="0.1524" layer="91"/>
+<wire x1="254" y1="55.88" x2="254" y2="58.42" width="0.1524" layer="91"/>
+<pinref part="OUT" gate="G$1" pin="OUT"/>
+<wire x1="254" y1="58.42" x2="256.54" y2="58.42" width="0.1524" layer="91"/>
+<junction x="254" y="58.42"/>
+</segment>
+</net>
+<net name="+9V" class="0">
+<segment>
+<pinref part="R12" gate="G$1" pin="1"/>
+<pinref part="D7" gate="G$1" pin="C"/>
+<wire x1="-10.16" y1="55.88" x2="0" y2="55.88" width="0.1524" layer="91"/>
+<wire x1="0" y1="55.88" x2="2.54" y2="55.88" width="0.1524" layer="91"/>
+<wire x1="-10.16" y1="53.34" x2="-10.16" y2="55.88" width="0.1524" layer="91"/>
+<pinref part="C15" gate="1" pin="+"/>
+<wire x1="0" y1="53.34" x2="0" y2="55.88" width="0.1524" layer="91"/>
+<junction x="0" y="55.88"/>
+<pinref part="V1" gate="+9V" pin="+9V"/>
+<wire x1="-10.16" y1="55.88" x2="-10.16" y2="58.42" width="0.1524" layer="91"/>
+<junction x="-10.16" y="55.88"/>
+</segment>
+</net>
