File: #Misc/Ibanez MT10/mt10.sch (EAGLE design)
At the start: 39 parts, among them IC1 MC1458P, IC2 MC1458P

Commit message: 20180102
Parts:
- removed AC_ADAPTOR: DCJACK, pedals-jacks:DC_KOBICONN
- removed BATTERY: BATTERY, pedals-jacks:BATTERY
- removed IC2: MC1458P, pedals-integrated circuits:DUALTH
- removed OUTPUT: (no value), pedals-jacks:MONO
- removed POT1: 500kA, pedals-potentiometers:POTS16MM
- removed POT2: 20kA, pedals-potentiometers:POTS16MM
- removed POT3: 100kB, pedals-potentiometers:POTS16MM
- added 1101: BATTERY, pedals-jacks:BATTERY
- added C12, C13: 1u, pedals-capacitors-elec:0500
- added C14, C15: 100n, pedals-capacitors-film:CER/FILMBOX.1
- added C16: 10u, pedals-capacitors-elec:0500
- added C17, C18: 47n, pedals-capacitors-film:CER/FILMBOX.1
- added C19, C20, C21: 1n, pedals-capacitors-film:CER/FILMBOX.1
- added C22: 100u, pedals-capacitors-elec:0500
- added C23: 47u, pedals-capacitors-elec:0500
- added D4, D5, D6: MA165, pedals-diodes:DO35.2
- added D7: (no value), pedals-diodes:DO35.2
- added JK2: INPUT, pedals-jacks:STEREO3PADS
- added JK3: DCJACK, pedals-jacks:DC_KOBICONN
- added LED1: LED, pedals-diodes:LED
- added Q1, Q2: K246Y, pedals-transistors:2N5457
- added R17, R21, R26, R35, R36: 10k, pedals-resistors:R_.3B
- added R18, R19, R20: 510k, pedals-resistors:R_.3B
- added R22: 470R, pedals-resistors:R_.3B
- added R23: 100k, pedals-resistors:R_.3B
- added R24, R25, R30, R33: 1M, pedals-resistors:R_.3B
- added R27, R28: 56k, pedals-resistors:R_.3B
- added R29: 22k, pedals-resistors:R_.3B
- added R31: 3.6k, pedals-resistors:R_.3B
- added R32: 22R, pedals-resistors:R_.3B
- added R34: 330k, pedals-resistors:R_.3B
- added SW1: MOMENTARY, pedals-switches:MOMENTARY
- added TR1, TR2, TR3, TR4, TR5, TR6: C1815BL, pedals-transistors:2SC828A
- added VR1: 500kA, pedals-potentiometers:POTS16MM
- added VR2, VR4: 250kA, pedals-potentiometers:POTS16MM
- added VR3: 50kA, pedals-potentiometers:POTS16MM
- added VR5: 100kB, pedals-potentiometers:POTS16MM
- added ZD1: (no value), pedals-diodes:ZENER.1
- C1: value 10u -> 20n; device pedals-capacitors-elec:0500 -> pedals-capacitors-film:CER/FILMBOX.1
- C10, C3: device pedals-capacitors-film:CER/FILMBOX.1 -> pedals-capacitors-elec:0500
- C11: value 4.7u -> 1n; device pedals-capacitors-elec:0500 -> pedals-capacitors-film:CER/FILMBOX.1
- C2: value 1u -> 10u
- C4: value 1u -> 51p
- C5: value 50p -> 220n
- C6: value 50n -> 68n
- C7: value 220n -> 33n; device pedals-capacitors-elec:0500 -> pedals-capacitors-film:CER/FILMBOX.1
- C8: value 220u -> 15n; device pedals-capacitors-elec:0500 -> pedals-capacitors-film:CER/FILMBOX.1
- C9: value 1u -> 330p
- D1: value 1N4001 -> MA165
- D2, D3: value SILICON -> MA165
- IC1: value MC1458P -> CA3260E
- JK1: value (none) -> INPUT
- R1, R16: value 10k -> 1k
- R11: value 1k -> 1M
- R12: value 220R -> 10k
- R13, R9: value 1k -> 47k
- R14: value 100k -> 1k
- R15: value 220R -> 510k
- R2: value 10k -> 510k
- R3: value 1k -> 9.1k
- R4: value 510k -> 22k
- R5: value 100k -> 10k
- R6: value 10k -> 220R
- R7: value 4.7k -> 1M
- R8: value 51k -> 2.7k
- renumbered INPUT to JK1
Connections:
- new net N$24: C13.-, VR5.2
- new net N$25: C13.+, Q1.D, R15.2
- new net N$26: C18.1, D6.C, R25.1
- new net N$27: C15.2, Q1.S, Q2.S, R19.2
- new net N$29: C19.2, C20.2, C21.1, R32.2, R33.1, R34.2
- new net N$30: C14.1, Q2.D, R18.2
- new net N$31: R24.1, R29.1, TR5.C
- new net N$32: C19.1, R27.2, TR4.B
- new net N$33: D6.A, Q2.G
- new net N$34: C20.1, R28.2, TR5.B
- new net N$36: 1101.P$1, JK3.R
- new net N$37: R30.2, TR6.B
- new net N$38: LED1.A, TR6.C, ZD1.A
- new net N$39: R25.2, R26.1, R30.1, TR4.C
- new net N$40: R31.1, ZD1.C
- new net N$41: D5.A, Q1.G
- new net N$42: C17.1, D5.C, R24.2
- new net N$43: R32.1, SW1.P
- new net N$44: C16.-, JK2.T, R23.2
- new net N$45: C16.+, R22.2
- new net N$46: R21.2, R22.1, TR3.E
- new net N$47: C15.1, R20.2, TR3.B
- new net N$54: C6.1, C8.1, VR3.1
- new net VB1: C9.1, VR2.3
- net +9V: now also C22.+, D7.C, JK3.S, R26.2, R29.2, R31.2, R33.2, R35.1, TR1.C, TR2.C, TR3.C; no longer AC_ADAPTOR.S, D1.C, IC2_PWR.V+, R1.1
- net GND: now also C17.2, C18.2, C2.-, C21.2, C22.-, C23.-, D7.A, JK2.R, JK2.S, JK3.T, LED1.C, R17.1, R21.1, R23.1, R27.1, R28.1, R34.1, R36.1, R4.1, R5.1, SW1.S, TR4.E, TR5.E, TR6.E; no longer AC_ADAPTOR.T, C1.-, C7.-, D1.A, IC2_PWR.V-, OUTPUT.SLEEVE, R16.1, R2.1
- net N$1: now also C1.2; no longer R3.1
- net N$10: now also IC1_B.+IN, R6.2; no longer C5.2, D2.C, D3.A, IC1_B.-IN, POT1.2, POT1.3
- net N$11: now also D1.A, D2.C; no longer POT1.1, R8.2
- net N$12: no longer D2.A, D3.C, IC1_B.OUT, R9.1
- net N$13: now also D3.C, D4.A; no longer C6.1, R7.1
- net N$14: now also C7.1, R10.1, VR2.1; no longer C8.+, POT2.2
- net N$15: now also R16.2, TR2.B; no longer C7.+, IC2_B.+IN, POT2.1, R10.2, R9.2
- net N$16: now also R10.2, VR4.1; no longer C8.-, R12.1
- net N$17: now also R14.2, VR5.3; no longer POT3.3, R13.2
- net N$18: now also C6.2, C7.2, R9.2; no longer C9.1, R13.1
- net N$19: now also IC1_A.+IN, R11.2, VR2.2; no longer C10.2, POT3.2
- net N$2: now also 1101.P$2; no longer BATTERY.P$2
- net N$20: now also C10.-, R12.1; no longer C10.1, IC2_A.+IN, R14.2
- net N$21: now also C11.2, IC1_A.-IN, R12.2, R13.1; no longer IC2_A.-IN, IC2_A.OUT, R15.1
- net N$22: now also C11.1, C12.+, IC1_A.OUT, R13.2; no longer C11.+, R15.2
- net N$23: now also C12.-, R14.1; no longer C11.-, OUTPUT.TIP, R16.2
- net N$28: now also C14.2, R17.2, TR2.E; no longer AC_ADAPTOR.R, BATTERY.P$1
- net N$3: now also C1.1, R1.1; no longer IC2_B.-IN, POT2.3, R11.1
- net N$4: now also R1.2, R2.2, TR1.B; no longer C9.2, IC2_B.OUT, R11.2
- net N$5: now also C2.+, R2.1, R3.1, R4.2; no longer C2.-, R3.2
- net N$6: now also C3.+, R16.1, R5.2, TR1.E; no longer C2.+, IC1_A.+IN, R4.2
- net N$7: now also D1.C, D3.A, IC1_B.-IN, R8.2, VR1.1; no longer C3.1, IC1_A.-IN, IC1_A.OUT
- net N$8: now also C4.1, C9.2, D2.A, D4.C, IC1_B.OUT, R9.1, VR1.2, VR1.3; no longer C3.2, R5.2
- net N$9: now also C3.-, R6.1; no longer C4.1, IC1_B.+IN, R6.2
- net VB: now also C10.+, C23.+, C5.2, C8.2, R11.1, R15.1, R18.1, R19.1, R20.1, R3.2, R35.2, R36.2, R7.1, VR3.2, VR3.3, VR4.2, VR4.3, VR5.1; no longer C1.+, C6.2, POT3.1, R1.2, R10.1, R12.2, R14.1, R2.2, R4.1, R5.1, R6.1
Other:
- note added: "01"
- note added: "02"
- note added: "03"
- note added: "04"
- note added: "1"
- note added: "2"
- note added: "3"
- note added: "4"
- note added: "6"
- note added: "7"
- note added: "8"
- note added: "CR1"
- note added: "CR2"
- moved on the sheet: C2, C4, C5, C6, C9, D1, D2, D3, IC1_A, IC1_B, IC1_PWR, R1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

Commit message: 20180125
Connections:
- net +9V: now also R3.2
- net VB: no longer R3.2
Other:
- note added: "BASS"
- note added: "DISTORTION"
- note added: "LEVEL"
- note added: "MIDDLE"
- note added: "TREBLE"
Changed lines of the file:
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@@
 <?xml version="1.0" encoding="utf-8"?>
 <!DOCTYPE eagle SYSTEM "eagle.dtd">
-<eagle version="8.2.0">
+<eagle version="8.5.1">
 <drawing>
 <settings>
 <setting alwaysvectorfont="no"/>
+<setting keepoldvectorfont="yes"/>
 <setting verticaltext="up"/>
 </settings>
-<grid distance="0.1" unitdist="inch" unit="inch" style="lines" multiple="1" display="yes" altdistance="0.01" altunitdist="inch" altunit="inch"/>
+<grid distance="0.1" unitdist="inch" unit="inch" style="lines" multiple="1" display="no" altdistance="0.01" altunitdist="inch" altunit="inch"/>
 <layers>
 <layer number="1" name="Top" color="4" fill="1" visible="no" active="no"/>
@@
 <part name="R2" library="pedals-resistors" deviceset="R_" device=".3B" value="510k"/>
 <part name="R3" library="pedals-resistors" deviceset="R_" device=".3B" value="9.1k"/>
-<part name="VB101" library="gm-supply" deviceset="VB" device=""/>
 <part name="R4" library="pedals-resistors" deviceset="R_" device=".3B" value="22k"/>
 <part name="C2" library="pedals-capacitors-elec" deviceset="050" device="0" value="10u"/>
@@
 <part name="V1" library="gm-supply" deviceset="+9V" device=""/>
 <part name="GND3" library="gm-supply" deviceset="GND" device=""/>
+<part name="V2" library="gm-supply" deviceset="+9V" device=""/>
 </parts>
 <sheets>
@@
 <circle x="187.96" y="-86.36" radius="0.381" width="0.1524" layer="95"/>
 <text x="188.214" y="-86.106" size="1.778" layer="95">04</text>
+<text x="93.98" y="134.62" size="1.778" layer="95">DISTORTION</text>
+<text x="132.08" y="134.62" size="1.778" layer="95">MIDDLE</text>
+<text x="167.64" y="134.62" size="1.778" layer="95">TREBLE</text>
+<text x="205.74" y="134.62" size="1.778" layer="95">BASS</text>
+<text x="238.76" y="134.62" size="1.778" layer="95">LEVEL</text>
 </plain>
 <instances>
@@
 <instance part="R2" gate="G$1" x="48.26" y="27.94" rot="R90"/>
 <instance part="R3" gate="G$1" x="38.1" y="27.94" rot="R90"/>
-<instance part="VB101" gate="G$1" x="38.1" y="38.1"/>
 <instance part="R4" gate="G$1" x="38.1" y="12.7" rot="R90"/>
 <instance part="C2" gate="1" x="48.26" y="15.24" rot="MR270"/>
@@
 <instance part="V1" gate="+9V" x="137.16" y="-40.64"/>
 <instance part="GND3" gate="GND" x="187.96" y="-78.74" rot="R180"/>
+<instance part="V2" gate="+9V" x="38.1" y="38.1"/>
 </instances>
 <busses>
@@
 <pinref part="VB103" gate="G$1" pin="VB"/>
 <wire x1="73.66" y1="-30.48" x2="73.66" y2="-27.94" width="0.1524" layer="91"/>
-</segment>
-<segment>
-<pinref part="VB101" gate="G$1" pin="VB"/>
-<pinref part="R3" gate="G$1" pin="2"/>
-<wire x1="38.1" y1="35.56" x2="38.1" y2="33.02" width="0.1524" layer="91"/>
 </segment>
 <segment>
@@
 <wire x1="137.16" y1="-45.72" x2="137.16" y2="-43.18" width="0.1524" layer="91"/>
 </segment>
+<segment>
+<pinref part="R3" gate="G$1" pin="2"/>
+<wire x1="38.1" y1="35.56" x2="38.1" y2="33.02" width="0.1524" layer="91"/>
+<pinref part="V2" gate="+9V" pin="+9V"/>
+</segment>
 </net>
