File: #Misc/Ibanez OD855/od855.sch (EAGLE design)
At the start: 73 parts, among them IC101 RC4558, Q101 2SC1815BL, Q102 1SK44SP, Q103 2SC1815BL, Q104 2SK44SP, Q105 2SC1815BL, Q106 2SC1815BL, Q107 2SC1815BL

Commit message: 20171230
Parts:
- removed C113: 1n, pedals-capacitors-film:CER/FILMBOX.1
- removed FOOTSW: MOMENTARY, pedals-switches:MOMENTARY
- added C118, C119: 1n, pedals-capacitors-film:CER/FILMBOX.1
- added C120: 47u, pedals-capacitors-elec:0500
- added C121: 100u, pedals-capacitors-elec:0500
- added R134: 10k, pedals-resistors:R_.3B
- added SW1: MOMENTARY, pedals-switches:MOMENTARY
- C103: value 47n -> 100n; device pedals-capacitors-film:CER/FILMBOX.1 -> pedals-capacitors-elec:0500
- C104: value 51p -> 470p
- C105: value 220n -> 1u; device pedals-capacitors-elec:0500 -> pedals-capacitors-film:CER/FILMBOX.1
- C106: value 220n -> 470n
- C107: value 1u -> 20p
- C108: value 100n -> 4.7u; device pedals-capacitors-film:CER/FILMBOX.1 -> pedals-capacitors-elec:0500
- C109: value 10u -> 2n; device pedals-capacitors-elec:0500 -> pedals-capacitors-film:CER/FILMBOX.1
- C110: value 47n -> 100n
- C112: value 47n -> 10u; device pedals-capacitors-film:CER/FILMBOX.1 -> pedals-capacitors-elec:0500
- C114: value 1n -> 47n
- C115: value 1n -> 100n
- C116: value 47u -> 47n; device pedals-capacitors-elec:0500 -> pedals-capacitors-film:CER/FILMBOX.1
- C117: value 100u -> 1n; device pedals-capacitors-elec:0500 -> pedals-capacitors-film:CER/FILMBOX.1
- D101, D102: value MA150 -> 1N60
- DISTORTION: value 500kA -> 50kC
- LEVEL: value 100kB -> 10kB
- R101, R111: value 1k -> 10k
- R103: value 10k -> 3k
- R104: value 4.7k -> 3k
- R105: value 10k -> 680R
- R106: value 51k -> 100k
- R107: value 1k -> 3k
- R108: value 220R -> 10k
- R109: value 10k -> 100k
- R110: value 1k -> 470R
- R113: value 10k -> 1M
- R114: value 100R -> 510k
- R116, R130: value 1M -> 100R
- R117: value 510k -> 10k
- R119: value 1M -> 510k
- R121: value 62k -> 1M
- R122: value 22k -> 62k
- R123: value 1M -> 22k
- R124: value 22R -> 1M
- R125: value 56k -> 22R
- R129: value 100R -> 56k
- R131: value 36k -> 1M
- R132: value 10k -> 36k
- renumbered BATTERY to 11, DC to DC1
Connections:
- new net N$43: DISTORTION.3, R110.2
- new net N$44: C106.-, R110.1
- net +9V: now also C121.+, R122.2, R128.2, R134.1; no longer C117.+, R121.2, R127.2, R133.1
- net GND: now also C109.2, C114.2, C116.2, C119.2, C120.-, C121.-, D101.A, D102.C, DISTORTION.2, R105.1, R117.1, R123.1, R127.1, R130.1, R133.1, SW1.S; no longer C105.-, C110.2, C112.2, C113.2, C116.-, C117.-, FOOTSW.S, R108.1, R113.1, R122.1, R125.1, R128.1, R132.1
- net N$10: now also C104.1, C105.2, IC101_A.OUT; no longer C105.+, IC101_B.+IN, R109.2, TONE.1
- net N$11: now also C106.+, C107.2, R109.1; no longer R110.1, TONE.3
- net N$12: now also C105.1, IC101_B.+IN, R108.2; no longer C107.2, IC101_B.OUT, R110.2
- net N$13: now also IC101_B.OUT, R109.2
- net N$14: now also C108.+, R111.2; no longer C106.+, TONE.2
- net N$15: now also C108.-, C109.1, D101.C, D102.A, LEVEL.3; no longer C106.-, R108.2
- net N$16: now also C110.2, LEVEL.2; no longer LEVEL.3, R111.2
- net N$17: now also C110.1, R112.2; no longer LEVEL.2
- net N$18: now also C111.2, R119.2; no longer C108.2, R117.2
- net N$20: now also C114.1, R113.2; no longer C110.1, R116.2
- net N$22: now also C116.1, R121.2; no longer C112.1, R119.2
- net N$23: now also C111.1, R114.2; no longer C108.1, R112.2
- net N$24: now also R115.2, R116.1; no longer R113.2, R114.1
- net N$25: now also C112.+, R116.2; no longer C109.+, R114.2
- net N$26: now also C112.-, R117.2; no longer C109.-, R115.2
- net N$27: now also C115.1; no longer C111.1
- net N$29: now also R113.1, R128.1, R131.2; no longer R116.1, R127.1, R130.2
- net N$30: now also R131.1; no longer R130.1
- net N$31: now also R121.1; no longer R119.1
- net N$32: now also C118.1, R129.2; no longer C115.1, R128.2
- net N$34: now also C117.1, R127.2; no longer C114.1, R125.2
- net N$36: now also C117.2, C118.2, C119.1, R124.1, R125.2; no longer C113.1, C114.2, C115.2, R123.1, R124.2
- net N$37: now also R130.2; no longer R129.2
- net N$38: now also R122.1, R124.2; no longer R121.1, R122.2
- net N$39: now also R125.1, SW1.P; no longer FOOTSW.P, R124.1
- net N$4: now also C115.2; no longer C111.2
- net N$40: now also R132.1; no longer R131.1
- net N$41: now also R132.2; no longer R131.2
- net N$5: now also R104.1; no longer IC101_A.+IN, R105.2
- net N$6: now also C103.+, TONE.2; no longer C103.1, C104.2, D101.C, D102.A, IC101_A.-IN, R106.1
- net N$7: now also IC101_A.+IN, R104.2, TONE.1; no longer DISTORTION.1
- net N$8: now also C103.-, R105.2; no longer C104.1, D101.A, D102.C, DISTORTION.2, IC101_A.OUT, R107.1
- net N$9: now also C104.2, IC101_A.-IN, R107.1, TONE.3; no longer C103.2, R104.2
- net VB: now also C120.+, R106.1, R108.1, R114.1, R119.1, R134.2; no longer C116.+, R104.1, R105.1, R109.1, R117.1, R132.2
Other:
- note removed: "15"
- note removed: "6"
- moved on the sheet: C102, C104, C106, C107, C110, C111, C114, C115, D101, D102, D103, D104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

Commit message: 20180125
Other:
- moved on the sheet: C115, C116, C117, C118, C119, C120, C121, D104, D106, D107, D108, DC1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
