File: #Misc/Ibanez TS5/ts5.sch (EAGLE design)
At the start: 73 parts, among them IC101 RC4558, Q101 2SC1815BL, Q102 1SK44SP, Q103 2SC1815BL, Q104 2SK44SP, Q105 2SC1815BL, Q106 2SC1815BL, Q107 2SC1815BL

Commit message: 20171230
Parts:
- removed BATTERY: BATTERY, pedals-jacks:BATTERY
- removed C107: 1u, pedals-capacitors-film:CER/FILMBOX.1
- removed C108, C111: 100n, pedals-capacitors-film:CER/FILMBOX.1
- removed C109: 10u, pedals-capacitors-elec:0500
- removed C110, C112: 47n, pedals-capacitors-film:CER/FILMBOX.1
- removed C113, C114, C115: 1n, pedals-capacitors-film:CER/FILMBOX.1
- removed C116: 47u, pedals-capacitors-elec:0500
- removed C117: 100u, pedals-capacitors-elec:0500
- removed D103, D104, D106: MA150, pedals-diodes:DO35.2
- removed D107: RD4.7EB, pedals-diodes:ZENER.2
- removed D108: W03C, pedals-diodes:DO35.2
- removed DC: DCJACK, pedals-jacks:DC_KOBICONN
- removed DISTORTION: 500kA, pedals-potentiometers:POTS16MM
- removed FOOTSW: MOMENTARY, pedals-switches:MOMENTARY
- removed LED: LED, pedals-diodes:LED
- removed LEVEL: 100kB, pedals-potentiometers:POTS16MM
- removed OUTPUT: (no value), pedals-jacks:MONO
- removed Q102: 1SK44SP, pedals-transistors:2N5457
- removed Q103: 2SC1815BL, pedals-transistors:2N3904
- removed Q104: 2SK44SP, pedals-transistors:2N5457
- removed Q105, Q106, Q107: 2SC1815BL, pedals-transistors:2SC828A
- removed R109, R113, R115, R132, R133: 10k, pedals-resistors:R_.3B
- removed R111: 1k, pedals-resistors:R_.3B
- removed R112, R117, R118: 510k, pedals-resistors:R_.3B
- removed R114, R129: 100R, pedals-resistors:R_.3B
- removed R116, R119, R130: 1M, pedals-resistors:R_.3B
- removed R121: 62k, pedals-resistors:R_.3B
- removed R122: 22k, pedals-resistors:R_.3B
- removed R124: 22R, pedals-resistors:R_.3B
- removed R125, R126, R127, R128: 56k, pedals-resistors:R_.3B
- removed R131: 36k, pedals-resistors:R_.3B
- removed TONE: 20kG, pedals-potentiometers:POTS16MM
- added 1101: BATTERY, pedals-jacks:BATTERY
- added C1: 100u, pedals-capacitors-elec:0500
- added C13: 1u, pedals-capacitors-film:CER/FILMBOX.1
- added C15, C18: 100n, pedals-capacitors-film:CER/FILMBOX.1
- added C16, C17: 47n, pedals-capacitors-film:CER/FILMBOX.1
- added C19: 10u, pedals-capacitors-elec:0500
- added C2: 47u, pedals-capacitors-elec:0500
- added C3, C4, C5: 1n, pedals-capacitors-film:CER/FILMBOX.1
- added D1: 1N4148, pedals-diodes:DO35.2
- added D4, D5: 1N4002, pedals-diodes:DO35.2
- added JK1: DCJACK, pedals-jacks:DC_KOBICONN
- added JK3: (no value), pedals-jacks:STEREO
- added LED1: TLR124, pedals-diodes:LED
- added Q1, Q2: K1180, pedals-transistors:2N5457
- added R1, R2, R21, R33, R9: 10k, pedals-resistors:R_.3B
- added R10: 3.3k, pedals-resistors:R_.3B
- added R24: 1k, pedals-resistors:R_.3B
- added R27, R28, R32: 510k, pedals-resistors:R_.3B
- added R3: 22R, pedals-resistors:R_.3B
- added R30, R31, R4: 1M, pedals-resistors:R_.3B
- added R34: 470R, pedals-resistors:R_.3B
- added R35: 100k, pedals-resistors:R_.3B
- added R5: 330k, pedals-resistors:R_.3B
- added R6, R7: 56k, pedals-resistors:R_.3B
- added SW1: MOMENTARY, pedals-switches:MOMENTARY
- added TR1, TR2: C1815BL, pedals-transistors:2SC828A
- added TR5: C1815BL, pedals-transistors:2N3904
- added VR1: 500kA, pedals-potentiometers:POTS16MM
- added VR2: 20kG, pedals-potentiometers:POTS16MM
- added VR3: 100kB, pedals-potentiometers:POTS16MM
- added ZD1: HZ5B1, pedals-diodes:ZENER.2
- C9: value 51p -> 47p
- D2, D3: value MA150 -> 1N4002
- IC1: value RC4558 -> NJM4558D
- JK2: value (none) -> INPUT
- R8: value 1M -> 22k
- TR3: value 2SC1815BL -> C1815BL
- renumbered C101 to C6, C102 to C8, C103 to C10, C104 to C9, C105 to C11, C106 to C12, D101 to D2, D102 to D3, IC101 to IC1, INPUT to JK2, Q101 to TR3, R101 to R11, R102 to R12, R103 to R15, R104 to R18, R105 to R17, R106 to R19, R107 to R20, R108 to R22, R110 to R23, R123 to R8
Connections:
- removed net N$28: BATTERY.P$1, DC.R
- removed net N$39: FOOTSW.P, R124.1
- removed net N$40: LED.C, R131.1
- removed net N$41: D107.C, R131.2
- removed net N$42: D107.A, Q107.C
- net +9V: now also C1.+, D1.C, JK1.S, LED1.A, R1.1, R4.2, R8.2, R9.2, TR5.C; no longer C117.+, D108.C, DC.S, LED.A, Q103.C, R121.2, R126.2, R127.2, R133.1
- net GND: now also C1.-, C16.2, C17.2, C2.-, C3.2, D1.A, JK1.T, JK3.T, R2.1, R33.1, R35.1, R5.1, R6.1, R7.1, SW1.S, TR1.E, TR2.E; no longer C110.2, C112.2, C113.2, C116.-, C117.-, D108.A, DC.T, FOOTSW.S, LEVEL.1, OUTPUT.SLEEVE, R113.1, R115.1, R122.1, R125.1, R128.1, R129.1, R132.1
- net N$10: now also R21.2, VR2.1; no longer R109.2, TONE.1
- net N$11: now also VR2.3; no longer TONE.3
- net N$12: now also C13.2; no longer C107.2
- net N$13: now also C19.-, R34.1, R35.2; no longer C107.1, R111.1
- net N$14: now also VR2.2; no longer TONE.2
- net N$16: now also R24.2, VR3.3; no longer LEVEL.3, R111.2
- net N$17: now also Q2.D, VR3.2; no longer LEVEL.2, Q102.D
- net N$18: now also C15.1, Q1.D, R27.2; no longer C108.2, Q102.S, Q104.S, R117.2
- net N$19: now also C18.2, Q1.S, Q2.S, R28.2; no longer D103.A, Q102.G
- net N$2: now also 1101.P$2; no longer BATTERY.P$2
- net N$20: now also D5.A, Q2.G; no longer C110.1, D103.C, R116.2
- net N$21: now also C17.1, D5.C, R31.2; no longer D104.A, Q104.G
- net N$22: now also C13.1, R24.1; no longer C112.1, D104.C, R119.2
- net N$23: now also C18.1, R32.2, TR5.B; no longer C108.1, Q103.B, R112.2
- net N$24: now also C19.+, R33.2, TR5.E; no longer Q103.E, R113.2, R114.1
- net N$25: now also JK3.S, R34.2; no longer C109.+, R114.2
- net N$26: now also C3.1, C4.2, C5.2, R3.1, R4.1, R5.2; no longer C109.-, OUTPUT.TIP, R115.2
- net N$27: now also D4.A, Q1.G; no longer C111.1, Q104.D, R118.2
- net N$29: now also R10.1, R30.1, R9.1, TR2.C; no longer Q106.C, R116.1, R127.1, R130.2
- net N$30: now also C16.1, D4.C, R30.2; no longer Q107.B, R130.1
- net N$31: now also R31.1, R8.1, TR1.C; no longer Q105.C, R119.1, R126.1
- net N$32: now also C5.1, R7.2, TR2.B; no longer C115.1, Q106.B, R128.2
- net N$34: now also C4.1, R6.2, TR1.B; no longer C114.1, Q105.B, R125.2
- net N$35: now also R3.2, SW1.P; no longer D106.A, Q105.E, Q106.E, Q107.E
- net N$36: now also 1101.P$1, JK1.R; no longer C113.1, C114.2, C115.2, R124.2, R8.1
- net N$37: now also R10.2, ZD1.A; no longer D106.C, R129.2
- net N$38: now also LED1.C, ZD1.C; no longer R121.1, R122.2, R8.2
- net N$4: now also C15.2; no longer C111.2
- net N$7: now also VR1.1; no longer DISTORTION.1
- net N$8: now also VR1.2, VR1.3; no longer DISTORTION.2
- net VB: now also C2.+, R1.2, R2.2, R21.1, R27.1, R28.1, R32.1, VR3.1; no longer C116.+, R109.1, R112.1, R117.1, R118.1, R132.2, R133.2
Other:
- note removed: "1"
- note removed: "10"
- note removed: "11"
- note removed: "12"
- note removed: "13"
- note removed: "15"
- note removed: "2"
- note removed: "3"
- note removed: "4"
- note removed: "5"
- note removed: "6"
- note removed: "7"
- note removed: "8"
- note removed: "9"

Commit message: 20180125
Other:
- note added: "DIST."
- note added: "LEVEL"
- note added: "TONE"
- moved on the sheet: R21
Changed lines of the file:
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@@
 <?xml version="1.0" encoding="utf-8"?>
 <!DOCTYPE eagle SYSTEM "eagle.dtd">
-<eagle version="8.2.0">
+<eagle version="8.5.1">
 <drawing>
 <settings>
 <setting alwaysvectorfont="no"/>
+<setting keepoldvectorfont="yes"/>
 <setting verticaltext="up"/>
 </settings>
@@
 <text x="172.212" y="-57.658" size="1.778" layer="95" rot="MR0">CR1</text>
 <text x="197.612" y="-57.658" size="1.778" layer="95" rot="MR0">CR2</text>
+<text x="91.44" y="106.68" size="1.778" layer="95">DIST.</text>
+<text x="127" y="106.68" size="1.778" layer="95">TONE</text>
+<text x="179.578" y="106.68" size="1.778" layer="95">LEVEL</text>
 </plain>
 <instances>
@@
 <instance part="C11" gate="1" x="119.38" y="38.1" rot="MR270"/>
 <instance part="GND108" gate="GND" x="119.38" y="25.4"/>
-<instance part="R21" gate="G$1" x="137.16" y="35.56" rot="R90"/>
-<instance part="VB106" gate="G$1" x="137.16" y="25.4" rot="R180"/>
+<instance part="R21" gate="G$1" x="134.62" y="35.56" rot="R90"/>
+<instance part="VB106" gate="G$1" x="134.62" y="25.4" rot="R180"/>
 <instance part="VR2" gate="G$1" x="129.54" y="99.06" rot="R270"/>
 <instance part="V104" gate="+9V" x="149.86" y="55.88"/>
@@
 <pinref part="VB106" gate="G$1" pin="VB"/>
 <pinref part="R21" gate="G$1" pin="1"/>
-<wire x1="137.16" y1="27.94" x2="137.16" y2="30.48" width="0.1524" layer="91"/>
+<wire x1="134.62" y1="27.94" x2="134.62" y2="30.48" width="0.1524" layer="91"/>
 </segment>
 <segment>
@@
 <wire x1="119.38" y1="40.64" x2="119.38" y2="43.18" width="0.1524" layer="91"/>
 <pinref part="R21" gate="G$1" pin="2"/>
-<wire x1="137.16" y1="40.64" x2="137.16" y2="43.18" width="0.1524" layer="91"/>
+<wire x1="134.62" y1="40.64" x2="134.62" y2="43.18" width="0.1524" layer="91"/>
 <pinref part="IC1" gate="_B" pin="+IN"/>
-<wire x1="137.16" y1="43.18" x2="142.24" y2="43.18" width="0.1524" layer="91"/>
-<wire x1="119.38" y1="43.18" x2="137.16" y2="43.18" width="0.1524" layer="91"/>
+<wire x1="134.62" y1="43.18" x2="142.24" y2="43.18" width="0.1524" layer="91"/>
+<wire x1="119.38" y1="43.18" x2="134.62" y2="43.18" width="0.1524" layer="91"/>
 <junction x="119.38" y="43.18"/>
-<junction x="137.16" y="43.18"/>
-</segment>
-</net>
+<junction x="134.62" y="43.18"/>
+</segment>
+</net>
