File: #Misc/MXR Distortion III/distortion3_redraw.sch (EAGLE design)
At the start: 43 parts, among them IC1 MC33178P, Q1 MPS-A14, Q4 2N3820

Commit message: 20180125
Parts:
- removed BAT1: BATTERY, pedals-jacks:BATTERY
- removed C11: (no value), pedals-capacitors-film:CER/FILMBOX.1
- removed DCJACK: (no value), pedals-jacks:DC_KOBICONN
- removed IN: (no value), pedals-jacks:STEREO
- removed OUT: (no value), pedals-jacks:MONO_JACK
- removed Q4: 2N3820, transistor-small-signal:2N3820
- removed R19: 2.2M, pedals-resistors:R_.3B
- removed S1: (no value), pedals-switches:DPDT
Connections:
- removed net N$1: BAT1.P$2, IN.R
- removed net N$2: BAT1.P$1, DCJACK.R
- removed net N$23: OUT.TIP, S1_A.3, S1_B.1
- removed net N$24: S1_B.2, VR1.2
- removed net N$3: IN.T, S1_A.2
- removed net N$9: C11.1, Q4.G, R19.1, S1_B.3
- new net OUT: VR1.2
- net GND: no longer C11.2, DCJACK.T, IN.S, OUT.SLEEVE, Q4.D
- net N$7: no longer Q4.S
- net N$8: no longer S1_A.1
- net VR: no longer DCJACK.S, R19.2
Other:
- note added: "DISTORTION"
- note added: "OUTPUT"
- note added: "TONE"
- moved on the sheet: C7, C8, C9, D3, R10, R13, R8, R9
