File: #Misc/Proco Rat/rat.sch (EAGLE design)
At the start: 45 parts, among them IC1 LM308N, Q1 2N5458, Q2 2N5458

Commit message: 20180125
Parts:
- R1, R6: value 47 -> 47R
- R7: value 560 -> 560R
Other:
- note added: "FILTER"
- note added: "GAIN"
- note added: "LEVEL"
Changed lines of the file:
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@@
 <?xml version="1.0" encoding="utf-8"?>
 <!DOCTYPE eagle SYSTEM "eagle.dtd">
-<eagle version="8.2.0">
+<eagle version="8.5.1">
 <drawing>
 <settings>
 <setting alwaysvectorfont="no"/>
+<setting keepoldvectorfont="yes"/>
 <setting verticaltext="up"/>
 </settings>
-<grid distance="0.1" unitdist="inch" unit="inch" style="lines" multiple="1" display="yes" altdistance="0.01" altunitdist="inch" altunit="inch"/>
+<grid distance="0.1" unitdist="inch" unit="inch" style="lines" multiple="1" display="no" altdistance="0.01" altunitdist="inch" altunit="inch"/>
 <layers>
 <layer number="1" name="Top" color="4" fill="1" visible="no" active="no"/>
@@
 <part name="C8" library="pedals-capacitors-film" deviceset="CER/FILM" device="2" value="30p"/>
 <part name="C7" library="pedals-capacitors-film" deviceset="CER/FILM" device="2" value="100p"/>
-<part name="R6" library="pedals-resistors" deviceset="R_" device=".3B" value="47"/>
-<part name="R7" library="pedals-resistors" deviceset="R_" device=".3B" value="560"/>
+<part name="R6" library="pedals-resistors" deviceset="R_" device=".3B" value="47R"/>
+<part name="R7" library="pedals-resistors" deviceset="R_" device=".3B" value="560R"/>
 <part name="C7_" library="pedals-capacitors-elec" deviceset="050" device="0" value="4.7u"/>
 <part name="C6" library="pedals-capacitors-elec" deviceset="050" device="0" value="2.2u"/>
@@
 <part name="GND104" library="gm-supply" deviceset="GND" device=""/>
 <part name="GND102" library="gm-supply" deviceset="GND" device=""/>
-<part name="R1" library="pedals-resistors" deviceset="R_" device=".3B" value="47"/>
+<part name="R1" library="pedals-resistors" deviceset="R_" device=".3B" value="47R"/>
 <part name="D1" library="pedals-diodes" deviceset="DO35" device=".2" value="1N4001"/>
 <part name="R2" library="pedals-resistors" deviceset="R_" device=".3B" value="100k"/>
@@
 <sheet>
 <plain>
+<text x="80.772" y="45.72" size="1.778" layer="95">GAIN</text>
+<text x="133.35" y="81.026" size="1.778" layer="95">FILTER</text>
+<text x="203.708" y="86.106" size="1.778" layer="95">LEVEL</text>
 </plain>
 <instances>
