File: #Misc/Seymour Duncan TweakFuzz/tweakfuzz.sch (EAGLE design)
At the start: 34 parts, among them P1 500kA, P2 1kB, Q1 MMBT3904, Q2 MMBT4401, SW1 1P6T, SW2 3PDT

Commit message: 20180125
Other:
- note added: "GAIN"
- note added: "TWEAK"
- note added: "VOLUME"
Changed lines of the file:
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@@
 <?xml version="1.0" encoding="utf-8"?>
 <!DOCTYPE eagle SYSTEM "eagle.dtd">
-<eagle version="8.2.0">
+<eagle version="8.5.1">
 <drawing>
 <settings>
 <setting alwaysvectorfont="no"/>
+<setting keepoldvectorfont="yes"/>
 <setting verticaltext="up"/>
 </settings>
-<grid distance="0.1" unitdist="inch" unit="inch" style="lines" multiple="1" display="yes" altdistance="0.01" altunitdist="inch" altunit="inch"/>
+<grid distance="0.1" unitdist="inch" unit="inch" style="lines" multiple="1" display="no" altdistance="0.01" altunitdist="inch" altunit="inch"/>
 <layers>
 <layer number="1" name="Top" color="4" fill="1" visible="no" active="no"/>
@@
 <text x="174.498" y="131.826" size="1.778" layer="95" rot="R90">blk</text>
 <text x="200.406" y="105.41" size="1.778" layer="95">gry</text>
+<text x="147.32" y="78.74" size="1.778" layer="95">GAIN</text>
+<text x="167.64" y="111.76" size="1.778" layer="95">VOLUME</text>
+<text x="55.88" y="104.14" size="1.778" layer="95">TWEAK</text>
 </plain>
 <instances>
