File: #Misc/Boss BF-2/bf2.sch (EAGLE design)
At the start: 143 parts, among them IC1 uPC4558C, IC2 uPC4558, IC3 MN3207, IC4 MN3102, IC5 TL022CP, IC6 LM78L05, Q1 2SC732TM-GR, Q10 2SC945-P, Q11 2SC945-P, Q2 2SC732TM-GR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

Commit message: 20180125
Parts:
- Q1, Q2, Q3: value 2SC732TM-GR -> 2SC732TM
- R64: value 470R -> 56R
- VR6: value (none) -> 22kB
- renumbered C116 to C7, R120 to R39, R126 to R10
Other:
- moved on the sheet: VR2

Commit message: 20180207
Parts:
- Q8: value 2N3906- -> 2SC945-P; device pedals-transistors:2N3906- -> pedals-transistors:2SC828A
Connections:
- net +9V: no longer IC5_PWR.V+
- net GND: now also Q8.E; no longer Q8.C
- net VA: now also IC5_PWR.V+, Q8.C; no longer Q8.E
Other:
- note added: "BIAS"
- note added: "CL"
- note added: "DEPTH"
- note added: "MANUAL"
- note added: "RATE"
- note added: "RES"
- moved on the sheet: AC_ADAPTOR, C25, C26, C27, C28, C29, C30, C31, C32, C33, C34, C35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
