File: #Misc/Boss BF-2/bf2_redraw.sch (EAGLE design)
At the start: 137 parts, among them IC1 uPC4558C, IC2 uPC4558, IC3 MN3207, IC4 MN3102, IC5 TL022CP, IC6 LM78L05, Q1 2SC732TM-GR, Q10 2SC945-P, Q11 2SC945-P, Q2 2SC732TM-GR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

Commit message: 20180125
Parts:
- Q1, Q2, Q3: value 2SC732TM-GR -> 2SC732TM
- R120: value 1.5k -> R39
- VR6: value (none) -> 22kB
- renumbered C116 to C7, R126 to R10
Changed lines of the file:
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@@
 <?xml version="1.0" encoding="utf-8"?>
 <!DOCTYPE eagle SYSTEM "eagle.dtd">
-<eagle version="8.2.0">
+<eagle version="8.5.1">
 <drawing>
 <settings>
 <setting alwaysvectorfont="no"/>
+<setting keepoldvectorfont="yes"/>
 <setting verticaltext="up"/>
 </settings>
@@
 <part name="R1" library="pedals-resistors" deviceset="R_" device=".3B" value="1k"/>
 <part name="C1" library="pedals-capacitors-film" deviceset="CER/FILM" device="BOX.1" value="47n"/>
-<part name="Q1" library="pedals-transistors" deviceset="2SC828A" device="" value="2SC732TM-GR"/>
+<part name="Q1" library="pedals-transistors" deviceset="2SC828A" device="" value="2SC732TM"/>
 <part name="R2" library="pedals-resistors" deviceset="R_" device=".3B" value="470k"/>
 <part name="C25" library="pedals-capacitors-elec" deviceset="040" device="0" value="33u"/>
@@
 <part name="C9" library="pedals-capacitors-film" deviceset="CER/FILM" device="BOX.1" value="150p"/>
 <part name="GND115" library="gm-supply" deviceset="GND" device=""/>
-<part name="Q2" library="pedals-transistors" deviceset="2SC828A" device="" value="2SC732TM-GR"/>
+<part name="Q2" library="pedals-transistors" deviceset="2SC828A" device="" value="2SC732TM"/>
 <part name="V105" library="gm-supply" deviceset="+9V" device=""/>
 <part name="R16" library="pedals-resistors" deviceset="R_" device=".3B" value="10k"/>
@@
 <part name="IC4" library="pedals-integrated circuits" deviceset="CLOCK" device="" value="MN3102"/>
 <part name="IC3" library="pedals-integrated circuits" deviceset="BL3208" device="" value="MN3207"/>
-<part name="VR6" library="pedals-potentiometers" deviceset="POTS" device="16MM"/>
+<part name="VR6" library="pedals-potentiometers" deviceset="POTS" device="16MM" value="22kB"/>
 <part name="GND118" library="gm-supply" deviceset="GND" device=""/>
 <part name="IC6" library="pedals-regulators" deviceset="LM78L05" device=""/>
@@
 <part name="C16" library="pedals-capacitors-film" deviceset="CER/FILM" device="BOX.1" value="330p"/>
 <part name="R22" library="pedals-resistors" deviceset="R_" device=".3B" value="10k"/>
-<part name="Q3" library="pedals-transistors" deviceset="2SC828A" device="" value="2SC732TM-GR"/>
+<part name="Q3" library="pedals-transistors" deviceset="2SC828A" device="" value="2SC732TM"/>
 <part name="GND127" library="gm-supply" deviceset="GND" device=""/>
 <part name="GND128" library="gm-supply" deviceset="GND" device=""/>
@@
 <part name="D5" library="pedals-diodes" deviceset="DO35" device=".2" value="1S2473"/>
 <part name="VR4" library="pedals-potentiometers" deviceset="POTS" device="16MM" value="50kC"/>
-<part name="R126" library="pedals-resistors" deviceset="R_" device=".3B" value="39k"/>
+<part name="R10" library="pedals-resistors" deviceset="R_" device=".3B" value="39k"/>
 <part name="VR5" library="pedals-potentiometers" deviceset="POTS" device="16MM" value="22kB"/>
 <part name="GND136" library="gm-supply" deviceset="GND" device=""/>
-<part name="C116" library="pedals-capacitors-film" deviceset="CER/FILM" device="BOX.1" value="47n"/>
+<part name="C7" library="pedals-capacitors-film" deviceset="CER/FILM" device="BOX.1" value="47n"/>
 <part name="C30" library="pedals-capacitors-film" deviceset="CER/FILM" device="BOX.1" value="47p"/>
 <part name="R49" library="pedals-resistors" deviceset="R_" device=".3B" value="33k"/>
@@
 <part name="GND109" library="gm-supply" deviceset="GND" device=""/>
 <part name="GND110" library="gm-supply" deviceset="GND" device=""/>
-<part name="R120" library="pedals-resistors" deviceset="R_" device=".3B" value="1.5k"/>
+<part name="R120" library="pedals-resistors" deviceset="R_" device=".3B" value="R39"/>
 <part name="C27" library="pedals-capacitors-elec" deviceset="040" device="0" value="6.3u"/>
 <part name="C28" library="pedals-capacitors-elec" deviceset="040" device="0" value="6.3u"/>
@@
 <instance part="R32" gate="G$1" x="500.38" y="40.64"/>
 <instance part="C24" gate="1" x="510.54" y="40.64" rot="MR180"/>
-<instance part="R33" gate="G$1" x="518.16" y="33.02" rot="R270"/>
+<instance part="R33" gate="G$1" x="518.16" y="33.02" rot="MR270"/>
 <instance part="GND141" gate="GND" x="518.16" y="22.86"/>
 <instance part="V109" gate="+9V" x="414.02" y="53.34"/>
@@
 <instance part="D5" gate="G$1" x="447.04" y="27.94" rot="MR270"/>
 <instance part="VR4" gate="G$1" x="439.42" y="78.74" rot="MR0"/>
-<instance part="R126" gate="G$1" x="190.5" y="78.74"/>
+<instance part="R10" gate="G$1" x="190.5" y="78.74"/>
 <instance part="VR5" gate="G$1" x="205.74" y="78.74" rot="R90"/>
 <instance part="GND136" gate="GND" x="439.42" y="66.04"/>
-<instance part="C116" gate="G$1" x="219.71" y="78.74"/>
+<instance part="C7" gate="G$1" x="219.71" y="78.74"/>
 <instance part="C30" gate="G$1" x="247.65" y="-10.16"/>
 <instance part="R49" gate="G$1" x="236.22" y="-38.1"/>
@@
 <junction x="147.32" y="50.8"/>
 <wire x1="147.32" y1="60.96" x2="147.32" y2="78.74" width="0.1524" layer="91"/>
-<pinref part="R126" gate="G$1" pin="1"/>
+<pinref part="R10" gate="G$1" pin="1"/>
 <wire x1="147.32" y1="78.74" x2="185.42" y2="78.74" width="0.1524" layer="91"/>
 <junction x="147.32" y="60.96"/>
@@
 <wire x1="213.36" y1="30.48" x2="213.36" y2="27.94" width="0.1524" layer="91"/>
 <junction x="213.36" y="30.48"/>
-<wire x1="213.36" y1="30.48" x2="228.6" y2="30.48" width="0.1524" layer="91"/>
-<wire x1="228.6" y1="30.48" x2="228.6" y2="53.34" width="0.1524" layer="91"/>
+<wire x1="213.36" y1="30.48" x2="226.06" y2="30.48" width="0.1524" layer="91"/>
+<wire x1="226.06" y1="30.48" x2="226.06" y2="53.34" width="0.1524" layer="91"/>
 <pinref part="C10" gate="G$1" pin="2"/>
-<wire x1="228.6" y1="53.34" x2="231.14" y2="53.34" width="0.1524" layer="91"/>
+<wire x1="226.06" y1="53.34" x2="231.14" y2="53.34" width="0.1524" layer="91"/>
 </segment>
 </net>
@@
 <wire x1="205.74" y1="86.36" x2="198.12" y2="86.36" width="0.1524" layer="91"/>
 <wire x1="198.12" y1="86.36" x2="198.12" y2="78.74" width="0.1524" layer="91"/>
-<pinref part="R126" gate="G$1" pin="2"/>
+<pinref part="R10" gate="G$1" pin="2"/>
 <wire x1="195.58" y1="78.74" x2="198.12" y2="78.74" width="0.1524" layer="91"/>
 <pinref part="VR5" gate="G$1" pin="3"/>
@@
 <net name="N$59" class="0">
 <segment>
-<pinref part="C116" gate="G$1" pin="2"/>
+<pinref part="C7" gate="G$1" pin="2"/>
 <pinref part="VR5" gate="G$1" pin="1"/>
 <wire x1="215.9" y1="78.74" x2="212.09" y2="78.74" width="0.1524" layer="91"/>
@@
 <segment>
 <pinref part="VR4" gate="G$1" pin="2"/>
-<pinref part="C116" gate="G$1" pin="1"/>
+<pinref part="C7" gate="G$1" pin="1"/>
 <wire x1="434.34" y1="78.74" x2="223.52" y2="78.74" width="0.1524" layer="91"/>
 </segment>

Commit message: 20180207
Parts:
- Q8: value 2N3906- -> 2SC945-P; device pedals-transistors:2N3906- -> pedals-transistors:2SC828A
Connections:
- net +9V: no longer IC5_PWR.V+
- net GND: now also Q8.E; no longer Q8.C
- net VA: now also IC5_PWR.V+, Q8.C; no longer Q8.E
Other:
- note added: "BIAS"
- note added: "CL"
- note added: "DEPTH"
- note added: "MANUAL"
- note added: "RATE"
- note added: "RES"
- moved on the sheet: R42, R43, R44, VR1, VR2
Changed lines of the file:
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@@
 <part name="VA106" library="gm-supply" deviceset="VA" device=""/>
 <part name="IC5" library="pedals-integrated circuits" deviceset="DUAL" device="TH" value="TL022CP"/>
-<part name="V104" library="gm-supply" deviceset="+9V" device=""/>
 <part name="GND111" library="gm-supply" deviceset="GND" device=""/>
 <part name="C26" library="pedals-capacitors-film" deviceset="CER/FILM" device="BOX.1" value="10n"/>
@@
 <part name="R36" library="pedals-resistors" deviceset="R_" device=".3B" value="180k"/>
 <part name="VR2" library="pedals-potentiometers" deviceset="POTS" device="16MM" value="50kB"/>
-<part name="Q8" library="pedals-transistors" deviceset="2N3906" device="-"/>
 <part name="R43" library="pedals-resistors" deviceset="R_" device=".3B" value="150k"/>
 <part name="VA104" library="gm-supply" deviceset="VA" device=""/>
@@
 <part name="IN" library="gm-supply" deviceset="IN" device=""/>
 <part name="OUT" library="gm-supply" deviceset="OUT" device=""/>
+<part name="Q8" library="pedals-transistors" deviceset="2SC828A" device="" value="2SC945-P"/>
+<part name="VA1" library="gm-supply" deviceset="VA" device=""/>
 </parts>
 <sheets>
@@
 <circle x="157.48" y="-27.94" radius="0.381" width="0.1524" layer="95"/>
 <text x="156.972" y="-27.432" size="1.778" layer="95">13</text>
+<text x="203.2" y="71.12" size="1.778" layer="95">RES</text>
+<text x="447.04" y="76.2" size="1.778" layer="95" rot="R90">RES</text>
+<text x="231.14" y="22.098" size="1.778" layer="95" rot="R90">BIAS</text>
+<text x="212.344" y="-42.672" size="1.778" layer="95" rot="R90">CL</text>
+<text x="189.484" y="-49.53" size="1.778" layer="95" rot="R90">DEPTH</text>
+<text x="146.812" y="-35.56" size="1.778" layer="95">RATE</text>
+<text x="143.764" y="-75.692" size="1.778" layer="95" rot="R90">MANUAL</text>
 </plain>
 <instances>
@@
 <instance part="GND118" gate="GND" x="233.68" y="15.24"/>
 <instance part="IC6" gate="G$1" x="71.12" y="-27.94"/>
-<instance part="D9" gate="G$1" x="71.12" y="-43.18" rot="R270"/>
+<instance part="D9" gate="G$1" x="71.12" y="-43.18" rot="MR270"/>
 <instance part="GND105" gate="GND" x="71.12" y="-60.96"/>
 <instance part="C40" gate="1" x="83.82" y="-35.56" rot="MR270"/>
@@
 <instance part="IC5" gate="_B" x="129.54" y="-27.94" rot="MR180"/>
 <instance part="IC5" gate="_PWR" x="129.54" y="-27.94"/>
-<instance part="V104" gate="+9V" x="129.54" y="-17.78"/>
 <instance part="GND111" gate="GND" x="129.54" y="-38.1"/>
 <instance part="C26" gate="G$1" x="128.27" y="-7.62"/>
@@
 <instance part="C28" gate="1" x="190.5" y="-17.78" rot="MR0"/>
 <instance part="R36" gate="G$1" x="149.86" y="-2.54"/>
-<instance part="VR2" gate="G$1" x="195.58" y="-43.18"/>
-<instance part="Q8" gate="G$1" x="185.42" y="-71.12"/>
-<instance part="R43" gate="G$1" x="177.8" y="-63.5" rot="R90"/>
-<instance part="VA104" gate="G$1" x="177.8" y="-53.34"/>
-<instance part="R44" gate="G$1" x="177.8" y="-78.74" rot="R90"/>
-<instance part="GND113" gate="GND" x="177.8" y="-88.9"/>
-<instance part="GND114" gate="GND" x="187.96" y="-88.9"/>
-<instance part="R42" gate="G$1" x="170.18" y="-71.12"/>
-<instance part="VA105" gate="G$1" x="187.96" y="-53.34"/>
-<instance part="VR1" gate="G$1" x="152.4" y="-71.12"/>
-<instance part="VA103" gate="G$1" x="152.4" y="-58.42"/>
-<instance part="GND112" gate="GND" x="152.4" y="-88.9"/>
+<instance part="VR2" gate="G$1" x="195.58" y="-45.72"/>
+<instance part="R43" gate="G$1" x="175.26" y="-63.5" rot="R90"/>
+<instance part="VA104" gate="G$1" x="175.26" y="-53.34"/>
+<instance part="R44" gate="G$1" x="175.26" y="-78.74" rot="R90"/>
+<instance part="GND113" gate="GND" x="175.26" y="-88.9"/>
+<instance part="GND114" gate="GND" x="182.88" y="-88.9"/>
+<instance part="R42" gate="G$1" x="167.64" y="-71.12"/>
+<instance part="VA105" gate="G$1" x="182.88" y="-53.34"/>
+<instance part="VR1" gate="G$1" x="149.86" y="-71.12"/>
+<instance part="VA103" gate="G$1" x="149.86" y="-58.42"/>
+<instance part="GND112" gate="GND" x="149.86" y="-88.9"/>
 <instance part="R48" gate="G$1" x="241.3" y="-78.74" rot="R90"/>
 <instance part="D7" gate="G$1" x="436.88" y="-45.72" rot="MR270"/>
@@
 <instance part="IN" gate="G$1" x="25.4" y="48.26"/>
 <instance part="OUT" gate="G$1" x="523.24" y="40.64"/>
+<instance part="Q8" gate="G$1" x="180.34" y="-71.12"/>
+<instance part="VA1" gate="G$1" x="129.54" y="-17.78"/>
 </instances>
 <busses>
@@
 <segment>
 <pinref part="VR2" gate="G$1" pin="1"/>
-<wire x1="187.96" y1="-81.28" x2="195.58" y2="-81.28" width="0.1524" layer="91"/>
-<wire x1="195.58" y1="-81.28" x2="195.58" y2="-49.53" width="0.1524" layer="91"/>
-<pinref part="Q8" gate="G$1" pin="C"/>
-<wire x1="187.96" y1="-76.2" x2="187.96" y2="-81.28" width="0.1524" layer="91"/>
+<wire x1="182.88" y1="-81.28" x2="195.58" y2="-81.28" width="0.1524" layer="91"/>
+<wire x1="195.58" y1="-81.28" x2="195.58" y2="-52.07" width="0.1524" layer="91"/>
+<wire x1="182.88" y1="-76.2" x2="182.88" y2="-81.28" width="0.1524" layer="91"/>
 <pinref part="GND114" gate="GND" pin="GND"/>
-<wire x1="187.96" y1="-86.36" x2="187.96" y2="-81.28" width="0.1524" layer="91"/>
-<junction x="187.96" y="-81.28"/>
+<wire x1="182.88" y1="-86.36" x2="182.88" y2="-81.28" width="0.1524" layer="91"/>
+<junction x="182.88" y="-81.28"/>
+<pinref part="Q8" gate="G$1" pin="E"/>
 </segment>
 <segment>
 <pinref part="R44" gate="G$1" pin="1"/>
 <pinref part="GND113" gate="GND" pin="GND"/>
-<wire x1="177.8" y1="-83.82" x2="177.8" y2="-86.36" width="0.1524" layer="91"/>
+<wire x1="175.26" y1="-83.82" x2="175.26" y2="-86.36" width="0.1524" layer="91"/>
 </segment>
 <segment>
 <pinref part="GND112" gate="GND" pin="GND"/>
 <pinref part="VR1" gate="G$1" pin="1"/>
-<wire x1="152.4" y1="-86.36" x2="152.4" y2="-77.47" width="0.1524" layer="91"/>
+<wire x1="149.86" y1="-86.36" x2="149.86" y2="-77.47" width="0.1524" layer="91"/>
 </segment>
 <segment>
@@
 <pinref part="IC1" gate="_PWR" pin="V+"/>
 <pinref part="V111" gate="+9V" pin="+9V"/>
-</segment>
-<segment>
-<pinref part="IC5" gate="_PWR" pin="V+"/>
-<pinref part="V104" gate="+9V" pin="+9V"/>
 </segment>
 <segment>
@@
 <segment>
 <pinref part="VA105" gate="G$1" pin="VA"/>
-<pinref part="Q8" gate="G$1" pin="E"/>
-<wire x1="187.96" y1="-55.88" x2="187.96" y2="-66.04" width="0.1524" layer="91"/>
+<wire x1="182.88" y1="-55.88" x2="182.88" y2="-66.04" width="0.1524" layer="91"/>
+<pinref part="Q8" gate="G$1" pin="C"/>
 </segment>
 <segment>
 <pinref part="R43" gate="G$1" pin="2"/>
 <pinref part="VA104" gate="G$1" pin="VA"/>
-<wire x1="177.8" y1="-58.42" x2="177.8" y2="-55.88" width="0.1524" layer="91"/>
+<wire x1="175.26" y1="-58.42" x2="175.26" y2="-55.88" width="0.1524" layer="91"/>
 </segment>
 <segment>
 <pinref part="VA103" gate="G$1" pin="VA"/>
 <pinref part="VR1" gate="G$1" pin="3"/>
-<wire x1="152.4" y1="-60.96" x2="152.4" y2="-64.77" width="0.1524" layer="91"/>
+<wire x1="149.86" y1="-60.96" x2="149.86" y2="-64.77" width="0.1524" layer="91"/>
+</segment>
+<segment>
+<pinref part="IC5" gate="_PWR" pin="V+"/>
+<pinref part="VA1" gate="G$1" pin="VA"/>
 </segment>
 </net>
@@
 <junction x="104.14" y="-50.8"/>
 <junction x="114.3" y="-50.8"/>
-<wire x1="114.3" y1="-50.8" x2="172.72" y2="-50.8" width="0.1524" layer="91"/>
-<wire x1="172.72" y1="-50.8" x2="172.72" y2="-33.02" width="0.1524" layer="91"/>
+<wire x1="114.3" y1="-50.8" x2="165.1" y2="-50.8" width="0.1524" layer="91"/>
+<wire x1="165.1" y1="-50.8" x2="165.1" y2="-33.02" width="0.1524" layer="91"/>
 <pinref part="IC5" gate="_A" pin="+IN"/>
-<wire x1="172.72" y1="-33.02" x2="175.26" y2="-33.02" width="0.1524" layer="91"/>
+<wire x1="165.1" y1="-33.02" x2="175.26" y2="-33.02" width="0.1524" layer="91"/>
 </segment>
 </net>
@@
 <junction x="195.58" y="-17.78"/>
 <pinref part="VR2" gate="G$1" pin="3"/>
-<wire x1="195.58" y1="-30.48" x2="195.58" y2="-36.83" width="0.1524" layer="91"/>
+<wire x1="195.58" y1="-30.48" x2="195.58" y2="-39.37" width="0.1524" layer="91"/>
 <junction x="195.58" y="-30.48"/>
 </segment>
@@
 <segment>
 <pinref part="VR2" gate="G$1" pin="2"/>
-<wire x1="200.66" y1="-43.18" x2="205.74" y2="-43.18" width="0.1524" layer="91"/>
-<wire x1="205.74" y1="-43.18" x2="205.74" y2="-91.44" width="0.1524" layer="91"/>
+<wire x1="200.66" y1="-45.72" x2="205.74" y2="-45.72" width="0.1524" layer="91"/>
+<wire x1="205.74" y1="-45.72" x2="205.74" y2="-91.44" width="0.1524" layer="91"/>
 <pinref part="R48" gate="G$1" pin="1"/>
 <wire x1="205.74" y1="-91.44" x2="241.3" y2="-91.44" width="0.1524" layer="91"/>
@@
 <segment>
 <pinref part="R42" gate="G$1" pin="2"/>
+<wire x1="172.72" y1="-71.12" x2="175.26" y2="-71.12" width="0.1524" layer="91"/>
+<pinref part="R43" gate="G$1" pin="1"/>
+<wire x1="175.26" y1="-71.12" x2="177.8" y2="-71.12" width="0.1524" layer="91"/>
+<wire x1="175.26" y1="-68.58" x2="175.26" y2="-71.12" width="0.1524" layer="91"/>
+<pinref part="R44" gate="G$1" pin="2"/>
+<wire x1="175.26" y1="-71.12" x2="175.26" y2="-73.66" width="0.1524" layer="91"/>
+<junction x="175.26" y="-71.12"/>
 <pinref part="Q8" gate="G$1" pin="B"/>
-<wire x1="175.26" y1="-71.12" x2="177.8" y2="-71.12" width="0.1524" layer="91"/>
-<pinref part="R43" gate="G$1" pin="1"/>
-<wire x1="177.8" y1="-71.12" x2="182.88" y2="-71.12" width="0.1524" layer="91"/>
-<wire x1="177.8" y1="-68.58" x2="177.8" y2="-71.12" width="0.1524" layer="91"/>
-<pinref part="R44" gate="G$1" pin="2"/>
-<wire x1="177.8" y1="-71.12" x2="177.8" y2="-73.66" width="0.1524" layer="91"/>
-<junction x="177.8" y="-71.12"/>
 </segment>
 </net>
@@
 <pinref part="VR1" gate="G$1" pin="2"/>
 <pinref part="R42" gate="G$1" pin="1"/>
-<wire x1="157.48" y1="-71.12" x2="165.1" y2="-71.12" width="0.1524" layer="91"/>
-</segment>
-</net>
+<wire x1="154.94" y1="-71.12" x2="162.56" y2="-71.12" width="0.1524" layer="91"/>
+</segment>
+</net>
