File: #Misc/Boss CE-3/ce3.sch (EAGLE design)
At the start: 136 parts, among them IC1 NJM4558DD, IC2 NJM4558DD, IC3 MN3207, IC4 MN3102, IC5 TL022, Q1 2SK30A-Y, Q10 2SC945-P, Q11 2SC945-P, Q12 2SC945-P, Q2 2SK30A-Y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

Commit message: 20180207
Parts:
- added VR3: 10kB, pedals-potentiometers:POTS16MM
- C30: value 470p -> 10n
- R3: value 33k -> 10k
- R54: value 2.7k -> 4.7k
- R63: value 56k -> 100R
- renumbered J1 to OUTPUT_B, J101 to INPUT, J102 to OUTPUT_A, JK1 to AC_ADAPTOR
Connections:
- new net N$78: R54.2, VR3.1
- new net N$79: R64.1, VR3.3
- net N$6: now also VR3.2; no longer R54.2, R64.1
Other:
- note added: "DEPTH"
- note added: "I"
- note added: "II"
- note added: "MODE"
- note added: "RATE"
- moved on the sheet: C20, R54, R64
