File: #Misc/Boss DS-1/ds1_redraw.sch (EAGLE design)
At the start: 137 parts, among them IC1 uPC4558C, IC2 uPC4558, IC3 MN3207, IC4 MN3102, IC5 TL022CP, IC6 LM78L05, Q1 2SC732TM-GR, Q10 2SC945-P, Q11 2SC945-P, Q2 2SC732TM-GR, Q3 2SC732TM-GR, Q4 1SK30A-Y, Q5 2SA733-P, Q6 2SC945-P, Q7 2SC945-P, Q8 2N3906-, Q9 2SC945-P, SW101 MOMENTARY

Commit message: 20171220
Parts:
- removed C10: 33n, pedals-capacitors-film:CER/FILMBOX.1
- removed C116, C38: 47n, pedals-capacitors-film:CER/FILMBOX.1
- removed C24: 1u, pedals-capacitors-elec:0400
- removed C25: 33u, pedals-capacitors-elec:0400
- removed C26, C33: 10n, pedals-capacitors-film:CER/FILMBOX.1
- removed C27, C28: 6.3u, pedals-capacitors-elec:0400
- removed C29, C40: 47u, pedals-capacitors-elec:0400
- removed C30: 47p, pedals-capacitors-film:CER/FILMBOX.1
- removed C31: 5p, pedals-capacitors-film:CER/FILMBOX.1
- removed C32: 22u, pedals-capacitors-elec:0400
- removed C34, C35: 470p, pedals-capacitors-film:CER/FILMBOX.1
- removed C36, C37: 220p, pedals-capacitors-film:CER/FILMBOX.1
- removed C39: 100u, pedals-capacitors-elec:0400
- removed D3, D8: 1S2473, pedals-diodes:DO35.2
- removed IC1: uPC4558C, pedals-integrated circuits:DUALTH
- removed IC2: uPC4558, pedals-integrated circuits:DUALTH
- removed IC3: MN3207, pedals-integrated circuits:BL3208
- removed IC4: MN3102, pedals-integrated circuits:CLOCK
- removed IC5: TL022CP, pedals-integrated circuits:DUALTH
- removed IC6: LM78L05, pedals-regulators:LM78L05
- removed LED: SLP1358, pedals-diodes:LED
- removed Q10, Q11: 2SC945-P, pedals-transistors:2SC828A
- removed R120: 1.5k, pedals-resistors:R_.3B
- removed R126: 39k, pedals-resistors:R_.3B
- removed R26: 47k, pedals-resistors:R_.3B
- removed R27, R53, R61, R62: 1M, pedals-resistors:R_.3B
- removed R38, R57, R58: 100k, pedals-resistors:R_.3B
- removed R40, R41: 10k, pedals-resistors:R_.3B
- removed R42: 68k, pedals-resistors:R_.3B
- removed R43: 150k, pedals-resistors:R_.3B
- removed R44: 470k, pedals-resistors:R_.3B
- removed R46: 330k, pedals-resistors:R_.3B
- removed R47, R51, R52: 4.7k, pedals-resistors:R_.3B
- removed R48: 220k, pedals-resistors:R_.3B
- removed R49, R50: 33k, pedals-resistors:R_.3B
- removed R54: 1k, pedals-resistors:R_.3B
- removed R55, R56, R59, R60: 56k, pedals-resistors:R_.3B
- removed R63: 3.9k, pedals-resistors:R_.3B
- removed SW101: MOMENTARY, pedals-switches:MOMENTARY
- removed VR4: 50kC, pedals-potentiometers:POTS16MM
- removed VR5: 22kB, pedals-potentiometers:POTS16MM
- removed VR6: (no value), pedals-potentiometers:POTS16MM
- removed VR7: 470kB, pedals-potentiometers:POTS16MM
- added C7: 250p, pedals-capacitors-film:CER/FILMBOX.1
- added D10: SLP1358, pedals-diodes:LED
- added IC: TA7136P, pedals-integrated circuits:SINGLETH
- added R10, R123, R127: 100k, pedals-resistors:R_.3B
- added SW: MOMENTARY, pedals-switches:MOMENTARY
- C11: value 1u -> 22n; device pedals-capacitors-elec:0400 -> pedals-capacitors-film:CER/FILMBOX.1
- C12: value 1u -> 100n; device pedals-capacitors-elec:0400 -> pedals-capacitors-film:CER/FILMBOX.1
- C13: value 33n -> 47n
- C14: value 3.9n -> 1u; device pedals-capacitors-film:CER/FILMBOX.1 -> pedals-capacitors-elec:0400
- C15: value 8.2 -> 47u; device pedals-capacitors-film:CER/FILMBOX.1 -> pedals-capacitors-elec:0400
- C16: value 330p -> 470p
- C17: value 220n -> 470p; device pedals-capacitors-elec:0400 -> pedals-capacitors-film:CER/FILMBOX.1
- C18: value 1n -> 220p
- C19: value 150p -> 220p
- C2: value 1u -> 470n
- C20: value 220n -> 470n; device pedals-capacitors-elec:0400 -> pedals-capacitors-film:CER/FILMBOX.1
- C21: value 47n -> 470n
- C22: value 100p -> 10n
- C23: value 6.8n -> 100u; device pedals-capacitors-film:CER/FILMBOX.1 -> pedals-capacitors-elec:0400
- C3: value 6.8n -> 47n
- C4: value 100p -> 250p
- C5: value 220p -> 470n; device pedals-capacitors-film:CER/FILMBOX.1 -> pedals-capacitors-elec:0400
- C6: value 47n -> 150p
- C8: value 12n -> 1u; device pedals-capacitors-film:CER/FILMBOX.1 -> pedals-capacitors-elec:0400
- C9: value 150p -> 470n
- Q4: value 1SK30A-Y -> 2SC945-P; device pedals-transistors:2N3819TO-92S -> pedals-transistors:2SC828A
- Q5: value 2SA733-P -> 2SC945-P; device pedals-transistors:2N3906- -> pedals-transistors:2SC828A
- Q6: value 2SC945-P -> 2SK30ATM-GR; device pedals-transistors:2SC828A -> pedals-transistors:2N3819TO-92S
- Q7: value 2SC945-P -> 2SK30ATM-Y; device pedals-transistors:2SC828A -> pedals-transistors:2N3819TO-92S
- Q8: value 2N3906- -> 2SK30ATM-Y; device pedals-transistors:2N3906- -> pedals-transistors:2N3819TO-92S
- R11: value 4.7k -> 100k
- R12: value 47k -> 27k
- R13: value 10k -> 4.7k
- R14, R15: value 10k -> 2.2k
- R16: value 10k -> 6.8k
- R17: value 100k -> 6.8k
- R18: value 56k -> 10k
- R19: value 330k -> 1M
- R20, R5: value 10k -> 1M
- R21, R23: value 10k -> 100k
- R22: value 10k -> 1k
- R24: value 47k -> 10k
- R25: value 22k -> 10k
- R28, R31: value 47k -> 56k
- R29: value 27k -> 56k
- R30: value 10k -> 56k
- R32: value 470R -> 1M
- R33: value 100k -> 1M
- R34: value 33k -> 1M
- R35: value 33k -> 3.9k
- R36: value 180k -> 1M
- R37: value 220k -> 100R
- R4, R6: value 47k -> 100k
- R7: value 10k -> 470k
- R8: value 220k -> 10k
- R9: value 82k -> 22R
- VR1, VR2: value 50kB -> 100kB
- VR3: value 250kC -> 20kB
Connections:
- removed net N$18: D3.C, D4.A, IC2_B.OUT, R12.2, R14.1
- removed net N$24: C11.+, R17.1, VR6.2
- removed net N$46: C16.1, Q3.B, R22.2
- removed net N$51: C22.2, C23.2, IC1_A.-IN, R28.1, R29.2, R31.1
- removed net N$52: C21.2, Q4.S, R29.1
- removed net N$53: C20.-, Q4.D, R27.2
- removed net N$54: C22.1, IC1_A.OUT, R30.2, R31.2, R32.1
- removed net N$55: C24.+, R32.2
- removed net N$57: C23.1, R30.1
- removed net N$58: R126.2, VR5.2, VR5.3
- removed net N$59: C116.2, VR5.1
- removed net N$60: C21.1, VR4.3
- removed net N$61: C116.1, VR4.2
- removed net N$62: C31.1, Q5.B, R49.2, R50.1
- removed net N$63: D6.A, Q5.C, R51.2
- removed net N$64: C30.1, D6.C, IC4.P$7, R52.2
- removed net N$65: C30.2, C31.2, IC4.P$5, R49.1
- removed net N$66: Q7.C, R52.1
- removed net N$67: R46.2, VR7.2, VR7.3
- removed net N$68: Q6.B, Q6.C, R46.1, R47.1
- removed net N$69: C32.+, Q7.B, R47.2, R48.2
- removed net N$70: C26.2, IC5_B.-IN, R38.2
- removed net N$71: C29.+, IC5_A.+IN, R38.1, R40.1, R41.2
- removed net N$72: C26.1, IC5_B.OUT, R37.2, VR3.1, VR3.2
- removed net N$73: R120.1, VR3.3
- removed net N$74: IC5_B.+IN, R36.1, R37.1
- removed net N$75: C27.+, IC5_A.-IN, R120.2
- removed net N$76: C28.+, IC5_A.OUT, R36.2, VR2.3
- removed net N$77: C27.-, C28.-
- removed net N$78: R48.1, VR2.2
- removed net N$79: D8.C, R62.1
- removed net N$80: Q8.B, R42.2, R43.1, R44.2
- removed net N$81: R42.1, VR1.2
- removed net N$82: Q11.B, R62.2
- removed net N$85: R54.2, SW101.P
- removed net VA: C40.+, IC3.5, IC4.P$1, IC6.VO, Q5.E, Q8.E, R40.2, R43.2, R50.2, VR1.3, VR6.3, VR7.1
- new net N$1: C11.2, R15.2
- new net N$2: C12.1, R16.1, VR3.1
- net +9V: now also C23.+, IC.V+, R12.1, R24.1, R30.2, R31.2, R36.2, R8.2; no longer C39.+, IC1_PWR.V+, IC2_PWR.V+, IC5_PWR.V+, IC6.VI, Q2.C, R34.2, R53.2, R55.2, R56.2
- net GND: now also C15.-, C22.2, C23.-, C8.-, IC.V-, Q4.E, Q5.E, Q9.E, R21.1, R25.1, R28.1, R29.1, R6.1, R9.1, SW.P; no longer C11.-, C12.-, C14.2, C16.2, C18.2, C25.-, C29.-, C32.-, C33.2, C38.2, C39.-, C40.-, C9.2, D7.C, D9.C, IC1_PWR.V-, IC2_PWR.V-, IC3.1, IC4.P$3, IC5_PWR.V-, Q11.E, Q6.E, Q7.E, Q8.C, R16.1, R18.1, R33.2, R35.1, R41.1, R44.1, R51.1, R59.1, R60.1, SW101.S, VR1.1, VR2.1, VR4.1, VR6.1
- net N$10: now also Q2.E, R9.2; no longer C4.2, IC1_B.-IN, R4.2, R5.2, R6.1
- net N$11: now also C4.1, C5.+, Q2.C, R8.1; no longer IC1_B.+IN
- net N$12: now also C5.-, IC.-IN, R10.2; no longer C4.1, IC1_B.OUT, R28.2, R6.2, R8.1, R9.1
- net N$13: now also IC.ON2, R12.2; no longer C5.1, R8.2
- net N$14: now also IC.ON1; no longer C5.2, R9.2
- net N$15: now also C6.1, C7.1, IC.OUT, R14.1, VR1.1; no longer IC2_B.+IN, R13.2
- net N$16: now also IC.+IN, R11.2; no longer C6.1, IC2_B.-IN, R11.1, R12.1, R126.1
- net N$17: now also C7.2, R11.1, VR1.2; no longer D3.A, D4.C, R11.2
- net N$19: now also C8.+, R13.1; no longer C8.1, R14.2, R15.1
- net N$20: now also R13.2, VR1.3; no longer C9.1, Q2.B, R15.2
- net N$21: now also C9.2, R14.2; no longer C10.2, C8.2, Q2.E, R16.2
- net N$22: now also C11.1, C9.1, D4.C, D5.A, R16.2; no longer D9.A, IC6.GND
- net N$23: now also R15.1, R17.2, VR3.3; no longer C13.1, IC3.7, IC3.8, R18.2
- net N$25: now also VR2.3, VR3.2; no longer C10.1, IC3.3, R17.2
- net N$26: now also R18.1, VR2.2; no longer IC3.2, IC4.P$2
- net N$29: now also C16.2, Q4.C, R123.1, R30.1, R32.1; no longer C34.2, Q9.C, R55.1, R57.1
- net N$31: now also C17.1, Q5.C, R127.2, R31.1, R33.1, R34.1; no longer C35.1, Q10.C, R56.1, R58.2
- net N$32: now also C17.2, C18.1, Q4.B, R127.1, R28.2; no longer C35.2, C36.1, Q9.B, R58.1, R59.2
- net N$33: now also Q7.S, R18.2; no longer IC3.6, IC4.P$4
- net N$34: now also C16.1, C19.1, Q5.B, R123.2, R29.2; no longer C34.1, C37.1, Q10.B, R57.2, R60.2
- net N$35: now also C18.2, C19.2, C22.1, R36.1, R37.2; no longer LED.C, Q11.C
- net N$36: now also C21.2, D7.C, R33.2; no longer C33.1, C36.2, C37.2, R53.1, R54.1
- net N$37: now also D6.A, Q8.G; no longer D7.A, D8.A, Q10.E, Q9.E, R61.1
- net N$38: now also C20.2, D6.C, R32.2; no longer D5.A, Q4.G
- net N$39: now also D7.A, Q6.G, Q7.G; no longer C38.1, D5.C, R61.2
- net N$40: now also C13.2, Q7.D, Q8.D, R19.2; no longer C17.+, R24.1
- net N$41: now also C13.1, Q3.B, R20.2; no longer C13.2, R19.2, R20.1
- net N$42: now also D10.A, R35.1; no longer LED.A, R63.1
- net N$43: now also R35.2; no longer R63.2
- net N$44: now also Q3.E, R21.2, R22.1; no longer C14.1, R20.2, R21.1
- net N$45: now also C14.+, R22.2; no longer C15.1, R21.2, R22.1
- net N$47: now also D10.C, Q9.C; no longer C15.2, C17.-, Q3.E, R23.2
- net N$48: now also D9.A, R34.2; no longer C18.1, R24.2, R25.1, R26.1
- net N$49: now also R37.1, SW.S; no longer C19.2, IC2_A.-IN, R25.2
- net N$5: now also C3.2, Q6.D, R5.2; no longer C12.+, IC3.4, IC4.P$8
- net N$50: now also D9.C, Q9.B; no longer C19.1, C20.+, IC2_A.OUT, R26.2
- net N$8: now also Q6.S, Q8.S, R4.2; no longer C3.2, R4.1
- net N$9: now also C4.2, Q2.B, R6.2, R7.1; no longer R5.1
- net OUT: now also C14.-, R23.2; no longer C24.-, R33.1
- net VB: now also C12.2, C15.+, C20.1, C21.1, D4.A, D5.C, R10.1, R17.1, R20.1, R24.2, R25.2, R4.1, R5.1, VR2.1; no longer C25.+, IC1_A.+IN, IC2_A.+IN, R13.1, R27.1, R34.1, R35.2, R7.1
Other:
- note removed: "12"
- note removed: "13"
- moved on the sheet: C13, C16, C18, C19, C21, C22, C3, C4, C6, C9, D1, D2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

Commit message: 20180207
Parts:
- C20, C21: value 470n -> 47n
Other:
- note added: "DIST"
- note added: "LEVEL"
- note added: "TONE"
Changed lines of the file:
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@@
 <?xml version="1.0" encoding="utf-8"?>
 <!DOCTYPE eagle SYSTEM "eagle.dtd">
-<eagle version="8.2.0">
+<eagle version="8.5.1">
 <drawing>
 <settings>
 <setting alwaysvectorfont="no"/>
+<setting keepoldvectorfont="yes"/>
 <setting verticaltext="up"/>
 </settings>
-<grid distance="0.1" unitdist="inch" unit="inch" style="lines" multiple="1" display="yes" altdistance="0.01" altunitdist="inch" altunit="inch"/>
+<grid distance="0.1" unitdist="inch" unit="inch" style="lines" multiple="1" display="no" altdistance="0.01" altunitdist="inch" altunit="inch"/>
 <layers>
 <layer number="1" name="Top" color="4" fill="1" visible="no" active="no"/>
@@
 <part name="R32" library="pedals-resistors" deviceset="R_" device=".3B" value="1M"/>
 <part name="D7" library="pedals-diodes" deviceset="DO35" device=".2" value="1S2473"/>
-<part name="C21" library="pedals-capacitors-film" deviceset="CER/FILM" device="BOX.1" value="470n"/>
+<part name="C21" library="pedals-capacitors-film" deviceset="CER/FILM" device="BOX.1" value="47n"/>
 <part name="D6" library="pedals-diodes" deviceset="DO35" device=".2" value="1S2473"/>
-<part name="C20" library="pedals-capacitors-film" deviceset="CER/FILM" device="BOX.1" value="470n"/>
+<part name="C20" library="pedals-capacitors-film" deviceset="CER/FILM" device="BOX.1" value="47n"/>
 <part name="Q8" library="pedals-transistors" deviceset="2N3819" device="TO-92S" value="2SK30ATM-Y"/>
 <part name="R36" library="pedals-resistors" deviceset="R_" device=".3B" value="1M"/>
@@
 <sheet>
 <plain>
+<text x="177.8" y="30.48" size="1.778" layer="95" rot="R90">DIST</text>
+<text x="225.298" y="39.878" size="1.778" layer="95" rot="R90">TONE</text>
+<text x="235.458" y="32.512" size="1.778" layer="95" rot="R90">LEVEL</text>
 </plain>
 <instances>

Commit message: 20180529
Parts:
- added C10: 10n, pedals-capacitors-film:CER/FILMBOX.1
Connections:
- net N$22: now also C10.1
- net VB: now also C10.2
Other:
- moved on the sheet: C11, C12, C13, C14, C16, C17, C18, C19, C20, C21, C22, D10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
