File: #Misc/Boss DS-2/ds2_redraw.sch (EAGLE design)
At the start: 137 parts, among them IC1 uPC4558C, IC2 uPC4558, IC3 MN3207, IC4 MN3102, IC5 TL022CP, IC6 LM78L05, Q1 2SC732TM-GR, Q10 2SC945-P, Q11 2SC945-P, Q2 2SC732TM-GR, Q3 2SC732TM-GR, Q4 1SK30A-Y, Q5 2SA733-P, Q6 2SC945-P, Q7 2SC945-P, Q8 2N3906-, Q9 2SC945-P, SW101 MOMENTARY

Commit message: 20171220
Parts:
- removed C116: 47n, pedals-capacitors-film:CER/FILMBOX.1
- removed IC1: uPC4558C, pedals-integrated circuits:DUALTH
- removed IC2: uPC4558, pedals-integrated circuits:DUALTH
- removed IC3: MN3207, pedals-integrated circuits:BL3208
- removed IC4: MN3102, pedals-integrated circuits:CLOCK
- removed IC5: TL022CP, pedals-integrated circuits:DUALTH
- removed IC6: LM78L05, pedals-regulators:LM78L05
- removed Q6, Q9: 2SC945-P, pedals-transistors:2SC828A
- removed R120: 1.5k, pedals-resistors:R_.3B
- removed R126: 39k, pedals-resistors:R_.3B
- removed R22: 10k, pedals-resistors:R_.3B
- removed R27: 1M, pedals-resistors:R_.3B
- removed SW101: MOMENTARY, pedals-switches:MOMENTARY
- removed VR4: 50kC, pedals-potentiometers:POTS16MM
- removed VR5: 22kB, pedals-potentiometers:POTS16MM
- removed VR6: (no value), pedals-potentiometers:POTS16MM
- removed VR7: 470kB, pedals-potentiometers:POTS16MM
- added 16, Q16, Q19: 2SK-184GR, pedals-transistors:2N3819TO-92S
- added C41: 2.2n, pedals-capacitors-film:CER/FILMBOX.1
- added C42: 10u, pedals-capacitors-elec:0400
- added C43, C7: 47n, pedals-capacitors-film:CER/FILMBOX.1
- added C44: 1n, pedals-capacitors-film:CER/FILMBOX.1
- added C45: 22n, pedals-capacitors-film:CER/FILMBOX.1
- added D10, D11, D12, D13: 1SS-133, pedals-diodes:DO35.2
- added D14, D15: 1SS-188FM, pedals-diodes:DO35.2
- added Q106: 2SA-1048GR, pedals-transistors:2N3906-
- added Q12, Q18, Q22, Q23: 2SC-3378GR, pedals-transistors:2SC828A
- added Q13: 2SC945-P, pedals-transistors:2SC828A
- added Q14, Q15, Q20: 2SK-118Y, pedals-transistors:2N3819TO-92S
- added Q17: 2SA-1335GR, pedals-transistors:2N3906-
- added Q21: 2N3819TO-92S, pedals-transistors:2N3819TO-92S
- added R10: 1M, pedals-resistors:R_.3B
- added R154: 56k, pedals-resistors:R_.3B
- added R1A, R64, R68: 10k, pedals-resistors:R_.3B
- added R39, R69, R70, R71: 100k, pedals-resistors:R_.3B
- added R45, R72: 4.7k, pedals-resistors:R_.3B
- added R65: 2.2k, pedals-resistors:R_.3B
- added R66: 1.5k, pedals-resistors:R_.3B
- added R67: 220R, pedals-resistors:R_.3B
- added SW1: MOMENTARY, pedals-switches:MOMENTARY
- added SW2: (no value), pedals-switches:SPDT
- C1, C21: value 47n -> 10n
- C10: value 33n -> 1u; device pedals-capacitors-film:CER/FILMBOX.1 -> pedals-capacitors-elec:0400
- C11: value 1u -> 100u
- C12: value 1u -> 47n; device pedals-capacitors-elec:0400 -> pedals-capacitors-film:CER/FILMBOX.1
- C13: value 33n -> 10u; device pedals-capacitors-film:CER/FILMBOX.1 -> pedals-capacitors-elec:0400
- C14: value 3.9n -> 10u; device pedals-capacitors-film:CER/FILMBOX.1 -> pedals-capacitors-elec:0400
- C15: value 8.2 -> 1u; device pedals-capacitors-film:CER/FILMBOX.1 -> pedals-capacitors-elec:0400
- C16: value 330p -> 100u; device pedals-capacitors-film:CER/FILMBOX.1 -> pedals-capacitors-elec:0400
- C17: value 220n -> 47u
- C18: value 1n -> 47n
- C19: value 150p -> 10n
- C2: value 1u -> 10n; device pedals-capacitors-elec:0400 -> pedals-capacitors-film:CER/FILMBOX.1
- C20: value 220n -> 47n; device pedals-capacitors-elec:0400 -> pedals-capacitors-film:CER/FILMBOX.1
- C22: value 100p -> 10u; device pedals-capacitors-film:CER/FILMBOX.1 -> pedals-capacitors-elec:0400
- C23: value 6.8n -> 1u; device pedals-capacitors-film:CER/FILMBOX.1 -> pedals-capacitors-elec:0400
- C25: value 33u -> 6.8n; device pedals-capacitors-elec:0400 -> pedals-capacitors-film:CER/FILMBOX.1
- C26: value 10n -> 1n
- C27: value 6.3u -> 10u
- C28: value 6.3u -> 4.7n; device pedals-capacitors-elec:0400 -> pedals-capacitors-film:CER/FILMBOX.1
- C29: value 47u -> 470p; device pedals-capacitors-elec:0400 -> pedals-capacitors-film:CER/FILMBOX.1
- C3: value 6.8n -> 220p
- C30: value 47p -> 10u; device pedals-capacitors-film:CER/FILMBOX.1 -> pedals-capacitors-elec:0400
- C31: value 5p -> 1n
- C32: value 22u -> 100p; device pedals-capacitors-elec:0400 -> pedals-capacitors-film:CER/FILMBOX.1
- C33: value 10n -> 220n; device pedals-capacitors-film:CER/FILMBOX.1 -> pedals-capacitors-elec:0400
- C34: value 470p -> 2.2n
- C35: value 470p -> 10u; device pedals-capacitors-film:CER/FILMBOX.1 -> pedals-capacitors-elec:0400
- C36: value 220p -> 10u; device pedals-capacitors-film:CER/FILMBOX.1 -> pedals-capacitors-elec:0400
- C37: value 220p -> 6.8n
- C38: value 47n -> 1u; device pedals-capacitors-film:CER/FILMBOX.1 -> pedals-capacitors-elec:0400
- C39: value 100u -> 47n; device pedals-capacitors-elec:0400 -> pedals-capacitors-film:CER/FILMBOX.1
- C4: value 100p -> 470p
- C40: value 47u -> 47n; device pedals-capacitors-elec:0400 -> pedals-capacitors-film:CER/FILMBOX.1
- C6: value 47n -> 470p
- C8: value 12n -> 47n
- C9: value 150p -> 1u; device pedals-capacitors-film:CER/FILMBOX.1 -> pedals-capacitors-elec:0400
- D1: value RD11EB-3 -> MTZ5.6B
- D2: value RD5.1EB-3 -> S5500G; device pedals-diodes:ZENER.2 -> pedals-diodes:DO35.2
- D3, D4, D5, D6, D7, D8, D9: value 1S2473 -> 1SS-133
- LED: value SLP1358 -> LED
- Q1, Q2: value 2SC732TM-GR -> 2SC945-P
- Q10: value 2SC945-P -> 2SK-118Y; device pedals-transistors:2SC828A -> pedals-transistors:2N3819TO-92S
- Q11: value 2SC945-P -> 2SC-3378GR
- Q3: value 2SC732TM-GR -> 2SK-118Y; device pedals-transistors:2SC828A -> pedals-transistors:2N3819TO-92S
- Q4: value 1SK30A-Y -> 2SK-118Y
- Q5: value 2SA733-P -> 2SC-3378GR; device pedals-transistors:2N3906- -> pedals-transistors:2SC828A
- Q7: value 2SC945-P -> 2SC-2458GR
- Q8: value 2N3906- -> 2SA-1048GR
- R1: value 1k -> 1M
- R11: value 4.7k -> 100k
- R12: value 47k -> 4.7k
- R14, R21, R5: value 10k -> 100k
- R15: value 10k -> 4.7k
- R16, R23, R7: value 10k -> 1M
- R17, R38, R57: value 100k -> 4.7k
- R18, R60: value 56k -> 100k
- R19: value 330k -> 10k
- R2: value 470k -> 100R
- R24: value 47k -> 10k
- R25: value 22k -> 100k
- R26: value 47k -> 100k
- R29: value 27k -> 47k
- R3: value 10k -> 1.2k
- R31: value 47k -> 1M
- R32: value 470R -> 1M
- R33: value 100k -> 22k
- R34: value 33k -> 4.7k
- R35: value 33k -> 150k
- R36: value 180k -> 100k
- R37: value 220k -> 100k
- R4, R6: value 47k -> 56k
- R40: value 10k -> 1k
- R42: value 68k -> 10k
- R43: value 150k -> 4.7k
- R44: value 470k -> 22k
- R46: value 330k -> 33k
- R48: value 220k -> 150k
- R49: value 33k -> 100k
- R50: value 33k -> 2.2k
- R51: value 4.7k -> 2.2k
- R53, R62: value 1M -> 4.7k
- R55, R59: value 56k -> 1k
- R56: value 56k -> 1M
- R58: value 100k -> 15k
- R61: value 1M -> 100k
- R63: value 3.9k -> 100k
- R8: value 220k -> 56k
- R9: value 82k -> 100k
- VR1: value 50kB -> 250kD
- VR2: value 50kB -> 100kG
- VR3: value 250kC -> 50kA
Connections:
- removed net N$53: C20.-, Q4.D, R27.2
- removed net N$81: R42.1, VR1.2
- new net N$28: D6.A, Q15.G
- new net N$30: D7.A, Q14.G
- new net N$56: R55.1, VR1.1
- new net N$6: C36.-, D11.A, D12.C, R57.2
- new net N$83: C2.1, LED.C, R3.2
- new net N$84: R2.2, SW1.P
- net +9V: now also 16.D, C11.+, LED.A, Q106.E, Q7.C, Q8.E, R1.2, R15.2, R154.2, R25.2, R28.2, R4.2; no longer C39.+, D1.C, IC1_PWR.V+, IC2_PWR.V+, IC5_PWR.V+, IC6.VI, Q1.C, Q2.C, Q3.C, R34.2, R53.2, R55.2, R56.2
- net GND: now also C1.2, C14.-, C16.-, C17.-, C19.2, C2.2, C20.2, C21.2, C22.-, C25.2, C26.2, C33.-, C42.-, C44.2, C7.2, C8.2, D11.C, D12.A, D14.C, D15.A, D2.A, Q1.E, Q2.E, R12.1, R17.1, R19.1, R24.1, R30.1, R34.1, R38.1, R39.1, R43.1, R52.1, R53.1, R6.1, R66.1, R72.1, R8.1, SW1.S, SW2.O, VR3.1; no longer C12.-, C14.2, C16.2, C25.-, C29.-, C32.-, C33.2, C38.2, C39.-, C40.-, C9.2, D1.A, D7.C, D9.C, IC1_PWR.V-, IC2_PWR.V-, IC3.1, IC4.P$3, IC5_PWR.V-, Q11.E, Q6.E, Q7.E, Q8.C, R16.1, R18.1, R23.1, R3.1, R33.2, R41.1, R44.1, R59.1, R60.1, SW101.S, VR1.1, VR2.1, VR4.1, VR6.1
- net IN: now also R13.1; no longer R1.1
- net N$10: now also C15.-, Q21.D, R18.2; no longer C4.2, IC1_B.-IN, R4.2, R5.2, R6.1
- net N$11: now also D13.A, Q21.G; no longer IC1_B.+IN, R7.2
- net N$12: now also C38.+, Q21.S, R60.2; no longer C4.1, IC1_B.OUT, R28.2, R6.2, R8.1, R9.1
- net N$13: now also C38.-, R62.1; no longer C5.1, R8.2
- net N$14: now also C40.2, D14.A, D15.C, R62.2; no longer C5.2, C6.2, R9.2
- net N$15: now also C40.1, Q22.B, R63.2; no longer IC2_B.+IN, R13.2
- net N$16: now also Q22.E, R66.2, R67.2; no longer C6.1, IC2_B.-IN, R11.1, R12.1, R126.1
- net N$17: now also C42.+, R67.1; no longer D3.A, D4.C, R11.2
- net N$18: now also C39.2, C41.2, Q22.C, R65.1, R69.1; no longer D3.C, D4.A, IC2_B.OUT, R12.2, R14.1
- net N$19: now also C43.2, C45.2, Q23.E, R72.2; no longer C8.1, R14.2, R15.1
- net N$20: now also C43.1, R69.2, R70.1; no longer C9.1, Q2.B, R15.2
- net N$21: now also C44.1, Q23.B, R70.2; no longer C10.2, C8.2, Q2.E, R16.2
- net N$22: now also C45.1, R68.1, R71.2; no longer D9.A, IC6.GND
- net N$23: now also C41.1, R64.1; no longer C13.1, IC3.7, IC3.8, R18.2
- net N$24: now also Q15.D, R64.2, R68.2; no longer C11.+, R17.1, VR6.2
- net N$25: now also C39.1, Q14.D, R61.2; no longer C10.1, IC3.3, R17.2
- net N$26: now also Q14.S, Q15.S, Q16.G, R49.2; no longer IC3.2, IC4.P$2
- net N$29: now also C6.2, Q2.C, R10.1, R154.1, R9.1; no longer C34.2, Q9.C, R55.1, R57.1
- net N$3: now also C35.-, R57.1; no longer C1.2, R1.2
- net N$31: now also C4.1, D1.A, Q1.C, R4.1, R5.2, R7.1; no longer C35.1, Q10.C, R56.1, R58.2
- net N$32: now also C4.2, C5.1, Q2.B, R5.1, R8.2; no longer C35.2, C36.1, Q9.B, R58.1, R59.2
- net N$33: now also Q16.S, Q19.S, R53.2; no longer IC3.6, IC4.P$4
- net N$34: now also C3.1, C6.1, Q1.B, R6.2, R9.2; no longer C34.1, C37.1, Q10.B, R57.2, R60.2
- net N$35: now also C1.1, C3.2, C5.2, R1.1, R2.1; no longer LED.C, Q11.C
- net N$36: now also C8.1, D13.C, D4.C, R10.2; no longer C33.1, C36.2, C37.2, R53.1, R54.1
- net N$37: now also C9.+, Q4.S, R11.2; no longer D7.A, D8.A, Q10.E, Q9.E, R61.1
- net N$38: now also D4.A; no longer D5.A
- net N$39: now also C31.2, Q16.D, Q17.B, R50.1; no longer C38.1, D5.C, R61.2
- net N$4: now also C14.+, Q7.B, R15.1; no longer C1.1, Q1.B, R2.2
- net N$40: now also C31.1, Q17.C, Q18.B, R51.2; no longer C17.+, R24.1
- net N$41: now also C36.+, R58.2, R59.1; no longer C13.2, R19.2, R20.1
- net N$42: now also C13.-, Q5.B, R21.2; no longer LED.A, R63.1
- net N$43: now also C7.1, D3.C, R7.2; no longer D2.A, R63.2
- net N$44: now also C32.2, D8.C, D9.A, Q19.G, R54.2, R55.2; no longer C14.1, R20.2, R21.1
- net N$45: now also C34.2, D8.A, D9.C; no longer C15.1, R21.2, R22.1
- net N$46: now also C30.+, C37.2, R46.2, R58.1; no longer C16.1, Q3.B, R22.2
- net N$47: now also C9.-, VR3.2; no longer C15.2, C17.-, Q3.E, R23.2
- net N$48: now also C23.+, Q3.S, Q4.D, R36.2; no longer C18.1, R24.2, R25.1, R26.1
- net N$49: now also C10.-, Q5.E, R12.2; no longer C19.2, IC2_A.-IN, R25.2
- net N$5: now also D10.A, Q20.G; no longer C12.+, IC3.4, IC4.P$8
- net N$50: now also C10.+, Q3.D, R14.2; no longer C19.1, C20.+, IC2_A.OUT, R26.2
- net N$51: now also C34.1, Q20.D, R56.1; no longer C22.2, C23.2, IC1_A.-IN, R28.1, R29.2, R31.1
- net N$52: now also C28.1, C29.1, Q13.C, R33.2, R45.1, R46.1, R47.1; no longer C21.2, Q4.S, R29.1
- net N$54: now also D3.A, Q3.G; no longer C22.1, IC1_A.OUT, R30.2, R31.2, R32.1
- net N$55: now also C33.+, R54.1; no longer C24.+, R32.2
- net N$57: now also R45.2, VR2.1; no longer C23.1, R30.1
- net N$58: now also R59.2, VR2.3; no longer R126.2, VR5.2, VR5.3
- net N$59: now also C37.1, VR2.2; no longer C116.2, VR5.1
- net N$60: now also C29.2, C30.-, Q13.B, R35.2, R48.1; no longer C21.1, VR4.3
- net N$61: now also D5.A, Q10.G; no longer C116.1, VR4.2
- net N$62: now also C22.+, Q13.E, R34.2; no longer C31.1, Q5.B, R49.2, R50.1
- net N$63: now also C28.2, Q12.B, R44.1; no longer D6.A, Q5.C, R51.2
- net N$64: now also C21.1, Q10.S, R32.1; no longer C30.1, D6.C, IC4.P$7, R52.2
- net N$65: now also Q10.D, R32.2, R33.1, R44.2; no longer C30.2, C31.2, IC4.P$5, R49.1
- net N$66: now also Q12.E, R42.2, R43.2; no longer Q7.C, R52.1
- net N$67: now also C26.1, C27.-, R41.2, R42.1; no longer R46.2, VR7.2, VR7.3
- net N$68: now also C25.1, R41.1; no longer Q6.B, Q6.C, R46.1, R47.1
- net N$69: now also C19.1, R1A.1, R28.1, R29.2; no longer C32.+, Q7.B, R47.2, R48.2
- net N$7: now also C12.2, R13.2; no longer C2.-, Q1.E, R3.2
- net N$70: now also C27.+, VR3.3; no longer C26.2, IC5_B.-IN, R38.2
- net N$71: now also Q106.B, R29.1; no longer C29.+, IC5_A.+IN, R38.1, R40.1, R41.2
- net N$72: now also C32.1, C35.+, Q18.E, Q20.S, R52.2, R56.2, VR1.2, VR1.3; no longer C26.1, IC5_B.OUT, R37.2, VR3.1, VR3.2
- net N$73: now also Q8.B, R25.1, R26.1; no longer R120.1, VR3.3
- net N$74: now also Q8.C, R23.2, R24.2; no longer IC5_B.+IN, R36.1, R37.1
- net N$75: now also C20.1, D10.C, D5.C, D7.C, R31.2; no longer C27.+, IC5_A.-IN, R120.2
- net N$76: now also R1A.2, SW2.P; no longer C28.+, IC5_A.OUT, R36.2, VR2.3
- net N$77: now also C23.-, Q11.B, R37.2; no longer C27.-, C28.-
- net N$78: now also C24.+, Q11.E, R38.2; no longer R48.1, VR2.2
- net N$79: now also Q106.C, R26.2, R30.2, R31.1; no longer D8.C, R62.1
- net N$8: now also 16.G, C12.1, R16.2; no longer C2.+, C3.2, R4.1
- net N$80: now also C24.-, R39.2, R40.1; no longer Q8.B, R42.2, R43.1, R44.2
- net N$82: now also D1.C, R3.1; no longer Q11.B, R62.2
- net N$85: now also C18.1, D6.C, R23.1; no longer R54.2, SW101.P
- net N$9: now also 16.S, C13.+, C15.+, R17.2; no longer C3.1, R5.1
- net OUT: now also R40.2; no longer C24.-, R33.1
- net VA: now also C16.+, Q11.C, Q12.C, Q17.E, Q18.C, Q19.D, Q23.C, Q5.C, Q7.E, R20.2, R47.2, R48.2, R65.2; no longer C40.+, IC3.5, IC4.P$1, IC6.VO, Q5.E, Q8.E, R40.2, R43.2, VR1.3, VR6.3, VR7.1
- net VB: now also C17.+, R11.1, R14.1, R16.1, R18.1, R19.2, R20.1, R21.1, R36.1, R37.1, R49.1, R60.1, R61.1, R63.1, R71.1; no longer C25.+, IC1_A.+IN, IC2_A.+IN, R13.1, R19.1, R2.1, R27.1, R34.1, R35.2, R7.1
Other:
- note removed: "12"
- note removed: "13"
- moved on the sheet: C1, C11, C17, C18, C19, C21, C24, C26, C27, C3, C31, C34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

Commit message: 20180529
Parts:
- removed Q106: 2SA-1048GR, pedals-transistors:2N3906-
- removed R154: 56k, pedals-resistors:R_.3B
- removed R1A: 10k, pedals-resistors:R_.3B
- added Q9: 2SA-1048GR, pedals-transistors:2N3906-
- added R1 : 10k, pedals-resistors:R_.3B
- added R22: 56k, pedals-resistors:R_.3B
- R69, R70: value 100k -> 22k
- renumbered 16 to Q6
Connections:
- net +9V: now also Q9.E, R22.2; no longer Q106.E, Q6.D, R154.2
- net N$29: now also R22.1; no longer R154.1
- net N$37: now also Q4.D; no longer Q4.S
- net N$48: now also Q4.S; no longer Q4.D
- net N$69: now also R1 .1; no longer R1A.1
- net N$71: now also Q9.B; no longer Q106.B
- net N$76: now also R1 .2; no longer R1A.2
- net N$79: now also Q9.C; no longer Q106.C
- net VA: now also Q6.D
Other:
- moved on the sheet: C1, C10, C13, C18, C19, C2, C21, C22, C23, C24, C25, C26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
