File: #Misc/Boss HM-2/hm2_redraw.sch (EAGLE design)
At the start: 118 parts, among them Q1 2N5457, Q10 2N5457, Q4 2N5457, Q5 2N5457, SW1 MOMENTARY

Commit message: 20180207
Parts:
- ICA3: value (none) -> M5216L
- R24: value 10k -> 68k
Connections:
- removed net N$35: D6.C, D7.A, R30.1
- new net N$1: D6.A, D7.C, R30.1
- net N$33: now also D6.C, D7.A; no longer D6.A, D7.C
- net N$63: now also C8.-; no longer C8.+
- net N$64: now also C8.+; no longer C8.-
Changed lines of the file:
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@@
 <?xml version="1.0" encoding="utf-8"?>
 <!DOCTYPE eagle SYSTEM "eagle.dtd">
-<eagle version="8.2.0">
+<eagle version="8.5.1">
 <drawing>
 <settings>
 <setting alwaysvectorfont="no"/>
+<setting keepoldvectorfont="yes"/>
 <setting verticaltext="up"/>
 </settings>
-<grid distance="0.1" unitdist="inch" unit="inch" style="lines" multiple="1" display="yes" altdistance="0.01" altunitdist="inch" altunit="inch"/>
+<grid distance="0.1" unitdist="inch" unit="inch" style="lines" multiple="1" display="no" altdistance="0.01" altunitdist="inch" altunit="inch"/>
 <layers>
 <layer number="1" name="Top" color="4" fill="1" visible="no" active="no"/>
@@
 <part name="GND11" library="gm-supply" deviceset="GND" device=""/>
 <part name="C15" library="pedals-capacitors-elec" deviceset="040" device="0" value="1u"/>
-<part name="R24" library="pedals-resistors" deviceset="R_" device=".3B" value="10k"/>
+<part name="R24" library="pedals-resistors" deviceset="R_" device=".3B" value="68k"/>
 <part name="VB5" library="gm-supply" deviceset="VB" device=""/>
 <part name="V4" library="gm-supply" deviceset="+9V" device=""/>
 <part name="GND12" library="gm-supply" deviceset="GND" device=""/>
-<part name="ICA3" library="pedals-integrated circuits" deviceset="DUAL" device="TH"/>
+<part name="ICA3" library="pedals-integrated circuits" deviceset="DUAL" device="TH" value="M5216L"/>
 <part name="R52" library="pedals-resistors" deviceset="R_" device=".3B" value="3.3k"/>
 <part name="C33" library="pedals-capacitors-film" deviceset="CER/FILM" device="BOX.1" value="470p"/>
@@
 <instance part="C12" gate="1" x="233.68" y="45.72"/>
 <instance part="R23" gate="G$1" x="246.38" y="45.72"/>
-<instance part="D6" gate="G$1" x="261.62" y="50.8"/>
-<instance part="D7" gate="G$1" x="259.08" y="40.64" rot="MR0"/>
+<instance part="D6" gate="G$1" x="259.08" y="50.8" rot="MR0"/>
+<instance part="D7" gate="G$1" x="261.62" y="40.64"/>
 <instance part="R30" gate="G$1" x="274.32" y="45.72"/>
 <instance part="D8" gate="G$1" x="292.1" y="40.64" rot="R90"/>
@@
 <instance part="R9" gate="G$1" x="81.28" y="-40.64" rot="R90"/>
 <instance part="GND18" gate="GND" x="81.28" y="-50.8"/>
-<instance part="C8" gate="1" x="86.36" y="-33.02"/>
+<instance part="C8" gate="1" x="88.9" y="-33.02" rot="MR0"/>
 <instance part="R14" gate="G$1" x="101.6" y="-40.64" rot="R90"/>
 <instance part="VB10" gate="G$1" x="101.6" y="-50.8" rot="R180"/>
@@
 <wire x1="251.46" y1="45.72" x2="254" y2="45.72" width="0.1524" layer="91"/>
 <wire x1="254" y1="45.72" x2="254" y2="50.8" width="0.1524" layer="91"/>
-<pinref part="D6" gate="G$1" pin="A"/>
+<pinref part="D6" gate="G$1" pin="C"/>
 <wire x1="254" y1="50.8" x2="256.54" y2="50.8" width="0.1524" layer="91"/>
-<wire x1="254" y1="45.72" x2="254" y2="40.64" width="0.1524" layer="91"/>
-<pinref part="D7" gate="G$1" pin="C"/>
-<wire x1="254" y1="40.64" x2="256.54" y2="40.64" width="0.1524" layer="91"/>
+<pinref part="D7" gate="G$1" pin="A"/>
+<wire x1="256.54" y1="40.64" x2="254" y2="40.64" width="0.1524" layer="91"/>
+<wire x1="254" y1="40.64" x2="254" y2="45.72" width="0.1524" layer="91"/>
 <junction x="254" y="45.72"/>
-</segment>
-</net>
-<net name="N$35" class="0">
-<segment>
-<pinref part="D6" gate="G$1" pin="C"/>
-<wire x1="264.16" y1="50.8" x2="266.7" y2="50.8" width="0.1524" layer="91"/>
-<wire x1="266.7" y1="50.8" x2="266.7" y2="45.72" width="0.1524" layer="91"/>
-<pinref part="D7" gate="G$1" pin="A"/>
-<wire x1="266.7" y1="45.72" x2="266.7" y2="40.64" width="0.1524" layer="91"/>
-<wire x1="266.7" y1="40.64" x2="264.16" y2="40.64" width="0.1524" layer="91"/>
-<pinref part="R30" gate="G$1" pin="1"/>
-<wire x1="266.7" y1="45.72" x2="269.24" y2="45.72" width="0.1524" layer="91"/>
-<junction x="266.7" y="45.72"/>
 </segment>
 </net>
@@
 <pinref part="R9" gate="G$1" pin="2"/>
 <wire x1="81.28" y1="-30.48" x2="81.28" y2="-33.02" width="0.1524" layer="91"/>
-<pinref part="C8" gate="1" pin="+"/>
+<pinref part="C8" gate="1" pin="-"/>
 <wire x1="81.28" y1="-33.02" x2="81.28" y2="-35.56" width="0.1524" layer="91"/>
 <wire x1="81.28" y1="-33.02" x2="83.82" y2="-33.02" width="0.1524" layer="91"/>
@@
 <net name="N$64" class="0">
 <segment>
-<pinref part="C8" gate="1" pin="-"/>
 <pinref part="Q5" gate="G$1" pin="D"/>
-<wire x1="91.44" y1="-33.02" x2="101.6" y2="-33.02" width="0.1524" layer="91"/>
 <pinref part="R14" gate="G$1" pin="2"/>
 <wire x1="101.6" y1="-33.02" x2="104.14" y2="-33.02" width="0.1524" layer="91"/>
 <wire x1="101.6" y1="-33.02" x2="101.6" y2="-35.56" width="0.1524" layer="91"/>
+<pinref part="C8" gate="1" pin="+"/>
+<wire x1="91.44" y1="-33.02" x2="101.6" y2="-33.02" width="0.1524" layer="91"/>
 <junction x="101.6" y="-33.02"/>
 </segment>
@@
 </segment>
 </net>
+<net name="N$1" class="0">
+<segment>
+<pinref part="R30" gate="G$1" pin="1"/>
+<wire x1="266.7" y1="45.72" x2="269.24" y2="45.72" width="0.1524" layer="91"/>
+<pinref part="D6" gate="G$1" pin="A"/>
+<wire x1="264.16" y1="50.8" x2="266.7" y2="50.8" width="0.1524" layer="91"/>
+<wire x1="266.7" y1="50.8" x2="266.7" y2="45.72" width="0.1524" layer="91"/>
+<pinref part="D7" gate="G$1" pin="C"/>
+<wire x1="264.16" y1="40.64" x2="266.7" y2="40.64" width="0.1524" layer="91"/>
+<wire x1="266.7" y1="40.64" x2="266.7" y2="45.72" width="0.1524" layer="91"/>
+<junction x="266.7" y="45.72"/>
+</segment>
+</net>

Commit message: 20180529
Other:
- moved on the sheet: C17, C18, C19, C2, C20, C21, C23, C24, C25, C8, D10, D13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
