File: #Misc/Boss HM-3/hm3.sch (EAGLE design)
At the start: 118 parts, among them IC1 M5218AL, IC2 M5218AL, Q1 2SK184GR, Q10 2SC2458QR, Q11 2SC2458QR, Q12 2SC3378GR, Q2 2SK118Y, Q3 2SK118Y, Q4 2SK118Y, Q5 2SC2458QR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

Commit message: 20180529
Parts:
- C14: value 47n -> 10n
- C15: value 1u -> 10u
- C27: value 220p -> 10n
- C29: value 47n -> 39n
- C30: value 47n -> 8.2n
- C31: value 47n -> 22n
- C32: value 47n -> 1.2n
- C33: value 1u -> 1.5u
- C34: value 47n -> 68n
- C39: value 56k -> 100R
- D9: value Q5688Q -> SS688Q
- Q10, Q11, Q9: value 2SC2458QR -> 2SC3378GR
- R40: value 56k -> 1M
- R41, R46, R49: value 3.3k -> 10k
- R42: value 3.3k -> 1k
- R43, R45, R48: value 3.3k -> 100k
- R44, R47: value 3.3k -> 330R
Connections:
- net N$47: now also C16.-; no longer C16.+
- net N$48: now also C16.+; no longer C16.-
- net N$49: now also C17.-; no longer C17.+
- net N$51: now also C35.-; no longer C35.+
- net N$52: now also C35.+; no longer C35.-
- net N$57: now also C17.+; no longer C17.-
