File: #Misc/Boss SD-1/sd1.sch (EAGLE design)
At the start: 74 parts, among them Q1 2SK30ATM-Y, Q2 2N5457, Q3 2SC945-P, Q4 2SC945-P, Q5 2SC732TM-GR, Q6 2SC732TM-GR

Commit message: 20171111
Parts:
- R30: value 56k -> 3.9k
Changed lines of the file:
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@@
 <setting verticaltext="up"/>
 </settings>
-<grid distance="0.1" unitdist="inch" unit="inch" style="lines" multiple="1" display="yes" altdistance="0.01" altunitdist="inch" altunit="inch"/>
+<grid distance="0.1" unitdist="inch" unit="inch" style="lines" multiple="1" display="no" altdistance="0.01" altunitdist="inch" altunit="inch"/>
 <layers>
 <layer number="1" name="Top" color="4" fill="1" visible="no" active="no"/>
@@
 <part name="GND117" library="gm-supply" deviceset="GND" device=""/>
 <part name="C9" library="pedals-capacitors-film" deviceset="CER/FILM" device="BOX.1" value="47n"/>
-<part name="R30" library="pedals-resistors" deviceset="R_" device=".3B" value="56k"/>
+<part name="R30" library="pedals-resistors" deviceset="R_" device=".3B" value="3.9k"/>
 <part name="D2" library="pedals-diodes" deviceset="ZENER" device=".2" value="RD5.1EB-3"/>
 <part name="V1" library="gm-supply" deviceset="+9V" device=""/>

Commit message: 20180529
Connections:
- net +9V: now also IC_PWR.V+
- net GND: now also IC_PWR.V-
Other:
- moved on the sheet: C6, R9, VR1, VR3
Changed lines of the file:
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@@
 <?xml version="1.0" encoding="utf-8"?>
 <!DOCTYPE eagle SYSTEM "eagle.dtd">
-<eagle version="8.2.0">
+<eagle version="8.5.1">
 <drawing>
 <settings>
 <setting alwaysvectorfont="no"/>
+<setting keepoldvectorfont="yes"/>
 <setting verticaltext="up"/>
 </settings>
@@
 <part name="V1" library="gm-supply" deviceset="+9V" device=""/>
 <part name="LED" library="pedals-diodes" deviceset="LED" device="" value="SLP1358"/>
+<part name="V2" library="gm-supply" deviceset="+9V" device=""/>
+<part name="GND1" library="gm-supply" deviceset="GND" device=""/>
 </parts>
 <sheets>
@@
 <text x="20.574" y="45.974" size="1.778" layer="95">7</text>
 <text x="20.574" y="43.434" size="1.778" layer="95">17</text>
-<circle x="86.36" y="78.74" radius="0.381" width="0.1524" layer="95"/>
-<circle x="109.22" y="78.74" radius="0.381" width="0.1524" layer="95"/>
-<text x="109.474" y="78.994" size="1.778" layer="95">4</text>
-<text x="86.106" y="78.994" size="1.778" layer="95" align="bottom-right">2</text>
-<circle x="124.46" y="78.74" radius="0.381" width="0.1524" layer="95"/>
-<circle x="144.78" y="78.74" radius="0.381" width="0.1524" layer="95"/>
-<text x="123.952" y="78.994" size="1.778" layer="95" align="bottom-right">5</text>
-<text x="145.288" y="78.994" size="1.778" layer="95">8</text>
+<circle x="86.36" y="81.28" radius="0.381" width="0.1524" layer="95"/>
+<circle x="109.22" y="81.28" radius="0.381" width="0.1524" layer="95"/>
+<text x="109.474" y="81.534" size="1.778" layer="95">4</text>
+<text x="86.106" y="81.534" size="1.778" layer="95" align="bottom-right">2</text>
+<circle x="124.46" y="81.28" radius="0.381" width="0.1524" layer="95"/>
+<circle x="144.78" y="81.28" radius="0.381" width="0.1524" layer="95"/>
+<text x="123.952" y="81.534" size="1.778" layer="95" align="bottom-right">5</text>
+<text x="145.288" y="81.534" size="1.778" layer="95">8</text>
 <circle x="190.5" y="43.18" radius="0.381" width="0.1524" layer="95"/>
 <circle x="190.5" y="27.94" radius="0.381" width="0.1524" layer="95"/>
 <text x="190.754" y="43.434" size="1.778" layer="95">9</text>
 <text x="190.246" y="28.194" size="1.778" layer="95" align="bottom-right">1</text>
-<circle x="134.62" y="78.74" radius="0.381" width="0.1524" layer="95"/>
-<text x="134.112" y="78.994" size="1.778" layer="95" align="bottom-right">11</text>
+<circle x="134.62" y="81.28" radius="0.381" width="0.1524" layer="95"/>
+<text x="134.112" y="81.534" size="1.778" layer="95" align="bottom-right">11</text>
 <circle x="195.58" y="35.56" radius="0.381" width="0.1524" layer="95"/>
 <text x="195.834" y="35.814" size="1.778" layer="95">10</text>
@@
 <text x="259.334" y="-50.546" size="1.778" layer="95">18</text>
 <text x="259.334" y="-37.846" size="1.778" layer="95">15</text>
-<text x="93.98" y="91.44" size="1.778" layer="95">DRIVE</text>
-<text x="132.08" y="91.44" size="1.778" layer="95">TONE</text>
+<text x="93.98" y="93.98" size="1.778" layer="95">DRIVE</text>
+<text x="132.08" y="93.98" size="1.778" layer="95">TONE</text>
 <text x="187.96" y="50.8" size="1.778" layer="95">LEVEL</text>
 </plain>
@@
 <instance part="D4" gate="G$1" x="99.06" y="63.5"/>
 <instance part="R5" gate="G$1" x="86.36" y="71.12" rot="R90"/>
-<instance part="VR1" gate="G$1" x="97.79" y="83.82" rot="MR90"/>
-<instance part="R9" gate="G$1" x="154.94" y="58.42"/>
-<instance part="C6" gate="G$1" x="153.67" y="68.58"/>
-<instance part="VR3" gate="G$1" x="134.62" y="83.82" rot="R270"/>
+<instance part="VR1" gate="G$1" x="97.79" y="86.36" rot="MR90"/>
+<instance part="R9" gate="G$1" x="154.94" y="66.04"/>
+<instance part="C6" gate="G$1" x="153.67" y="76.2"/>
+<instance part="VR3" gate="G$1" x="134.62" y="86.36" rot="R270"/>
 <instance part="C5" gate="G$1" x="134.62" y="72.39" rot="R90"/>
 <instance part="R8" gate="G$1" x="134.62" y="60.96" rot="R90"/>
@@
 <instance part="V1" gate="+9V" x="254" y="-10.16"/>
 <instance part="LED" gate="G$1" x="264.16" y="-45.72" rot="R90"/>
+<instance part="IC" gate="_PWR" x="154.94" y="45.72"/>
+<instance part="V2" gate="+9V" x="154.94" y="55.88"/>
+<instance part="GND1" gate="GND" x="154.94" y="35.56"/>
 </instances>
 <busses>
@@
 <wire x1="276.86" y1="22.86" x2="279.4" y2="22.86" width="0.1524" layer="91"/>
 <pinref part="GND117" gate="GND" pin="GND"/>
+</segment>
+<segment>
+<pinref part="IC" gate="_PWR" pin="V-"/>
+<pinref part="GND1" gate="GND" pin="GND"/>
 </segment>
 </net>
@@
 <pinref part="IC" gate="_B" pin="OUT"/>
 <wire x1="109.22" y1="43.18" x2="106.68" y2="43.18" width="0.1524" layer="91"/>
-<wire x1="109.22" y1="83.82" x2="109.22" y2="63.5" width="0.1524" layer="91"/>
+<wire x1="109.22" y1="86.36" x2="109.22" y2="63.5" width="0.1524" layer="91"/>
 <pinref part="D4" gate="G$1" pin="C"/>
 <wire x1="109.22" y1="63.5" x2="109.22" y2="55.88" width="0.1524" layer="91"/>
 <wire x1="101.6" y1="63.5" x2="109.22" y2="63.5" width="0.1524" layer="91"/>
 <pinref part="VR1" gate="G$1" pin="3"/>
-<wire x1="109.22" y1="83.82" x2="104.14" y2="83.82" width="0.1524" layer="91"/>
+<wire x1="109.22" y1="86.36" x2="104.14" y2="86.36" width="0.1524" layer="91"/>
 <pinref part="VR1" gate="G$1" pin="2"/>
-<wire x1="97.79" y1="88.9" x2="104.14" y2="88.9" width="0.1524" layer="91"/>
-<wire x1="104.14" y1="88.9" x2="104.14" y2="83.82" width="0.1524" layer="91"/>
-<junction x="104.14" y="83.82"/>
+<wire x1="97.79" y1="91.44" x2="104.14" y2="91.44" width="0.1524" layer="91"/>
+<wire x1="104.14" y1="91.44" x2="104.14" y2="86.36" width="0.1524" layer="91"/>
+<junction x="104.14" y="86.36"/>
 <junction x="109.22" y="63.5"/>
 <junction x="109.22" y="55.88"/>
@@
 <segment>
 <pinref part="R5" gate="G$1" pin="2"/>
-<wire x1="86.36" y1="76.2" x2="86.36" y2="83.82" width="0.1524" layer="91"/>
+<wire x1="86.36" y1="76.2" x2="86.36" y2="86.36" width="0.1524" layer="91"/>
 <pinref part="VR1" gate="G$1" pin="1"/>
-<wire x1="86.36" y1="83.82" x2="91.44" y2="83.82" width="0.1524" layer="91"/>
+<wire x1="86.36" y1="86.36" x2="91.44" y2="86.36" width="0.1524" layer="91"/>
 </segment>
 </net>
@@
 <pinref part="IC" gate="_A" pin="+IN"/>
 <wire x1="124.46" y1="43.18" x2="147.32" y2="43.18" width="0.1524" layer="91"/>
-<wire x1="124.46" y1="43.18" x2="124.46" y2="83.82" width="0.1524" layer="91"/>
+<wire x1="124.46" y1="43.18" x2="124.46" y2="86.36" width="0.1524" layer="91"/>
 <pinref part="VR3" gate="G$1" pin="1"/>
-<wire x1="124.46" y1="83.82" x2="128.27" y2="83.82" width="0.1524" layer="91"/>
+<wire x1="124.46" y1="86.36" x2="128.27" y2="86.36" width="0.1524" layer="91"/>
 <junction x="124.46" y="43.18"/>
 </segment>
@@
 <pinref part="IC" gate="_A" pin="-IN"/>
 <wire x1="147.32" y1="48.26" x2="144.78" y2="48.26" width="0.1524" layer="91"/>
-<wire x1="144.78" y1="48.26" x2="144.78" y2="58.42" width="0.1524" layer="91"/>
+<wire x1="144.78" y1="48.26" x2="144.78" y2="66.04" width="0.1524" layer="91"/>
 <pinref part="R9" gate="G$1" pin="1"/>
-<wire x1="144.78" y1="58.42" x2="149.86" y2="58.42" width="0.1524" layer="91"/>
-<wire x1="144.78" y1="58.42" x2="144.78" y2="68.58" width="0.1524" layer="91"/>
+<wire x1="144.78" y1="66.04" x2="149.86" y2="66.04" width="0.1524" layer="91"/>
+<wire x1="144.78" y1="66.04" x2="144.78" y2="76.2" width="0.1524" layer="91"/>
 <pinref part="C6" gate="G$1" pin="2"/>
-<wire x1="144.78" y1="68.58" x2="149.86" y2="68.58" width="0.1524" layer="91"/>
-<wire x1="144.78" y1="68.58" x2="144.78" y2="83.82" width="0.1524" layer="91"/>
+<wire x1="144.78" y1="76.2" x2="149.86" y2="76.2" width="0.1524" layer="91"/>
+<wire x1="144.78" y1="76.2" x2="144.78" y2="86.36" width="0.1524" layer="91"/>
 <pinref part="VR3" gate="G$1" pin="3"/>
-<wire x1="144.78" y1="83.82" x2="140.97" y2="83.82" width="0.1524" layer="91"/>
-<junction x="144.78" y="58.42"/>
-<junction x="144.78" y="68.58"/>
+<wire x1="144.78" y1="86.36" x2="140.97" y2="86.36" width="0.1524" layer="91"/>
+<junction x="144.78" y="66.04"/>
+<junction x="144.78" y="76.2"/>
 </segment>
 </net>
@@
 <segment>
 <pinref part="R9" gate="G$1" pin="2"/>
-<wire x1="160.02" y1="58.42" x2="165.1" y2="58.42" width="0.1524" layer="91"/>
-<wire x1="165.1" y1="58.42" x2="165.1" y2="45.72" width="0.1524" layer="91"/>
+<wire x1="160.02" y1="66.04" x2="165.1" y2="66.04" width="0.1524" layer="91"/>
+<wire x1="165.1" y1="66.04" x2="165.1" y2="45.72" width="0.1524" layer="91"/>
 <pinref part="IC" gate="_A" pin="OUT"/>
 <wire x1="165.1" y1="45.72" x2="162.56" y2="45.72" width="0.1524" layer="91"/>
 <pinref part="C6" gate="G$1" pin="1"/>
-<wire x1="157.48" y1="68.58" x2="165.1" y2="68.58" width="0.1524" layer="91"/>
-<wire x1="165.1" y1="68.58" x2="165.1" y2="58.42" width="0.1524" layer="91"/>
-<junction x="165.1" y="58.42"/>
+<wire x1="157.48" y1="76.2" x2="165.1" y2="76.2" width="0.1524" layer="91"/>
+<wire x1="165.1" y1="76.2" x2="165.1" y2="66.04" width="0.1524" layer="91"/>
+<junction x="165.1" y="66.04"/>
 <junction x="165.1" y="45.72"/>
 <pinref part="C7" gate="1" pin="+"/>
@@
 <pinref part="C5" gate="G$1" pin="1"/>
 <pinref part="VR3" gate="G$1" pin="2"/>
-<wire x1="134.62" y1="76.2" x2="134.62" y2="78.74" width="0.1524" layer="91"/>
+<wire x1="134.62" y1="76.2" x2="134.62" y2="81.28" width="0.1524" layer="91"/>
 </segment>
 </net>
@@
 <wire x1="254" y1="-15.24" x2="254" y2="-12.7" width="0.1524" layer="91"/>
 </segment>
-</net>
+<segment>
+<pinref part="IC" gate="_PWR" pin="V+"/>
+<pinref part="V2" gate="+9V" pin="+9V"/>
+</segment>
+</net>
