File: #Misc/Boss SD-2/sd2.sch (EAGLE design)
At the start: 105 parts, among them IC4 uPC4558C, IC5 HA1457, Q1 2SC732TM-GR, Q2 2SC945-P, Q3 2SC945-P, Q4 2SK30A, Q5 2SK30A, SW1 MOMENTARY

Commit message: 20180207
Parts:
- removed AC_ADAPTOR: (no value), pedals-jacks:DC_KOBICONN
- removed BATTERY: BATTERY, pedals-jacks:BATTERY
- removed C1: 47n, pedals-capacitors-film:CER/FILMBOX.1
- removed D2: 1S2473, pedals-diodes:DO35.2
- removed IC5: HA1457, pedals-integrated circuits:HA1457
- removed LED: LED, pedals-diodes:LED
- removed R1: 470R, pedals-resistors:R_.3B
- removed R17: 330R, pedals-resistors:R_.3B
- removed R23: 33k, pedals-resistors:R_.3B
- removed VR1, VR2, VR3, VR4, VR5, VR6, VR7, VR8: 10kG, pedals-potentiometers:POTS16MM
- added 1101: BATTERY, pedals-jacks:BATTERY
- added C32, C37: 22n, pedals-capacitors-film:CER/FILMBOX.1
- added C33: 27n, pedals-capacitors-film:CER/FILMBOX.1
- added C34, C38, C48: 47n, pedals-capacitors-film:CER/FILMBOX.1
- added C35, C46: 1u, pedals-capacitors-elec:0400
- added C36, C47: 2.7n, pedals-capacitors-film:CER/FILMBOX.1
- added C39: 15n, pedals-capacitors-film:CER/FILMBOX.1
- added C40: 10u, pedals-capacitors-elec:0400
- added C41: 470p, pedals-capacitors-film:CER/FILMBOX.1
- added C42: 220p, pedals-capacitors-film:CER/FILMBOX.1
- added C43: 100n, pedals-capacitors-film:CER/FILMBOX.1
- added C44, C45: 100u, pedals-capacitors-elec:0400
- added D10, D11, D13, D16, D8, D9: 1SS133, pedals-diodes:DO35.2
- added D12: S5500G, pedals-diodes:DO35.2
- added D14, D15, D6, GREEN, RED: LED, pedals-diodes:LED
- added JK1: (no value), pedals-jacks:DC_KOBICONN
- added Q10, Q12, Q7: 2SC3378GR, pedals-transistors:2N3904
- added Q11, Q13, Q15, Q8, Q9: 2SK118Y, pedals-transistors:2N5457
- added Q14: 2SK184GR, pedals-transistors:2N5457
- added Q6: RN2211, pedals-transistors:2N3904
- added R46, R47, R61, R90: 4.7k, pedals-resistors:R_.3B
- added R48, R65: 220k, pedals-resistors:R_.3B
- added R49, R56: 22k, pedals-resistors:R_.3B
- added R50, R60: 47k, pedals-resistors:R_.3B
- added R51, R63: 1M, pedals-resistors:R_.3B
- added R52, R53: 1k, pedals-resistors:R_.3B
- added R54, R62: 10k, pedals-resistors:R_.3B
- added R55: 12k, pedals-resistors:R_.3B
- added R57, R58, R59: 100k, pedals-resistors:R_.3B
- added R64: 2.2k, pedals-resistors:R_.3B
- added REMOTE: (no value), pedals-jacks:MONO
- added SW2: MOMENTARY, pedals-switches:MOMENTARY
- added VR1A, VR1B: 250kA, pedals-potentiometers:POTS16MM
- added VR2A, VR2B: 10kB, pedals-potentiometers:POTS16MM
- added VR3A, VR3B: 100kA, pedals-potentiometers:POTS16MM
- C10: value 1.5u -> 82n; device pedals-capacitors-elec:0400 -> pedals-capacitors-film:CER/FILMBOX.1
- C11: value 1u -> 470p; device pedals-capacitors-elec:0400 -> pedals-capacitors-film:CER/FILMBOX.1
- C12: value 10n -> 22n
- C13: value 56n -> 47n
- C14: value 15n -> 100p
- C15: value 39n -> 22p
- C16: value 10u -> 27n; device pedals-capacitors-elec:0400 -> pedals-capacitors-film:CER/FILMBOX.1
- C17: value 100u -> 8.2n; device pedals-capacitors-elec:0400 -> pedals-capacitors-film:CER/FILMBOX.1
- C18: value 47u -> 68n; device pedals-capacitors-elec:0400 -> pedals-capacitors-film:CER/FILMBOX.1
- C19: value 1u -> 68p; device pedals-capacitors-elec:0400 -> pedals-capacitors-film:CER/FILMBOX.1
- C2: value 39n -> 10n
- C20: value 47n -> 180p
- C21: value 470p -> 1u; device pedals-capacitors-film:CER/FILMBOX.1 -> pedals-capacitors-elec:0400
- C23: value 15n -> 47n
- C24: value 15n -> 39n
- C26: value 47n -> 1u; device pedals-capacitors-film:CER/FILMBOX.1 -> pedals-capacitors-elec:0400
- C27: value 15n -> 1u; device pedals-capacitors-film:CER/FILMBOX.1 -> pedals-capacitors-elec:0400
- C28: value 470p -> 4.7u; device pedals-capacitors-film:CER/FILMBOX.1 -> pedals-capacitors-elec:0400
- C29: value 470p -> 10u; device pedals-capacitors-film:CER/FILMBOX.1 -> pedals-capacitors-elec:0400
- C3: value 2.2n -> 220p
- C30: value 220p -> 10u; device pedals-capacitors-film:CER/FILMBOX.1 -> pedals-capacitors-elec:0400
- C31: value 220p -> 22n
- C4: value 1u -> 100p; device pedals-capacitors-elec:0400 -> pedals-capacitors-film:CER/FILMBOX.1
- C5: value 150n -> 47n; device pedals-capacitors-elec:0400 -> pedals-capacitors-film:CER/FILMBOX.1
- C6: value 8.2n -> 220p
- C7: value 330n -> 470p; device pedals-capacitors-elec:0400 -> pedals-capacitors-film:CER/FILMBOX.1
- C8: value 33n -> 47n
- C9: value 680n -> 47n; device pedals-capacitors-elec:0400 -> pedals-capacitors-film:CER/FILMBOX.1
- D1: value 1S2473 -> RD5.6EB3; device pedals-diodes:DO35.2 -> pedals-diodes:ZENER.2
- D3: value 1S2473 -> 1SS133
- D4: value (none) -> LED; device pedals-diodes:ZENER.2 -> pedals-diodes:LED
- D5: value 10E2 -> 1SS133
- IC1: value (none) -> 4011; device pedals-integrated circuits:DUALTH -> pedals-40xx-2:4011N
- IC2: value (none) -> M5218AL
- IC4: value uPC4558C -> M5218AL
- Q1: value 2SC732TM-GR -> 2SC945
- Q2: value 2SC945-P -> 2SC945
- Q3: value 2SC945-P -> RN2211; device pedals-transistors:2SC828A -> pedals-transistors:2N3904
- Q4, Q5: value 2SK30A -> RN2211; device pedals-transistors:2N5457 -> pedals-transistors:2N3906
- R10: value 100k -> 1k
- R11: value 100R -> 56k
- R12: value 100k -> 1M
- R13, R35, R43: value 1M -> 220k
- R14: value 1k -> 100k
- R15: value 10k -> 2.2k
- R16: value 100k -> 10k
- R18: value 100k -> 56k
- R19, R4: value 330R -> 56k
- R2: value 2.2k -> 100R
- R20: value 33k -> 1M
- R21: value 82k -> 220k
- R22, R6, R8: value 330R -> 1M
- R24: value 3.3k -> 100k
- R25: value 3.3k -> 2.2k
- R26: value 10k -> 47k
- R27: value 10k -> 220k
- R28: value 470k -> 4.7k
- R29: value 470k -> 1M
- R3: value 820R -> 100k
- R30: value 10k -> 100k
- R31: value 470k -> 10k
- R32: value 1M -> 560R
- R33: value 4.7k -> 220k
- R34: value 1M -> 47k
- R36: value 470R -> 10k
- R37: value 56k -> 680R
- R38: value 56k -> 15k
- R39: value 56k -> 33k
- R40: value 56k -> 1k
- R41: value 100k -> 470k
- R42: value 100k -> 220k
- R44: value 1M -> 4.7k
- R5: value 82k -> 100k
- R9: value 82k -> 470R
- SW1: value MOMENTARY -> (none); device pedals-switches:MOMENTARY -> pedals-switches:2P4T
Connections:
- new net N$68: C27.+, Q13.D, R48.1
- new net N$69: D9.A, Q13.G
- new net N$70: C19.2, IC3_B.-IN, R28.1, VR1A.1
- new net N$71: Q3.C, R14.2, R8.1
- new net N$72: Q5.C, R10.1
- new net N$73: Q4.C, R9.1
- new net N$74: GREEN.A, R9.2
- new net N$75: R10.2, RED.A
- new net N$76: D1.A, GREEN.C, RED.C
- new net N$77: Q6.C, R22.1, R24.2
- new net N$78: C8.1, D13.C, D9.C, R22.2
- new net N$79: C5.1, D3.C, D8.C, R8.2
- new net N$80: IC1B.O, Q3.B, Q5.B
- new net N$81: Q13.S, Q9.S, R45.1
- new net N$82: IC1A.I0, IC1A.I1, IC1B.I1, IC1C.I1, R21.2, SW1A.A
- new net N$83: IC1B.I0, IC1D.O
- new net N$84: IC1C.I0, IC1D.I0, IC1D.I1, SW1B.A
- new net N$85: R2.2, SW2.P
- new net N$86: C22.2, Q11.S
- new net N$87: IC1A.O, R6.2
- new net N$88: C23.1, D5.C, R6.1
- new net N$89: REMOTE.TIP, SW1B.3
- new net N$90: C22.1, Q10.B, R41.1
- new net N$91: C4.1, R5.2, SW1A.2, SW1B.1
- new net N$92: C21.+, Q10.E, R31.1
- new net N$93: C21.-, R30.1, R40.2
- new net N$94: OUTPUT.TIP, R40.1
- net +9V: now also C44.+, D12.C, JK1.S, Q10.C, Q12.C, Q14.D, Q4.E, Q5.E, Q7.C, R11.2, R12.2, R13.1, R14.1, R19.2, R21.1, R24.1, R61.1; no longer AC_ADAPTOR.S, C17.+, D4.C, D5.C, IC1_PWR.V+, IC5.V+, Q1.C, R13.2, R20.1, R38.2, R39.2
- net GND: now also C10.2, C2.2, C31.2, C32.2, C33.2, C39.2, C4.2, C44.-, C45.-, C5.2, C8.2, D1.C, D12.A, D14.C, D15.A, Q1.E, Q6.E, R16.2, R18.1, R30.2, R31.2, R37.2, R4.1, R44.2, R46.2, R47.2, R49.2, R54.2, R55.2, REMOTE.SLEEVE, SW1B.2, SW2.S, VR3A.1, VR3B.1; no longer C12.2, C16.-, C17.-, C18.-, C20.2, D5.A, IC1_PWR.V-, IC5.V-, R12.2, R15.2, R23.1, R37.1, R40.1, SW1.S
- net N$1: now also INPUT.T, R62.2; no longer C21.2, IC5.ON1
- net N$10: now also C14.2, C16.1, IC2_B.-IN, R25.2; no longer IC4_B.-IN, R26.1, VR8.1
- net N$11: now also C14.1, C9.2, IC2_B.OUT, R25.1; no longer IC4_B.OUT, R24.1, R26.2
- net N$12: now also Q7.E, R15.2, R16.1; no longer IC4_B.+IN, R27.2, VR8.3
- net N$13: now also C9.1, IC3_B.+IN, R27.1; no longer IC4_A.+IN, R24.2, VR1.3, VR2.3, VR3.3, VR4.3, VR5.3, VR6.3, VR7.3
- net N$14: now also C17.2, Q7.B, R26.2; no longer IC4_A.-IN, R25.1, VR1.1, VR2.1, VR3.1, VR4.1, VR5.1, VR6.1, VR7.1
- net N$15: now also C10.1, R28.2; no longer C19.-, IC4_A.OUT, R25.2
- net N$16: now also C16.2, C17.1, R15.1; no longer R2.2, VR8.2
- net N$17: now also IC1C.O, Q4.B, Q6.B; no longer C16.+, R2.1
- net N$18: now also C18.2, C19.1, VR1A.2, VR1A.3; no longer IC3_B.-IN, R17.1
- net N$19: now also C18.1, R38.2; no longer C13.2, IC3_B.+IN, R16.2
- net N$2: now also 1101.P$2, JK1.T; no longer BATTERY.P$2, D1.A
- net N$20: now also C20.2, IC3_A.-IN, R29.2, R38.1; no longer C10.+, C13.1, R17.2
- net N$21: now also C20.1, C30.+, IC3_A.OUT, R29.1; no longer C10.-, VR1.2
- net N$22: now also C30.-, R52.2; no longer C19.+, Q4.D, R32.2
- net N$23: now also C37.2, D14.A, D15.C, R52.1, R53.2; no longer C25.+, Q5.D, R43.2
- net N$24: now also C37.1, C40.-, R53.1, R54.1; no longer IC3_A.-IN, IC3_A.OUT, R8.1
- net N$25: now also C40.+, IC4_A.+IN, R57.1; no longer C8.2, IC3_A.+IN, R9.2
- net N$26: now also C41.2, D10.A, D11.C, IC4_A.-IN, R59.2, R60.1; no longer C8.1, C9.+, R8.2
- net N$27: now also 1101.P$1, JK1.R; no longer AC_ADAPTOR.R, BATTERY.P$1
- net N$28: now also C41.1, D10.C, D16.A, IC4_A.OUT, R59.1, R64.2; no longer AC_ADAPTOR.T, R1.1
- net N$29: now also C7.2, Q1.C, R11.1, R3.1; no longer C28.2, LED.C, Q3.C, R39.1, R42.1, R45.2
- net N$3: now also C34.2, R62.1; no longer C21.1, IC5.ON2
- net N$30: now also D11.A, D16.C; no longer D1.C, R1.2
- net N$31: now also C11.1, R19.1, R5.1, R7.2; no longer C29.1, R38.1, R41.2, R44.1
- net N$32: now also C11.2, C6.1, Q1.B, R18.2, R7.1; no longer C29.2, C30.1, Q3.B, R40.2, R41.1
- net N$33: now also R60.2; no longer C9.-, VR2.2
- net N$34: now also C3.1, C7.1, R3.2, R4.2; no longer C28.1, C31.1, R37.2, R42.2
- net N$35: now also C2.1, C3.2, C6.2, R12.1, R2.1; no longer D3.A, Q5.G
- net N$36: now also C39.1, R56.2, R64.1; no longer C12.1, C30.2, C31.2, R11.1, R13.1
- net N$37: now also C29.-, C38.1, R56.1; no longer D2.A, Q4.G
- net N$38: now also C38.2, R55.1; no longer IC1_B.-IN, IC1_B.OUT, R19.1
- net N$39: now also C29.+, R39.2; no longer C14.2, IC1_B.+IN, R18.2
- net N$4: now also C34.1, Q14.G, R63.1; no longer INPUT.T, R30.1
- net N$40: now also C42.2, IC4_B.-IN, R39.1, R58.2; no longer C14.1, C7.+, R19.2
- net N$41: now also C43.1, VR2A.3; no longer C7.-, VR3.2
- net N$42: now also C42.1, C43.2, IC4_B.OUT, R58.1; no longer Q4.S, Q5.S, R33.1, R35.1
- net N$43: now also C33.1, VR2A.1; no longer C26.2, C27.1, R33.2
- net N$44: now also VR2A.2, VR3A.3; no longer IC1_A.-IN, IC1_A.OUT, R6.1
- net N$45: now also R90.2, VR3A.2; no longer C6.2, IC1_A.+IN, R7.2
- net N$46: now also C25.-, R90.1; no longer C5.+, C6.1, R6.2
- net N$47: now also C25.+, Q11.D, R43.1; no longer C5.-, VR4.2
- net N$48: now also D8.A, Q11.G; no longer C27.2, R36.1
- net N$49: now also C35.+, Q9.D, R42.1; no longer C26.1, Q1.B, R34.1
- net N$5: now also C26.+, C46.+, Q12.B, Q14.S, R46.1; no longer C22.2, R30.2
- net N$50: now also D5.A, Q9.G; no longer IC2_B.-IN, IC2_B.OUT, R22.1
- net N$51: now also C35.-, Q12.E, R47.1; no longer C15.2, IC2_B.+IN, R21.2
- net N$52: now also C46.-, Q15.D, R65.1; no longer C15.1, C4.+, R22.2
- net N$53: now also C36.2, Q15.S, R50.1; no longer C4.-, VR5.2
- net N$54: now also D13.A, Q15.G; no longer Q1.E, R14.1, R15.1
- net N$55: now also C36.1, C47.1, C48.2; no longer C11.+, R14.2
- net N$56: now also C47.2, R49.1; no longer IC2_A.-IN, IC2_A.OUT, R4.1
- net N$57: now also C48.1, R51.1; no longer C3.2, R5.2
- net N$58: now also C15.2, C28.+, D4.A, D6.C, IC2_A.-IN, R36.2; no longer C2.2, C3.1, R4.2
- net N$59: now also R36.1, VR1B.1; no longer C2.1, VR6.2
- net N$6: now also C26.-, Q8.D, R33.1; no longer C22.1, IC5.+IN, R29.2
- net N$60: now also C15.1, D4.C, D6.A, IC2_A.OUT, R32.2, VR1B.2, VR1B.3; no longer C1.2, R3.2
- net N$61: now also C24.1, R20.2, R32.1; no longer C1.1, VR7.2
- net N$62: now also C28.-, R37.1; no longer C11.-, OUTPUT.TIP, R12.1
- net N$63: now also C12.2, R20.1; no longer C23.1, D3.C, R45.1
- net N$64: now also C12.1, VR2B.3; no longer C24.1, D2.C, R44.2
- net N$65: now also C32.1, VR2B.1; no longer R11.2, SW1.P
- net N$66: now also VR2B.2, VR3B.3; no longer LED.A, R10.1
- net N$67: now also C27.-, VR3B.2; no longer D4.A, R10.2
- net N$7: now also D3.A, Q8.G; no longer IC5.-IN, R28.2, R31.1
- net N$8: now also C13.2, Q8.S, R34.1; no longer C25.-, IC5.OUT, R27.1, R31.2
- net N$9: now also C13.1, IC2_B.+IN, R35.1; no longer C20.1, R28.1
- net VB: now also C45.+, IC3_A.+IN, IC4_B.+IN, R26.1, R27.2, R33.2, R41.2, R42.2, R43.2, R44.1, R45.2, R48.2, R50.2, R51.2, R57.2, R61.2, R63.2, R65.2; no longer C18.+, R16.1, R18.1, R20.2, R21.1, R23.2, R29.1, R3.1, R32.1, R36.2, R43.1, R5.1, R7.1, R9.1
Other:
- note added: "1"
- note added: "12"
- note added: "14"
- note added: "2"
- note added: "3"
- note added: "4"
- note added: "5"
- note added: "6"
- note added: "7"
- note added: "8"
- note added: "GAIN-C"
- note added: "GAIN-L"
- note added: "LEVEL-C"
- note added: "LEVEL-L"
- note added: "TONE-C"
- note added: "TONE-L"
- moved on the sheet: C12, C13, C14, C15, C2, C20, C22, C23, C24, C25, C3, C31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

Commit message: 20180529
Parts:
- added D7: LED, pedals-diodes:LED
- D6: value LED -> 1SS133; device pedals-diodes:LED -> pedals-diodes:DO35.2
- R20: value 1M -> 2.2k
Connections:
- new net N$95: D6.C, D7.A
- net N$58: now also D7.C; no longer D6.C
Other:
- note added: "MODE-SW"
- moved on the sheet: C13, C14, C16, D14, IC2_B, IC2_PWR, Q7, R15, R16, R25, R26, R34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
