File: #Misc/Boss TR-2/tr2_redraw.sch (EAGLE design)
At the start: 137 parts, among them IC1 uPC4558C, IC2 uPC4558, IC3 MN3207, IC4 MN3102, IC5 TL022CP, IC6 LM78L05, Q1 2SC732TM-GR, Q10 2SC945-P, Q11 2SC945-P, Q2 2SC732TM-GR, Q3 2SC732TM-GR, Q4 1SK30A-Y, Q5 2SA733-P, Q6 2SC945-P, Q7 2SC945-P, Q8 2N3906-, Q9 2SC945-P, SW101 MOMENTARY

Commit message: 20171220
Parts:
- removed C116, C38: 47n, pedals-capacitors-film:CER/FILMBOX.1
- removed C26, C33: 10n, pedals-capacitors-film:CER/FILMBOX.1
- removed C27, C28: 6.3u, pedals-capacitors-elec:0400
- removed C29, C40: 47u, pedals-capacitors-elec:0400
- removed C30: 47p, pedals-capacitors-film:CER/FILMBOX.1
- removed C31: 5p, pedals-capacitors-film:CER/FILMBOX.1
- removed C32: 22u, pedals-capacitors-elec:0400
- removed C34, C35: 470p, pedals-capacitors-film:CER/FILMBOX.1
- removed C36, C37: 220p, pedals-capacitors-film:CER/FILMBOX.1
- removed C39: 100u, pedals-capacitors-elec:0400
- removed D1: RD11EB-3, pedals-diodes:ZENER.2
- removed D7, D8, D9: 1S2473, pedals-diodes:DO35.2
- removed IC5: TL022CP, pedals-integrated circuits:DUALTH
- removed IC6: LM78L05, pedals-regulators:LM78L05
- removed LED: SLP1358, pedals-diodes:LED
- removed Q10, Q11, Q9: 2SC945-P, pedals-transistors:2SC828A
- removed Q8: 2N3906-, pedals-transistors:2N3906-
- removed R120: 1.5k, pedals-resistors:R_.3B
- removed R126: 39k, pedals-resistors:R_.3B
- removed R21: 10k, pedals-resistors:R_.3B
- removed R46: 330k, pedals-resistors:R_.3B
- removed R47, R51, R52: 4.7k, pedals-resistors:R_.3B
- removed R48: 220k, pedals-resistors:R_.3B
- removed R49, R50: 33k, pedals-resistors:R_.3B
- removed R53, R61, R62: 1M, pedals-resistors:R_.3B
- removed R54: 1k, pedals-resistors:R_.3B
- removed R55, R56, R59, R60: 56k, pedals-resistors:R_.3B
- removed R57, R58: 100k, pedals-resistors:R_.3B
- removed R63: 3.9k, pedals-resistors:R_.3B
- removed SW101: MOMENTARY, pedals-switches:MOMENTARY
- removed VR4: 50kC, pedals-potentiometers:POTS16MM
- removed VR5: 22kB, pedals-potentiometers:POTS16MM
- removed VR6: (no value), pedals-potentiometers:POTS16MM
- removed VR7: 470kB, pedals-potentiometers:POTS16MM
- added C7: 10p, pedals-capacitors-film:CER/FILMBOX.1
- added R10: 1M, pedals-resistors:R_.3B
- added R119: 12k, pedals-resistors:R_.3B
- added R39, R45: 100k, pedals-resistors:R_.3B
- added SW1: MOMENTARY, pedals-switches:MOMENTARY
- C1: value 47n -> 27n
- C10: value 33n -> 47u; device pedals-capacitors-film:CER/FILMBOX.1 -> pedals-capacitors-elec:0400
- C11, C2: value 1u -> 10u
- C12: value 1u -> 47n; device pedals-capacitors-elec:0400 -> pedals-capacitors-film:CER/FILMBOX.1
- C13: value 33n -> 47n
- C14: value 3.9n -> 10u; device pedals-capacitors-film:CER/FILMBOX.1 -> pedals-capacitors-elec:0400
- C15: value 8.2 -> 10n
- C16: value 330p -> 220p
- C17: value 220n -> 470p; device pedals-capacitors-elec:0400 -> pedals-capacitors-film:CER/FILMBOX.1
- C18: value 1n -> 10n
- C19: value 150p -> 47u; device pedals-capacitors-film:CER/FILMBOX.1 -> pedals-capacitors-elec:0400
- C20: value 220n -> 1u
- C21: value 47n -> 1u; device pedals-capacitors-film:CER/FILMBOX.1 -> pedals-capacitors-elec:0400
- C22: value 100p -> 220p
- C23: value 6.8n -> 470p
- C24: value 1u -> 47u
- C25: value 33u -> 47u
- C3: value 6.8n -> 1u; device pedals-capacitors-film:CER/FILMBOX.1 -> pedals-capacitors-elec:0400
- C4: value 100p -> 100n
- C5: value 220p -> 1u; device pedals-capacitors-film:CER/FILMBOX.1 -> pedals-capacitors-elec:0400
- C6: value 47n -> 10u; device pedals-capacitors-film:CER/FILMBOX.1 -> pedals-capacitors-elec:0400
- C8: value 12n -> 47n
- C9: value 150p -> 100u; device pedals-capacitors-film:CER/FILMBOX.1 -> pedals-capacitors-elec:0400
- D2: value RD5.1EB-3 -> 1SS133; device pedals-diodes:ZENER.2 -> pedals-diodes:DO35.2
- D3: value 1S2473 -> 1SS133
- D4: value 1S2473 -> 1N4004
- D5: value 1S2473 -> MTZ5.6B; device pedals-diodes:DO35.2 -> pedals-diodes:ZENER.2
- D6: value 1S2473 -> LN-28RP; device pedals-diodes:DO35.2 -> pedals-diodes:LED
- IC1: value uPC4558C -> M5207L01; device pedals-integrated circuits:DUALTH -> pedals-integrated circuits:M5207L01
- IC2: value uPC4558 -> M5218AL
- IC3: value MN3207 -> M5218AL; device pedals-integrated circuits:BL3208 -> pedals-integrated circuits:DUALTH
- IC4: value MN3102 -> M5218AL; device pedals-integrated circuits:CLOCK -> pedals-integrated circuits:DUALTH
- Q1, Q3: value 2SC732TM-GR -> 2SK118Y; device pedals-transistors:2SC828A -> pedals-transistors:2N3819TO-92S
- Q2: value 2SC732TM-GR -> 2SC2458GR
- Q4: value 1SK30A-Y -> 2SK184GR
- Q5: value 2SA733-P -> 2SC2458GR; device pedals-transistors:2N3906- -> pedals-transistors:2SC828A
- Q6: value 2SC945-P -> 2SA1048GR; device pedals-transistors:2SC828A -> pedals-transistors:2N3906-
- Q7: value 2SC945-P -> 2SC2458GR
- R11: value 4.7k -> 10k
- R12: value 47k -> 22k
- R15, R22, R7: value 10k -> 1M
- R17: value 100k -> 1.2k
- R18: value 56k -> 100
- R19: value 330k -> 10k
- R2, R44: value 470k -> 100k
- R23, R30, R40: value 10k -> 56k
- R24, R26, R6: value 47k -> 1M
- R25: value 22k -> 56k
- R27: value 1M -> 1.5k
- R28: value 47k -> 10k
- R29: value 27k -> 33k
- R3: value 10k -> 330k
- R31: value 47k -> 56k
- R32: value 470R -> 15k
- R34: value 33k -> 10k
- R35: value 33k -> 4.7k
- R36: value 180k -> 330k
- R37: value 220k -> 47k
- R38: value 100k -> 10k
- R4: value 47k -> 100k
- R41: value 10k -> 4.7k
- R42: value 68k -> 5.6k
- R43: value 150k -> 10k
- R8: value 220k -> 100k
- R9: value 82k -> 10k
- VR1: value 50kB -> 100kA
- VR2: value 50kB -> 100kB
- VR3: value 250kC -> 100kB
Connections:
- removed net IN: R1.1
- removed net N$37: D7.A, D8.A, Q10.E, Q9.E, R61.1
- removed net N$44: C14.1, R20.2, R21.1
- removed net N$48: C18.1, R24.2, R25.1, R26.1
- removed net N$50: C19.1, C20.+, IC2_A.OUT, R26.2
- removed net N$51: C22.2, C23.2, IC1_A.-IN, R28.1, R29.2, R31.1
- removed net N$52: C21.2, Q4.S, R29.1
- removed net N$53: C20.-, Q4.D, R27.2
- removed net N$54: C22.1, IC1_A.OUT, R30.2, R31.2, R32.1
- removed net N$55: C24.+, R32.2
- removed net N$57: C23.1, R30.1
- removed net N$58: R126.2, VR5.2, VR5.3
- removed net N$59: C116.2, VR5.1
- removed net N$60: C21.1, VR4.3
- removed net N$61: C116.1, VR4.2
- removed net N$62: C31.1, Q5.B, R49.2, R50.1
- removed net N$63: D6.A, Q5.C, R51.2
- removed net N$64: C30.1, D6.C, IC4.P$7, R52.2
- removed net N$65: C30.2, C31.2, IC4.P$5, R49.1
- removed net N$66: Q7.C, R52.1
- removed net N$67: R46.2, VR7.2, VR7.3
- removed net N$68: Q6.B, Q6.C, R46.1, R47.1
- removed net N$69: C32.+, Q7.B, R47.2, R48.2
- removed net N$70: C26.2, IC5_B.-IN, R38.2
- removed net N$71: C29.+, IC5_A.+IN, R38.1, R40.1, R41.2
- removed net N$72: C26.1, IC5_B.OUT, R37.2, VR3.1, VR3.2
- removed net N$73: R120.1, VR3.3
- removed net N$74: IC5_B.+IN, R36.1, R37.1
- removed net N$75: C27.+, IC5_A.-IN, R120.2
- removed net N$76: C28.+, IC5_A.OUT, R36.2, VR2.3
- removed net N$77: C27.-, C28.-
- removed net N$78: R48.1, VR2.2
- removed net N$79: D8.C, R62.1
- removed net N$80: Q8.B, R42.2, R43.1, R44.2
- removed net N$81: R42.1, VR1.2
- removed net N$82: Q11.B, R62.2
- removed net N$85: R54.2, SW101.P
- removed net OUT: C24.-, R33.1
- new net N$1: R20.2, VR2.1
- new net N$2: C10.+, IC2_B.+IN, R13.1, R14.2
- new net N$27: C9.+, D4.C, R13.2, R35.2, R41.2
- new net N$30: R119.2, VR1.1
- new net N$6: C1.2, C7.1, IC2_A.OUT, R12.2
- net +9V: now also IC1_B.+PWR, IC3_PWR.V+, IC4_PWR.V+, Q4.D, R17.1, R23.2, R25.2, R26.2, R36.2; no longer C39.+, D1.C, D2.C, IC1_PWR.V+, IC5_PWR.V+, IC6.VI, Q1.C, Q3.C, R53.2, R55.2, R56.2
- net GND: now also C10.-, C12.2, C13.2, C14.-, C15.2, C19.-, C24.-, C4.2, C9.-, D4.A, IC1_A.VC, IC1_B.-PWR, IC3_PWR.V-, IC4_PWR.V-, Q5.E, Q6.C, R11.1, R14.1, R30.1, R4.1, R40.1, R42.1, R43.1, R45.1, R5.1, SW1.S; no longer C12.-, C14.2, C16.2, C18.2, C29.-, C32.-, C33.2, C38.2, C39.-, C40.-, C9.2, D1.A, D7.C, D9.C, IC1_PWR.V-, IC3.1, IC4.P$3, IC5_PWR.V-, Q11.E, Q6.E, Q8.C, R16.1, R18.1, R23.1, R3.1, R33.2, R35.1, R41.1, R44.1, R51.1, R59.1, R60.1, SW101.S, VR1.1, VR2.1, VR4.1, VR6.1
- net N$10: now also D2.A, Q1.G; no longer C4.2, IC1_B.-IN, R4.2, R5.2, R6.1
- net N$11: now also C1.1, Q1.D, R2.2; no longer IC1_B.+IN, R7.2
- net N$12: now also C3.-, Q2.B, R3.2; no longer C4.1, IC1_B.OUT, R28.2, R6.2, R8.1, R9.1
- net N$13: now also C2.+, Q2.E, R5.2; no longer C5.1, R8.2
- net N$14: now also C2.-, R1.1, R4.2; no longer C5.2, C6.2, R9.2
- net N$15: now also C8.2, R16.2; no longer IC2_B.+IN, R13.2
- net N$16: now also C25.+, IC3_A.+IN, IC4_A.+IN, R20.1, R34.1, R39.1, R43.2; no longer C6.1, IC2_B.-IN, R11.1, R12.1, R126.1
- net N$17: now also R31.2, VR2.2; no longer D3.A, D4.C, R11.2
- net N$18: now also D3.A, Q3.G; no longer D3.C, D4.A, IC2_B.OUT, R12.2, R14.1
- net N$19: now also C18.2, IC4_B.+IN, R29.1, R36.1, R37.1, R45.2; no longer C8.1, R14.2, R15.1
- net N$20: now also IC4_B.-IN, R39.2; no longer C9.1, Q2.B, R15.2
- net N$21: now also C18.1, IC4_B.OUT, R37.2, VR2.3; no longer C10.2, C8.2, Q2.E, R16.2
- net N$22: now also R8.1, VR3.2; no longer D9.A, IC6.GND
- net N$23: now also C20.+, IC4_A.-IN, R31.1; no longer C13.1, IC3.7, IC3.8, R18.2
- net N$24: now also C21.+, IC4_A.OUT, R29.2, R38.1; no longer C11.+, R17.1, VR6.2
- net N$25: now also C20.-, C21.-; no longer C10.1, IC3.3, R17.2
- net N$26: now also IC3_A.-IN, R119.1, R38.2; no longer IC3.2, IC4.P$2
- net N$29: now also C23.2, D6.C, Q5.C, R22.1, R23.1, R44.1; no longer C34.2, Q9.C, R55.1, R57.1
- net N$3: now also C8.1, Q4.G, R15.2; no longer C1.2, R1.2
- net N$31: now also C17.1, Q7.C, R24.2, R25.1, R33.2; no longer C35.1, Q10.C, R56.1, R58.2
- net N$32: now also C16.1, C17.2, Q5.B, R30.2, R33.1; no longer C35.2, C36.1, Q9.B, R58.1, R59.2
- net N$33: now also IC3_A.OUT, R19.1, VR1.2, VR1.3; no longer IC3.6, IC4.P$4
- net N$34: now also C22.1, C23.1, Q7.B, R40.2, R44.2; no longer C34.1, C37.1, Q10.B, R57.2, R60.2
- net N$35: now also C12.1, D3.C, R22.2; no longer LED.C, Q11.C
- net N$36: now also C13.1, D2.C, R24.1; no longer C33.1, C36.2, C37.2, R53.1, R54.1
- net N$38: now also C11.+, IC3_B.+IN, R28.2, R32.1; no longer D5.A, Q4.G
- net N$39: now also IC3_B.-IN, R19.2, R27.1; no longer C38.1, D5.C, R61.2
- net N$4: now also C24.+, Q6.B, R41.1, R42.2; no longer C1.1, Q1.B, R2.2
- net N$40: now also IC3_B.OUT, R27.2, VR3.3; no longer C17.+, R24.1
- net N$41: now also R18.2, SW1.P; no longer C13.2, R19.2, R20.1
- net N$42: now also D5.C, R17.2; no longer LED.A, R63.1
- net N$43: now also D5.A, D6.A; no longer D2.A, R63.2
- net N$45: now also C4.1, IC1_B.VC, R10.1, R8.2; no longer C15.1, R21.2, R22.1
- net N$46: now also C15.1, C16.2, C22.2, R18.1, R26.1; no longer C16.1, Q3.B, R22.2
- net N$47: now also IC1_B.IN, R9.2; no longer C15.2, C17.-, Q3.E, R23.2
- net N$49: now also C6.-, R9.1; no longer C19.2, IC2_A.-IN, R25.2
- net N$5: now also C7.2, IC1_B.OUT, IC2_A.-IN, R12.1; no longer C12.+, IC3.4, IC4.P$8
- net N$7: now also C5.+, C6.+, Q4.S, R11.2; no longer C2.-, Q1.E, R3.2
- net N$8: now also C5.-, Q3.D, R7.2; no longer C2.+, C3.2, R4.1
- net N$9: now also C3.+, Q1.S, Q3.S, R6.2; no longer C3.1, R5.1
- net VA: now also C19.+, Q6.E, R32.2, R35.1, VR3.1; no longer C40.+, IC3.5, IC4.P$1, IC6.VO, Q5.E, Q8.E, R40.2, R43.2, R50.2, VR1.3, VR6.3, VR7.1
- net VB: now also C14.+, IC1_A.-PWR, IC2_B.-IN, IC2_B.OUT, R10.2, R15.1, R28.1, R3.1, R6.1; no longer C25.+, IC1_A.+IN, R13.1, R19.1, R27.1, R34.1, R35.2
Other:
- note removed: "12"
- note removed: "13"
- moved on the sheet: C1, C11, C13, C15, C16, C18, C2, C20, C22, C23, C24, C25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

Commit message: 20180529
Parts:
- R18: value 100 -> 100R
Changed lines of the file:
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@@
 <?xml version="1.0" encoding="utf-8"?>
 <!DOCTYPE eagle SYSTEM "eagle.dtd">
-<eagle version="8.2.0">
+<eagle version="8.5.1">
 <drawing>
 <settings>
 <setting alwaysvectorfont="no"/>
+<setting keepoldvectorfont="yes"/>
 <setting verticaltext="up"/>
 </settings>
-<grid distance="0.1" unitdist="inch" unit="inch" style="lines" multiple="1" display="yes" altdistance="0.01" altunitdist="inch" altunit="inch"/>
+<grid distance="0.1" unitdist="inch" unit="inch" style="lines" multiple="1" display="no" altdistance="0.01" altunitdist="inch" altunit="inch"/>
 <layers>
 <layer number="1" name="Top" color="4" fill="1" visible="no" active="no"/>
@@
 <part name="V112" library="gm-supply" deviceset="+9V" device=""/>
 <part name="C15" library="pedals-capacitors-film" deviceset="CER/FILM" device="BOX.1" value="10n"/>
-<part name="R18" library="pedals-resistors" deviceset="R_" device=".3B" value="100"/>
+<part name="R18" library="pedals-resistors" deviceset="R_" device=".3B" value="100R"/>
 <part name="GND127" library="gm-supply" deviceset="GND" device=""/>
 <part name="SW1" library="pedals-switches" deviceset="MOMENTARY" device=""/>
@@
 <instance part="VB108" gate="G$1" x="220.98" y="22.86" rot="R180"/>
 <instance part="Q1" gate="1" x="233.68" y="38.1" rot="R90"/>
-<instance part="D2" gate="G$1" x="236.22" y="25.4" rot="R270"/>
+<instance part="D2" gate="G$1" x="236.22" y="25.4" rot="MR270"/>
 <instance part="R6" gate="G$1" x="246.38" y="33.02" rot="R90"/>
 <instance part="VB109" gate="G$1" x="246.38" y="22.86" rot="R180"/>
@@
 <instance part="C5" gate="1" x="208.28" y="76.2"/>
 <instance part="VB106" gate="G$1" x="215.9" y="58.42" rot="R180"/>
-<instance part="D3" gate="G$1" x="226.06" y="60.96" rot="R270"/>
+<instance part="D3" gate="G$1" x="226.06" y="60.96" rot="MR270"/>
 <instance part="Q2" gate="G$1" x="264.16" y="40.64"/>
 <instance part="R5" gate="G$1" x="266.7" y="25.4" rot="R90"/>
