File: Analogman King of Tone/pcb/kot.brd (EAGLE design)
At the start: 59 x 71.3 mm, 44 parts, among them IC1 JRC4580, J1 POWER_JACK, X1 2510-

Commit message: 20171023
Parts:
- moved C13 87.8 mm to (47.0, 38.7), turned to 180 degrees
- moved C12 80.0 mm to (45.7, 33.7)
- moved R14 71.0 mm to (43.8, 46.4)
- moved C11 67.0 mm to (40.0, 15.2), turned to 270 degrees
- moved C10 59.5 mm to (36.8, 15.2), turned to 90 degrees
- moved R13 58.3 mm to (45.1, 16.5), turned to 270 degrees
- moved D6 48.5 mm to (31.8, 22.9), turned to 90 degrees
- moved C9 48.4 mm to (19.1, 30.5), turned to 90 degrees
- moved D2 42.2 mm to (26.7, 22.9), turned to 90 degrees
- moved R9 39.8 mm to (21.6, 39.4), turned to 270 degrees
- moved D3 39.5 mm to (21.6, 15.2)
- moved D7 39.0 mm to (29.2, 22.9), turned to 270 degrees
- moved R12 37.6 mm to (9.53, 15.2)
- moved D5 36.9 mm to (24.1, 22.9), turned to 270 degrees
- moved R10 35.2 mm to (21.6, 29.2), turned to 90 degrees
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Routing:
- net VB: track 0.00 -> 69.7 mm
- net N$19: track 0.00 -> 38.5 mm
- net N$17: track 0.00 -> 34.5 mm
- net N$21: track 0.00 -> 34.4 mm
- net N$18: track 0.00 -> 25.6 mm
- net N$9: track 0.00 -> 21.6 mm
- net N$15: track 0.00 -> 20.5 mm
- net N$3: track 0.00 -> 19.0 mm
- net N$5: track 0.00 -> 16.6 mm
- net VR: track 0.00 -> 15.5 mm
- net N$20: track 0.00 -> 13.8 mm
- net N$11: track 0.00 -> 12.9 mm
- net N$1: track 0.00 -> 9.72 mm
- net OUT: track 61.1 -> 52.1 mm
- net N$13: track 0.00 -> 6.88 mm
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
Commit message: 20171023-01
Parts:
- moved C4 1.35 mm to (44.2, 25.4), turned to 0 degrees
- moved C12 1.27 mm to (47.0, 33.7)
- moved R2 1.27 mm to (37.5, 29.2)
- moved R3 1.27 mm to (40.0, 29.2)
Routing:
- net +9V: track 0.00 -> 67.7 mm
- net IN: track 3.44 -> 32.8 mm
- net VR: track 15.5 -> 41.8 mm
- net N$20: track 13.8 -> 39.9 mm
- net VB: track 69.7 -> 92.3 mm
- net OUT: track 52.1 -> 74.4 mm
- net N$23: track 0.00 -> 13.1 mm
- net N$11: track 12.9 -> 12.3 mm

Commit message: 20171102
Routing:
- net VR: track 41.8 -> 41.1 mm
Changed lines of the file:
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@@
 <contactref element="C8" pad="1"/>
 <contactref element="R14" pad="1"/>
+<via x="8.89" y="8.5725" extent="1-16" drill="0.5" diameter="0.85"/>
+<via x="19.05" y="8.5725" extent="1-16" drill="0.5" diameter="0.85"/>
+<via x="39.37" y="8.763" extent="1-16" drill="0.5" diameter="0.85"/>
+<via x="49.53" y="8.763" extent="1-16" drill="0.5" diameter="0.85"/>
+<via x="54.1655" y="20.955" extent="1-16" drill="0.5" diameter="0.85"/>
+<via x="54.1655" y="31.115" extent="1-16" drill="0.5" diameter="0.85"/>
+<via x="55.0545" y="41.275" extent="1-16" drill="0.5" diameter="0.85"/>
+<via x="3.048" y="31.115" extent="1-16" drill="0.5" diameter="0.85"/>
+<via x="3.048" y="41.275" extent="1-16" drill="0.5" diameter="0.85"/>
+<via x="7.1755" y="14.224" extent="1-16" drill="0.5" diameter="0.85"/>
+<via x="9.906" y="14.224" extent="1-16" drill="0.5" diameter="0.85"/>
+<via x="36.322" y="20.955" extent="1-16" drill="0.5" diameter="0.85"/>
+<via x="33.4645" y="20.955" extent="1-16" drill="0.5" diameter="0.85"/>
+<via x="9.398" y="31.115" extent="1-16" drill="0.5" diameter="0.85"/>
+<via x="36.322" y="26.67" extent="1-16" drill="0.5" diameter="0.85"/>
+<via x="33.4645" y="26.67" extent="1-16" drill="0.5" diameter="0.85"/>
+<via x="36.195" y="35.56" extent="1-16" drill="0.5" diameter="0.85"/>
+<via x="33.5915" y="35.56" extent="1-16" drill="0.5" diameter="0.85"/>
+<via x="19.05" y="11.7475" extent="1-16" drill="0.5" diameter="0.85"/>
+<via x="39.37" y="16.1925" extent="1-16" drill="0.5" diameter="0.85"/>
+<via x="49.53" y="16.1925" extent="1-16" drill="0.5" diameter="0.85"/>
+<via x="46.0375" y="31.115" extent="1-16" drill="0.5" diameter="0.85"/>
+<via x="42.7355" y="31.115" extent="1-16" drill="0.5" diameter="0.85"/>
+<via x="46.99" y="37.465" extent="1-16" drill="0.5" diameter="0.85"/>
+<via x="45.085" y="42.545" extent="1-16" drill="0.5" diameter="0.85"/>
+<via x="40.64" y="42.545" extent="1-16" drill="0.5" diameter="0.85"/>
+<via x="17.526" y="16.51" extent="1-16" drill="0.5" diameter="0.85"/>
+<via x="17.526" y="19.05" extent="1-16" drill="0.5" diameter="0.85"/>
+<via x="17.526" y="24.13" extent="1-16" drill="0.5" diameter="0.85"/>
+<via x="7.1755" y="16.764" extent="1-16" drill="0.5" diameter="0.85"/>
+<via x="30.2895" y="51.435" extent="1-16" drill="0.5" diameter="0.85"/>
+<via x="24.7015" y="36.195" extent="1-16" drill="0.5" diameter="0.85"/>
+<via x="21.5265" y="37.465" extent="1-16" drill="0.5" diameter="0.85"/>
+<via x="22.1615" y="27.94" extent="1-16" drill="0.5" diameter="0.85"/>
+<via x="29.845" y="11.7475" extent="1-16" drill="0.5" diameter="0.85"/>
+<via x="7.8105" y="22.479" extent="1-16" drill="0.5" diameter="0.85"/>
+<via x="15.8115" y="45.72" extent="1-16" drill="0.5" diameter="0.85"/>
+<via x="8.8265" y="41.275" extent="1-16" drill="0.5" diameter="0.85"/>
 </signal>
 <signal name="VR">
@@
 <wire x1="25.589228125" y1="41.927778125" x2="29.827221875" y2="41.927778125" width="0.8128" layer="16"/>
 <wire x1="29.827221875" y1="41.927778125" x2="29.845" y2="41.91" width="0.8128" layer="16"/>
-<wire x1="29.845" y1="41.91" x2="34.29" y2="41.91" width="0.8128" layer="16"/>
-<wire x1="34.29" y1="41.91" x2="37.465" y2="38.735" width="0.8128" layer="16"/>
-<wire x1="37.465" y1="38.735" x2="37.465" y2="33.02" width="0.8128" layer="16"/>
+<wire x1="29.845" y1="41.91" x2="33.02" y2="41.91" width="0.8128" layer="16"/>
+<wire x1="33.02" y1="41.91" x2="37.465" y2="37.465" width="0.8128" layer="16"/>
+<wire x1="37.465" y1="37.465" x2="37.465" y2="33.02" width="0.8128" layer="16"/>
 <wire x1="13.335" y1="33.02" x2="15.875" y2="33.02" width="0.8128" layer="1"/>
 <wire x1="15.875" y1="33.02" x2="18.415" y2="30.48" width="0.8128" layer="1"/>

Commit message: 20171216
Changed lines of the file:
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@@
 <via x="15.8115" y="45.72" extent="1-16" drill="0.5" diameter="0.85"/>
 <via x="8.8265" y="41.275" extent="1-16" drill="0.5" diameter="0.85"/>
+<via x="36.195" y="45.72" extent="1-16" drill="0.5" diameter="0.85"/>
+<via x="33.5915" y="45.72" extent="1-16" drill="0.5" diameter="0.85"/>
 </signal>
 <signal name="VR">

Commit message: 20180529
Parts:
- R2, R3: value 22k -> 47k
Changed lines of the file:
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@@
 <?xml version="1.0" encoding="utf-8"?>
 <!DOCTYPE eagle SYSTEM "eagle.dtd">
-<eagle version="8.2.0">
+<eagle version="8.7.0">
 <drawing>
 <settings>
 <setting alwaysvectorfont="no"/>
+<setting keepoldvectorfont="yes"/>
 <setting verticaltext="up"/>
 </settings>
@@
 <param name="dpMaxLengthDifference" value="10mm"/>
 <param name="dpGapFactor" value="2.5"/>
-<param name="checkGrid" value="0"/>
 <param name="checkAngle" value="0"/>
 <param name="checkFont" value="1"/>
 <param name="checkRestrict" value="0"/>
+<param name="checkStop" value="0"/>
+<param name="checkValues" value="0"/>
 <param name="useDiameter" value="13"/>
 <param name="maxErrors" value="50"/>
@@
 <element name="OUTPUT" library="pedals-jacks" package="NMJ6HCD2" value="" x="43.053" y="61.0235" rot="R90"/>
 <element name="R1" library="pedals-resistors" package="R0207/3" value="47" x="29.845" y="45.72" rot="R270"/>
-<element name="R2" library="pedals-resistors" package="R0207/3" value="22k" x="37.465" y="29.21" rot="R270"/>
-<element name="R3" library="pedals-resistors" package="R0207/3" value="22k" x="40.005" y="29.21" rot="R270"/>
+<element name="R2" library="pedals-resistors" package="R0207/3" value="47k" x="37.465" y="29.21" rot="R270"/>
+<element name="R3" library="pedals-resistors" package="R0207/3" value="47k" x="40.005" y="29.21" rot="R270"/>
 <element name="PRESENCE" library="pedals-potentiometers" package="16MM" value="50kB" x="47.625" y="13.6525"/>
 <element name="VOLUME" library="pedals-potentiometers" package="16MM" value="100kA" x="47.625" y="44.196"/>
@@
 <contactref element="INPUT" pad="S"/>
 <polygon width="0.3048" layer="16" isolate="0.254">
-<vertex x="0" y="72.39"/>
-<vertex x="58.42" y="72.39"/>
-<vertex x="58.42" y="0.635"/>
-<vertex x="0" y="0.635"/>
+<vertex x="-0.635" y="73.025"/>
+<vertex x="59.055" y="73.025"/>
+<vertex x="59.055" y="0.635"/>
+<vertex x="-0.635" y="0.635"/>
 </polygon>
 <contactref element="J1" pad="PWR"/>
@@
 <contactref element="D1" pad="A"/>
 <polygon width="0.3048" layer="1" isolate="0.254">
-<vertex x="0" y="1.27"/>
-<vertex x="59.055" y="1.27"/>
-<vertex x="59.055" y="73.66"/>
-<vertex x="-0.635" y="73.66"/>
-<vertex x="-0.635" y="1.27"/>
+<vertex x="-1.27" y="1.27"/>
+<vertex x="59.69" y="1.27"/>
+<vertex x="59.69" y="73.66"/>
+<vertex x="-1.27" y="73.66"/>
 </polygon>
 <via x="57.5945" y="61.595" extent="1-16" drill="0.5" diameter="0.85"/>
@@
 <via x="36.322" y="26.67" extent="1-16" drill="0.5" diameter="0.85"/>
 <via x="33.4645" y="26.67" extent="1-16" drill="0.5" diameter="0.85"/>
-<via x="36.195" y="35.56" extent="1-16" drill="0.5" diameter="0.85"/>
-<via x="33.5915" y="35.56" extent="1-16" drill="0.5" diameter="0.85"/>
+<via x="36.322" y="35.56" extent="1-16" drill="0.5" diameter="0.85"/>
+<via x="33.4645" y="35.56" extent="1-16" drill="0.5" diameter="0.85"/>
 <via x="19.05" y="11.7475" extent="1-16" drill="0.5" diameter="0.85"/>
 <via x="39.37" y="16.1925" extent="1-16" drill="0.5" diameter="0.85"/>
 <via x="49.53" y="16.1925" extent="1-16" drill="0.5" diameter="0.85"/>
-<via x="46.0375" y="31.115" extent="1-16" drill="0.5" diameter="0.85"/>
-<via x="42.7355" y="31.115" extent="1-16" drill="0.5" diameter="0.85"/>
+<via x="46.0375" y="30.48" extent="1-16" drill="0.5" diameter="0.85"/>
+<via x="42.7355" y="30.48" extent="1-16" drill="0.5" diameter="0.85"/>
 <via x="46.99" y="37.465" extent="1-16" drill="0.5" diameter="0.85"/>
 <via x="45.085" y="42.545" extent="1-16" drill="0.5" diameter="0.85"/>
@@
 <via x="36.195" y="45.72" extent="1-16" drill="0.5" diameter="0.85"/>
 <via x="33.5915" y="45.72" extent="1-16" drill="0.5" diameter="0.85"/>
+<via x="21.3995" y="61.595" extent="1-16" drill="0.5" diameter="0.85"/>
+<via x="27.94" y="18.0975" extent="1-16" drill="0.5" diameter="0.85"/>
 </signal>
 <signal name="VR">
@@
 <contactref element="R7" pad="2"/>
 <wire x1="5.715" y1="38.1" x2="5.715" y2="40.64" width="0.254" layer="16"/>
-<wire x1="5.715" y1="40.64" x2="3.81" y2="42.545" width="0.254" layer="16"/>
-<wire x1="3.81" y1="42.545" x2="3.81" y2="44.45" width="0.254" layer="16"/>
+<wire x1="5.715" y1="40.64" x2="3.81" y2="42.2275" width="0.254" layer="16"/>
+<wire x1="3.81" y1="42.2275" x2="3.81" y2="44.45" width="0.254" layer="16"/>
 <wire x1="3.81" y1="44.45" x2="5.715" y2="46.355" width="0.254" layer="16"/>
 <wire x1="5.715" y1="30.48" x2="3.81" y2="32.385" width="0.254" layer="16"/>
@@
 <contactref element="R10" pad="1"/>
 <wire x1="13.335" y1="27.94" x2="15.875" y2="25.4" width="0.254" layer="16"/>
-<wire x1="19.05" y1="27.94" x2="21.59" y2="25.4" width="0.254" layer="16"/>
 <wire x1="15.875" y1="25.4" x2="16.9545" y2="25.4" width="0.254" layer="16"/>
 <wire x1="16.9545" y1="25.4" x2="17.4625" y2="25.908" width="0.254" layer="16"/>
@@
 <wire x1="17.4625" y1="27.432" x2="17.9705" y2="27.94" width="0.254" layer="16"/>
 <wire x1="17.9705" y1="27.94" x2="19.05" y2="27.94" width="0.254" layer="16"/>
+<wire x1="19.05" y1="27.94" x2="21.59" y2="25.4" width="0.254" layer="16"/>
 </signal>
 <signal name="N$12">
@@
 <contactref element="VOLUME" pad="3"/>
 <wire x1="52.705" y1="12.6525" x2="47.625" y2="12.6525" width="0.254" layer="16"/>
-<wire x1="45.085" y1="20.32" x2="45.085" y2="21.59" width="0.254" layer="1"/>
-<wire x1="45.085" y1="21.59" x2="47.625" y2="24.13" width="0.254" layer="1"/>
-<wire x1="47.625" y1="24.13" x2="47.625" y2="27.94" width="0.254" layer="1"/>
-<wire x1="47.625" y1="27.94" x2="42.545" y2="33.02" width="0.254" layer="1"/>
-<wire x1="42.545" y1="33.02" x2="42.545" y2="43.196" width="0.254" layer="1"/>
+<wire x1="45.085" y1="20.32" x2="45.085" y2="20.955" width="0.254" layer="1"/>
+<wire x1="45.085" y1="20.955" x2="47.625" y2="23.495" width="0.254" layer="1"/>
+<wire x1="47.625" y1="23.495" x2="47.625" y2="27.305" width="0.254" layer="1"/>
+<wire x1="47.625" y1="27.305" x2="42.545" y2="32.385" width="0.254" layer="1"/>
+<wire x1="42.545" y1="32.385" x2="42.545" y2="43.196" width="0.254" layer="1"/>
 <wire x1="47.625" y1="12.6525" x2="47.625" y2="12.7" width="0.254" layer="16"/>
 <wire x1="47.625" y1="12.6525" x2="47.625" y2="15.24" width="0.254" layer="16"/>
