File: MXR Blue Box/pcb/bluebox.brd (EAGLE design)
At the start: 59 x 87.8 mm, 58 parts, among them IC1 TL072, IC2 TL074, J1 POWER_JACK, Q1 2N5457, Q2 2N5457, Q3 2N5457, Q4 2N5457, Q5 2N3906-, X1 2510-

Commit message: 20171120
Parts:
- removed C11, C6, C7, C8, C9: 47n, pedals-capacitors-film:BOX_SMALL
- removed C12: 15u, pedals-capacitors-elec:050_020_1
- removed C13, C5: 10n, pedals-capacitors-film:BOX_SMALL
- removed IC1: TL072, pedals-integrated circuits:DIL0
- removed Q1, Q2, Q3, Q4: 2N5457, pedals-transistors:TO92-
- removed Q5: 2N3906-, pedals-transistors:TO92-
- removed R10, R13, R16, R27, R7: 22k, pedals-resistors:R0207/3
- removed R11, R12, R14, R15, R17, R4, R6, R8, R9: 10k, pedals-resistors:R0207/3
- removed R18, R19, R20, R22, R24, R26: 150k, pedals-resistors:R0207/3
- removed R21: 56k, pedals-resistors:R0207/3
- removed R23: 3.9M, pedals-resistors:R0207/3
- removed R25, R5: 470k, pedals-resistors:R0207/3
- moved D2 0.64 mm to (28.6, 47.2)
- moved R2 0.64 mm to (28.6, 38.1)
- moved C3 0.25 mm to (24.7, 35.3)
Connections:
- removed net N$10: C7.2, IC2.1, R8.2, R9.1
- removed net N$11: R27.1, SW1.1
- removed net N$12: IC2.6, R11.1, R9.2, SW1.2
- removed net N$13: C7.1, IC2.5, Q2.3, R10.2
- removed net N$14: C8.2, IC2.7, R11.2, R12.1
- removed net N$15: IC1.3, R25.2, R26.1
- removed net N$16: IC2.9, R12.2, R14.1
- removed net N$17: C8.1, IC2.10, Q3.3, R13.2
- removed net N$18: C9.2, IC2.8, R14.2, R15.1
- removed net N$20: IC2.13, R15.2, R17.1
- removed net N$21: C9.1, IC2.12, Q4.3, R16.2
- removed net N$22: IC2.14, R17.2, R18.1, R27.2
- removed net N$24: Q5.2, R18.2, R19.1, R20.1
- removed net N$25: C11.2, Q5.1, R20.2, R21.2
- removed net N$26: C13.2, IC1.2, R24.1
- removed net N$5: C5.2, R4.2
- removed net N$6: C6.2, IC1.6, IC1.7, R19.2, R6.1
- removed net N$7: IC2.2, R6.2, R8.1
- removed net N$8: C5.1, IC1.5, R5.1
- removed net N$9: C6.1, IC2.3, Q1.3, R7.2
- net GND: no longer C12.-, IC1.4, R21.1, R22.1
- net IN: no longer R4.1
- net N$19: no longer C13.1, IC1.1, R25.1
- net N$27: no longer C12.+, R23.1, R24.2, SPEED.2
- net OUT: no longer C11.1, R22.2
- net VA: no longer Q1.1, Q2.1, Q3.1, Q4.1, R23.2
- net VB: no longer Q1.2, Q2.2, Q3.2, Q4.2, Q5.3, R10.1, R13.1, R16.1, R26.2, R5.2, R7.1
- net VR: no longer IC1.8
Routing:
- net +9V: track 2.54 -> 102.0 mm
- net VB: track 109.7 -> 52.6 mm
- net N$6: track 51.3 -> 0.00 mm
- net N$24: track 45.4 -> 0.00 mm
- net N$14: track 36.4 -> 0.00 mm
- net N$13: track 33.2 -> 0.00 mm
- net VA: track 65.4 -> 35.3 mm
- net N$9: track 29.6 -> 0.00 mm
- net N$18: track 27.4 -> 0.00 mm
- net N$10: track 25.1 -> 0.00 mm
- net IN: track 45.7 -> 24.1 mm
- net N$12: track 21.2 -> 0.00 mm
- net N$17: track 18.1 -> 0.00 mm
- net N$11: track 17.9 -> 0.00 mm
- net N$15: track 15.9 -> 0.00 mm
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
Commit message: 20171216
Parts:
- removed TRIM1: 250k, pedals-potentiometers:RTRIM3296W
- added C11, C12: 47n, pedals-capacitors-film:BOX_SMALL
- added C13, C14: 1u, pedals-capacitors-elec:040_020
- added C15: 6.8n, pedals-capacitors-film:BOX_SMALL
- added C16, C5, C6: 100u, pedals-capacitors-elec:050_020
- added C7: 10n, pedals-capacitors-film:BOX_SMALL
- added C8: 1n, pedals-capacitors-film:BOX_SMALL
- added C9: 330p, pedals-capacitors-film:050X030_025_2
- added D3: 1N914, pedals-diodes:DO35-2
- added IC1: (no value), pedals-integrated circuits:DIL0
- added Q1, Q2, Q3: 2N3904, pedals-transistors:TO92-
- added R10, R7: 150k, pedals-resistors:R0207/3
- added R11, R16, R24, R8: 1M, pedals-resistors:R0207/3
- added R12, R14, R5: 10k, pedals-resistors:R0207/3
- added R13, R15, R17, R18, R19, R20, R21, R22, R23: 56k, pedals-resistors:R0207/3
- added R4: 330, pedals-resistors:R0207/3
- added R6: 2.2M, pedals-resistors:R0207/3
- added R9: 470k, pedals-resistors:R0207/3
- BLEND: value 500kC -> 100kB
- C10: value 47n -> 10u; device pedals-capacitors-film:BOX_SMALL -> pedals-capacitors-elec:050_020
- C2: value 100n -> 100u; device pedals-capacitors-film:050X030_025_2 -> pedals-capacitors-elec:050_020
- C3: value 100u -> 47u
- C4: value 47u -> 100n; device pedals-capacitors-elec:050_020 -> pedals-capacitors-film:050X030_025_2
- D2: value 5.1V -> 1N914; device pedals-diodes:DO41-2 -> pedals-diodes:DO35-2
- IC2: value TL074 -> 4013N
- LEVEL: value 1MB -> 100kB
- R2: value 10k -> 56k
- R3: value 680 -> 56k
- moved C10 47.1 mm to (5.40, 6.92), turned to 0 degrees
- moved R3 38.6 mm to (27.3, 6.35), turned to 90 degrees
- moved R2 31.8 mm to (29.8, 6.35)
- moved D2 28.5 mm to (6.99, 28.6)
- moved C3 27.3 mm to (23.5, 8.00)
- moved R1 25.0 mm to (38.1, 14.0)
- moved C2 22.9 mm to (41.9, 11.2), turned to 90 degrees
- moved C4 20.2 mm to (52.7, 24.1), turned to 90 degrees
- moved IC2 18.9 mm to (41.9, 25.4)
- moved SW1 18.8 mm to (47.6, 33.7)
- moved C1 15.1 mm to (22.2, 17.1), turned to 270 degrees
- moved X1 6.99 mm to (29.2, -3.17)
- moved D1 3.22 mm to (34.5, 48.9), turned to 0 degrees
- renumbered DEPTH to LEVEL, SPEED to BLEND
Connections:
- removed net VA: C10.2, LEVEL.1, LEVEL.2
- new net N$10: IC1.5, R11.1, R12.2
- new net N$11: IC1.7, R11.2, R13.1
- new net N$12: Q1.2, R13.2, R14.2
- new net N$13: Q2.2, R16.2
- new net N$14: Q2.1, R17.1, R18.1
- new net N$15: BLEND.3, R18.2, R19.2
- new net N$16: BLEND.1, R20.2, R21.1
- new net N$17: C12.1, R19.1, R20.1
- new net N$18: C14.+, D3.C, R17.2, R22.2, R23.2
- new net N$20: C13.-, D2.C, D3.A
- new net N$21: C12.2, LEVEL.3
- new net N$22: IC2.13, IC2.3, SW1.3
- new net N$23: IC2.12, IC2.9
- new net N$24: IC2.1, SW1.1
- new net N$25: IC2.2, IC2.5
- new net N$5: C8.1, IC1.3, R7.2, R8.2
- new net N$6: C9.2, IC1.2, R10.2, R9.1
- new net N$7: C11.2, C13.+, C9.1, IC1.1, R9.2
- new net N$8: C10.+, R10.1
- new net N$9: C11.1, IC1.6, R15.2
- new net VC: C4.1, C5.+, IC2.14, R4.2
- new net VD: C6.+, IC2.11, Q1.1, R16.1, R5.2
- net +9V: now also C16.+, R4.1, R5.1
- net GND: now also BLEND.2, C14.-, C15.2, C16.-, C2.-, C4.2, C5.-, C6.-, IC1.4, IC2.10, IC2.4, IC2.6, IC2.7, IC2.8, LEVEL.1, Q1.3, Q2.3, Q3.3, R14.1, R23.1, R3.1, R6.1; no longer C2.2, C4.-, IC2.11, TRIM1.1
- net IN: now also C7.2, R6.2
- net N$1: now also Q3.1, R21.2, R22.1; no longer R3.1, TRIM1.2
- net N$19: now also Q3.2, R24.1; no longer BLEND.1
- net N$27: now also R24.2, SW1.2; no longer BLEND.3
- net N$3: now also C7.1, R7.1; no longer LEVEL.3, R3.2
- net OUT: now also C15.1, LEVEL.2
- net VB: now also C10.-, C3.+, C8.2, R12.1, R15.1, R3.2, R8.1; no longer C10.1, C4.+, D2.C, TRIM1.3
- net VR: now also C2.+, IC1.8; no longer C2.1, C3.+, IC2.4
Routing:
- net OUT: track 20.0 -> 72.7 mm
- net VA: track 35.3 -> 0.00 mm
- net VD: track 0.00 -> 31.0 mm
- net N$9: track 0.00 -> 20.8 mm
- net N$21: track 0.00 -> 19.3 mm
- net N$6: track 0.00 -> 17.7 mm
- net N$18: track 0.00 -> 16.0 mm
- net N$10: track 0.00 -> 15.1 mm
- net N$22: track 0.00 -> 13.7 mm
- net N$14: track 0.00 -> 13.4 mm
- net N$19: track 6.35 -> 19.7 mm
- net N$11: track 0.00 -> 12.5 mm
- net N$7: track 0.00 -> 12.4 mm
- net N$5: track 0.00 -> 12.0 mm
- net N$17: track 0.00 -> 11.5 mm
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Other:
- board size 59 x 87.8 mm -> 59 x 80.2 mm

Commit message: 20180207
Routing:
- net IN: track 19.3 -> 18.6 mm
Changed lines of the file:
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@@
 <?xml version="1.0" encoding="utf-8"?>
 <!DOCTYPE eagle SYSTEM "eagle.dtd">
-<eagle version="8.2.0">
+<eagle version="8.5.1">
 <drawing>
 <settings>
 <setting alwaysvectorfont="no"/>
+<setting keepoldvectorfont="yes"/>
 <setting verticaltext="up"/>
 </settings>
 <grid distance="0.025" unitdist="inch" unit="inch" style="lines" multiple="1" display="yes" altdistance="0.0025" altunitdist="inch" altunit="inch"/>
 <layers>
-<layer number="1" name="Top" color="4" fill="1" visible="no" active="yes"/>
+<layer number="1" name="Top" color="4" fill="1" visible="yes" active="yes"/>
 <layer number="2" name="Route2" color="1" fill="3" visible="no" active="no"/>
 <layer number="3" name="Route3" color="4" fill="3" visible="no" active="no"/>
@@
 <param name="dpMaxLengthDifference" value="10mm"/>
 <param name="dpGapFactor" value="2.5"/>
-<param name="checkGrid" value="0"/>
 <param name="checkAngle" value="0"/>
 <param name="checkFont" value="1"/>
 <param name="checkRestrict" value="0"/>
+<param name="checkStop" value="0"/>
+<param name="checkValues" value="0"/>
 <param name="useDiameter" value="13"/>
 <param name="maxErrors" value="50"/>
@@
 <contactref element="IC2" pad="7"/>
 <contactref element="C16" pad="-"/>
+<via x="39.37" y="-0.762" extent="1-16" drill="0.5" diameter="0.85"/>
+<via x="48.26" y="-0.762" extent="1-16" drill="0.5" diameter="0.85"/>
+<via x="54.864" y="5.715" extent="1-16" drill="0.5" diameter="0.85"/>
+<via x="54.864" y="17.145" extent="1-16" drill="0.5" diameter="0.85"/>
+<via x="54.864" y="28.575" extent="1-16" drill="0.5" diameter="0.85"/>
+<via x="49.149" y="40.005" extent="1-16" drill="0.5" diameter="0.85"/>
+<via x="19.05" y="-0.762" extent="1-16" drill="0.5" diameter="0.85"/>
+<via x="10.16" y="-0.762" extent="1-16" drill="0.5" diameter="0.85"/>
+<via x="37.2745" y="40.005" extent="1-16" drill="0.5" diameter="0.85"/>
+<via x="37.2745" y="31.75" extent="1-16" drill="0.5" diameter="0.85"/>
+<via x="30.2895" y="40.005" extent="1-16" drill="0.5" diameter="0.85"/>
+<via x="30.2895" y="31.75" extent="1-16" drill="0.5" diameter="0.85"/>
+<via x="21.3995" y="40.005" extent="1-16" drill="0.5" diameter="0.85"/>
+<via x="10.6045" y="40.64" extent="1-16" drill="0.5" diameter="0.85"/>
+<via x="44.704" y="15.24" extent="1-16" drill="0.5" diameter="0.85"/>
+<via x="38.989" y="12.065" extent="1-16" drill="0.5" diameter="0.85"/>
+<via x="34.544" y="8.89" extent="1-16" drill="0.5" diameter="0.85"/>
+<via x="31.369" y="8.89" extent="1-16" drill="0.5" diameter="0.85"/>
+<via x="34.544" y="17.526" extent="1-16" drill="0.5" diameter="0.85"/>
+<via x="31.369" y="17.4625" extent="1-16" drill="0.5" diameter="0.85"/>
+<via x="33.274" y="24.511" extent="1-16" drill="0.5" diameter="0.85"/>
+<via x="27.559" y="17.4625" extent="1-16" drill="0.5" diameter="0.85"/>
+<via x="24.384" y="14.9225" extent="1-16" drill="0.5" diameter="0.85"/>
+<via x="21.844" y="10.16" extent="1-16" drill="0.5" diameter="0.85"/>
+<via x="8.509" y="10.16" extent="1-16" drill="0.5" diameter="0.85"/>
+<via x="8.509" y="14.9225" extent="1-16" drill="0.5" diameter="0.85"/>
+<via x="15.494" y="14.9225" extent="1-16" drill="0.5" diameter="0.85"/>
+<via x="19.939" y="24.511" extent="1-16" drill="0.5" diameter="0.85"/>
+<via x="3.3655" y="28.575" extent="1-16" drill="0.5" diameter="0.85"/>
+<via x="12.8905" y="28.575" extent="1-16" drill="0.5" diameter="0.85"/>
+<via x="15.621" y="36.195" extent="1-16" drill="0.5" diameter="0.85"/>
 </signal>
 <signal name="VR">
@@
 <contactref element="C7" pad="2"/>
 <wire x1="12.065" y1="-0.635" x2="12.065" y2="1.905" width="0.254" layer="16"/>
-<wire x1="12.065" y1="-0.635" x2="11.43" y2="-2.54" width="0.254" layer="1"/>
-<wire x1="11.43" y1="-2.54" x2="13.335" y2="-4.445" width="0.254" layer="1"/>
-<wire x1="13.335" y1="-4.445" x2="25.4" y2="-4.445" width="0.254" layer="1"/>
+<wire x1="12.065" y1="-0.635" x2="12.065" y2="-2.54" width="0.254" layer="1"/>
+<wire x1="12.065" y1="-2.54" x2="13.97" y2="-4.445" width="0.254" layer="1"/>
+<wire x1="13.97" y1="-4.445" x2="25.4" y2="-4.445" width="0.254" layer="1"/>
 </signal>
 <signal name="N$4">

Commit message: 20180529
Parts:
- removed C6: 100u, pedals-capacitors-elec:050_020
- R10: value 150k -> 1k
Connections:
- net GND: no longer C6.-
- net VD: no longer C6.+
Routing:
- net VD: track 31.0 -> 27.2 mm
Changed lines of the file:
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@@
 <?xml version="1.0" encoding="utf-8"?>
 <!DOCTYPE eagle SYSTEM "eagle.dtd">
-<eagle version="8.5.1">
+<eagle version="8.7.0">
 <drawing>
 <settings>
@@
 <element name="C5" library="pedals-capacitors-elec" package="050_020" value="100u" x="52.705" y="16.764" rot="R270"/>
 <element name="R5" library="pedals-resistors" package="R0207/3" value="10k" x="45.72" y="13.97" rot="R90"/>
-<element name="C6" library="pedals-capacitors-elec" package="050_020" value="100u" x="41.91" y="16.764" rot="R270"/>
 <element name="R6" library="pedals-resistors" package="R0207/3" value="2.2M" x="12.065" y="5.715" rot="R270"/>
 <element name="R7" library="pedals-resistors" package="R0207/3" value="150k" x="14.605" y="5.715" rot="R90"/>
@@
 <element name="R9" library="pedals-resistors" package="R0207/3" value="470k" x="9.525" y="15.875" rot="R90"/>
 <element name="C9" library="pedals-capacitors-film" package="050X030_025_2" value="330p" x="6.985" y="14.605" rot="R270"/>
-<element name="R10" library="pedals-resistors" package="R0207/3" value="150k" x="4.445" y="15.875" rot="R90"/>
+<element name="R10" library="pedals-resistors" package="R0207/3" value="1k" x="4.445" y="15.875" rot="R90"/>
 <element name="C11" library="pedals-capacitors-film" package="BOX_SMALL" value="47n" x="14.605" y="22.86" rot="R180"/>
 <element name="R11" library="pedals-resistors" package="R0207/3" value="1M" x="24.765" y="16.51" rot="R90"/>
@@
 <contactref element="INPUT" pad="S"/>
 <polygon width="0.3048" layer="16" isolate="0.254">
-<vertex x="0" y="72.39"/>
-<vertex x="58.42" y="72.39"/>
-<vertex x="58.42" y="-7.62"/>
-<vertex x="0" y="-7.62"/>
+<vertex x="-1.27" y="73.66"/>
+<vertex x="59.055" y="73.66"/>
+<vertex x="59.055" y="-7.62"/>
+<vertex x="-1.27" y="-7.62"/>
 </polygon>
 <contactref element="J1" pad="PWR"/>
@@
 <contactref element="C4" pad="2"/>
 <contactref element="C5" pad="-"/>
-<contactref element="C6" pad="-"/>
 <contactref element="R6" pad="1"/>
 <contactref element="IC1" pad="4"/>
@@
 <via x="39.37" y="-0.762" extent="1-16" drill="0.5" diameter="0.85"/>
 <via x="48.26" y="-0.762" extent="1-16" drill="0.5" diameter="0.85"/>
-<via x="54.864" y="5.715" extent="1-16" drill="0.5" diameter="0.85"/>
-<via x="54.864" y="17.145" extent="1-16" drill="0.5" diameter="0.85"/>
-<via x="54.864" y="28.575" extent="1-16" drill="0.5" diameter="0.85"/>
+<via x="54.61" y="5.715" extent="1-16" drill="0.5" diameter="0.85"/>
+<via x="54.61" y="17.145" extent="1-16" drill="0.5" diameter="0.85"/>
+<via x="54.61" y="28.575" extent="1-16" drill="0.5" diameter="0.85"/>
 <via x="49.149" y="40.005" extent="1-16" drill="0.5" diameter="0.85"/>
 <via x="19.05" y="-0.762" extent="1-16" drill="0.5" diameter="0.85"/>
 <via x="10.16" y="-0.762" extent="1-16" drill="0.5" diameter="0.85"/>
-<via x="37.2745" y="40.005" extent="1-16" drill="0.5" diameter="0.85"/>
-<via x="37.2745" y="31.75" extent="1-16" drill="0.5" diameter="0.85"/>
+<via x="33.2105" y="40.005" extent="1-16" drill="0.5" diameter="0.85"/>
+<via x="33.2105" y="31.75" extent="1-16" drill="0.5" diameter="0.85"/>
 <via x="30.2895" y="40.005" extent="1-16" drill="0.5" diameter="0.85"/>
 <via x="30.2895" y="31.75" extent="1-16" drill="0.5" diameter="0.85"/>
 <via x="21.3995" y="40.005" extent="1-16" drill="0.5" diameter="0.85"/>
-<via x="10.6045" y="40.64" extent="1-16" drill="0.5" diameter="0.85"/>
 <via x="44.704" y="15.24" extent="1-16" drill="0.5" diameter="0.85"/>
 <via x="38.989" y="12.065" extent="1-16" drill="0.5" diameter="0.85"/>
@@
 <via x="12.8905" y="28.575" extent="1-16" drill="0.5" diameter="0.85"/>
 <via x="15.621" y="36.195" extent="1-16" drill="0.5" diameter="0.85"/>
+<via x="3.3655" y="40.005" extent="1-16" drill="0.5" diameter="0.85"/>
+<via x="3.1115" y="17.145" extent="1-16" drill="0.5" diameter="0.85"/>
+<via x="24.384" y="24.511" extent="1-16" drill="0.5" diameter="0.85"/>
+<via x="10.414" y="24.511" extent="1-16" drill="0.5" diameter="0.85"/>
+<via x="44.704" y="19.685" extent="1-16" drill="0.5" diameter="0.85"/>
+<via x="45.339" y="32.385" extent="1-16" drill="0.5" diameter="0.85"/>
+<via x="9.7155" y="40.005" extent="1-16" drill="0.5" diameter="0.85"/>
 </signal>
 <signal name="VR">
@@
 <signal name="VD">
 <contactref element="R5" pad="2"/>
-<contactref element="C6" pad="+"/>
 <contactref element="Q1" pad="1"/>
 <contactref element="R16" pad="1"/>
 <contactref element="IC2" pad="11"/>
-<wire x1="45.702221875" y1="17.762221875" x2="41.911271875" y2="17.762221875" width="0.8128" layer="16"/>
 <wire x1="45.702221875" y1="17.762221875" x2="45.72" y2="17.78" width="0.8128" layer="16"/>
-<wire x1="41.911271875" y1="17.762221875" x2="41.911271875" y2="21.588728125" width="0.8128" layer="16"/>
 <wire x1="41.91" y1="21.59" x2="41.911271875" y2="21.588728125" width="0.8128" layer="16"/>
-<wire x1="41.911271875" y1="17.762221875" x2="41.292778125" y2="17.762221875" width="0.8128" layer="16"/>
-<wire x1="41.292778125" y1="17.762221875" x2="39.4335" y2="19.6215" width="0.8128" layer="16"/>
+<wire x1="39.4335" y1="19.6215" x2="41.292778125" y2="17.762221875" width="0.8128" layer="16"/>
 <wire x1="39.4335" y1="19.6215" x2="33.274" y2="19.6215" width="0.8128" layer="16"/>
 <wire x1="33.274" y1="19.6215" x2="31.4325" y2="21.463" width="0.8128" layer="16"/>
@@
 <wire x1="28.575" y1="31.115" x2="28.575" y2="28.575" width="0.8128" layer="16"/>
 <wire x1="28.575" y1="28.575" x2="29.21" y2="27.94" width="0.8128" layer="16"/>
+<wire x1="41.292778125" y1="17.762221875" x2="45.702221875" y2="17.762221875" width="0.8128" layer="16"/>
+<wire x1="39.4335" y1="19.6215" x2="41.91" y2="21.59" width="0" layer="19" extent="16-16"/>
 </signal>
 <signal name="N$5">
