File: MXR Phase 90/pcb/phase90.brd (EAGLE design)
At the start: 59 x 87.8 mm, 58 parts, among them IC1 TL072, IC2 TL074, J1 POWER_JACK, Q1 2N5457, Q2 2N5457, Q3 2N5457, Q4 2N5457, Q5 2N3906-, X1 2510-

Commit message: 20171216
Parts:
- moved R26 11.9 mm to (9.53, 36.2)
- moved C1 11.3 mm to (12.1, 19.7), turned to 180 degrees
- moved R1 11.2 mm to (23.5, 45.7)
- moved D1 10.8 mm to (21.0, 46.8), turned to 270 degrees
- moved R5 8.91 mm to (4.45, 26.0), turned to 90 degrees
- moved R2 8.03 mm to (26.0, 45.7), turned to 270 degrees
- moved X1 7.65 mm to (29.8, -2.54)
- moved C3 7.47 mm to (19.7, 40.9), turned to 270 degrees
- moved C4 7.11 mm to (36.2, 42.9), turned to 90 degrees
- moved R12 7.01 mm to (21.6, 8.26)
- moved R17 7.01 mm to (36.8, 8.26)
- moved C2 7.00 mm to (18.6, 17.1)
- moved R14 6.99 mm to (24.8, 8.26)
- moved R15 6.99 mm to (33.7, 8.26)
- moved R18 6.99 mm to (39.4, 8.26)
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Routing:
- net IN: track 45.7 -> 34.5 mm
- net N$2: track 88.6 -> 77.9 mm
- net N$6: track 51.3 -> 42.5 mm
- net VB: track 99.0 -> 90.2 mm
- net N$15: track 15.9 -> 7.62 mm
- net N$4: track 99.7 -> 92.9 mm
- net N$19: track 11.8 -> 18.0 mm
- net N$14: track 37.3 -> 31.8 mm
- net OUT: track 26.4 -> 21.2 mm
- net N$24: track 45.4 -> 40.7 mm
- net N$26: track 8.15 -> 12.0 mm
- net VR: track 51.5 -> 55.2 mm, vias 1 -> 0
- net +9V: track 102.0 -> 104.3 mm
- net N$18: track 24.2 -> 22.3 mm
- net VA: track 66.4 -> 64.7 mm
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Other:
- board size 59 x 87.8 mm -> 59 x 80.2 mm

Commit message: 20180207
Routing:
- net N$2: track 77.9 -> 78.7 mm
Changed lines of the file:
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@@
 <?xml version="1.0" encoding="utf-8"?>
 <!DOCTYPE eagle SYSTEM "eagle.dtd">
-<eagle version="8.2.0">
+<eagle version="8.5.1">
 <drawing>
 <settings>
 <setting alwaysvectorfont="no"/>
+<setting keepoldvectorfont="yes"/>
 <setting verticaltext="up"/>
 </settings>
@@
 <param name="dpMaxLengthDifference" value="10mm"/>
 <param name="dpGapFactor" value="2.5"/>
-<param name="checkGrid" value="0"/>
 <param name="checkAngle" value="0"/>
 <param name="checkFont" value="1"/>
 <param name="checkRestrict" value="0"/>
+<param name="checkStop" value="0"/>
+<param name="checkValues" value="0"/>
 <param name="useDiameter" value="13"/>
 <param name="maxErrors" value="50"/>
@@
 <contactref element="IC2" pad="11"/>
 <contactref element="IC1" pad="4"/>
+<via x="19.05" y="-2.54" extent="1-16" drill="0.5" diameter="0.85"/>
+<via x="9.525" y="-2.54" extent="1-16" drill="0.5" diameter="0.85"/>
+<via x="39.37" y="-2.54" extent="1-16" drill="0.5" diameter="0.85"/>
+<via x="55.499" y="5.715" extent="1-16" drill="0.5" diameter="0.85"/>
+<via x="55.499" y="17.145" extent="1-16" drill="0.5" diameter="0.85"/>
+<via x="55.499" y="28.575" extent="1-16" drill="0.5" diameter="0.85"/>
+<via x="55.499" y="40.005" extent="1-16" drill="0.5" diameter="0.85"/>
+<via x="2.9845" y="17.145" extent="1-16" drill="0.5" diameter="0.85"/>
+<via x="2.9845" y="28.575" extent="1-16" drill="0.5" diameter="0.85"/>
+<via x="2.9845" y="40.005" extent="1-16" drill="0.5" diameter="0.85"/>
+<via x="2.9845" y="5.715" extent="1-16" drill="0.5" diameter="0.85"/>
+<via x="30.2895" y="43.688" extent="1-16" drill="0.5" diameter="0.85"/>
+<via x="37.2745" y="40.005" extent="1-16" drill="0.5" diameter="0.85"/>
+<via x="49.784" y="28.575" extent="1-16" drill="0.5" diameter="0.85"/>
+<via x="43.434" y="28.575" extent="1-16" drill="0.5" diameter="0.85"/>
+<via x="40.4495" y="27.051" extent="1-16" drill="0.5" diameter="0.85"/>
+<via x="37.2745" y="27.051" extent="1-16" drill="0.5" diameter="0.85"/>
+<via x="33.4645" y="27.051" extent="1-16" drill="0.5" diameter="0.85"/>
+<via x="44.323" y="17.145" extent="1-16" drill="0.5" diameter="0.85"/>
+<via x="30.353" y="17.145" extent="1-16" drill="0.5" diameter="0.85"/>
+<via x="20.193" y="17.145" extent="1-16" drill="0.5" diameter="0.85"/>
+<via x="16.383" y="17.145" extent="1-16" drill="0.5" diameter="0.85"/>
+<via x="43.434" y="6.35" extent="1-16" drill="0.5" diameter="0.85"/>
+<via x="40.259" y="6.35" extent="1-16" drill="0.5" diameter="0.85"/>
+<via x="30.099" y="6.35" extent="1-16" drill="0.5" diameter="0.85"/>
+<via x="21.844" y="6.35" extent="1-16" drill="0.5" diameter="0.85"/>
+<via x="17.399" y="6.35" extent="1-16" drill="0.5" diameter="0.85"/>
+<via x="16.383" y="24.765" extent="1-16" drill="0.5" diameter="0.85"/>
+<via x="16.383" y="28.575" extent="1-16" drill="0.5" diameter="0.85"/>
+<via x="13.335" y="33.655" extent="1-16" drill="0.5" diameter="0.85"/>
+<via x="10.795" y="33.655" extent="1-16" drill="0.5" diameter="0.85"/>
 </signal>
 <signal name="VR">
@@
 <wire x1="7.252" y1="54.6735" x2="7.0485" y2="54.6735" width="0.254" layer="16"/>
 <wire x1="7.0485" y1="54.6735" x2="1.905" y2="49.53" width="0.254" layer="16"/>
-<wire x1="1.905" y1="49.53" x2="1.905" y2="6.35" width="0.254" layer="16"/>
-<wire x1="1.905" y1="6.35" x2="9.525" y2="-1.27" width="0.254" layer="16"/>
-<wire x1="9.525" y1="-1.27" x2="26.035" y2="-1.27" width="0.254" layer="16"/>
+<wire x1="1.905" y1="49.53" x2="1.905" y2="5.08" width="0.254" layer="16"/>
+<wire x1="1.905" y1="5.08" x2="8.255" y2="-1.27" width="0.254" layer="16"/>
+<wire x1="8.255" y1="-1.27" x2="26.035" y2="-1.27" width="0.254" layer="16"/>
 </signal>
 <signal name="VB">
@@
 <wire x1="28.575" y1="41.91" x2="31.75" y2="41.91" width="0.8128" layer="16"/>
 <wire x1="28.575" y1="41.91" x2="26.035" y2="41.91" width="0.8128" layer="16"/>
-<wire x1="26.035" y1="41.91" x2="24.13" y2="40.005" width="0.8128" layer="1"/>
-<wire x1="24.13" y1="40.005" x2="22.86" y2="40.005" width="0.8128" layer="1"/>
-<wire x1="20.32" y1="37.465" x2="22.86" y2="40.005" width="0.8128" layer="1"/>
 <wire x1="31.75" y1="41.91" x2="36.17595" y2="41.91" width="0.8128" layer="16"/>
 <wire x1="36.193728125" y1="41.927778125" x2="36.17595" y2="41.91" width="0.8128" layer="16"/>
@@
 <wire x1="4.445" y1="33.655" x2="8.255" y2="37.465" width="0.8128" layer="1"/>
 <wire x1="9.525" y1="37.465" x2="8.255" y2="37.465" width="0.8128" layer="1"/>
-<wire x1="9.525" y1="37.465" x2="20.32" y2="37.465" width="0.8128" layer="1"/>
 <wire x1="9.525" y1="40.005" x2="9.525" y2="37.465" width="0.8128" layer="1"/>
 <wire x1="50.165" y1="33.655" x2="46.99" y2="33.655" width="0.8128" layer="16"/>
@@
 <wire x1="42.545" y1="34.925" x2="42.545" y2="36.79444375" width="0.8128" layer="16"/>
 <wire x1="42.545" y1="36.79444375" x2="42.527221875" y2="36.812221875" width="0.8128" layer="16"/>
+<wire x1="9.525" y1="37.465" x2="21.59" y2="37.465" width="0.8128" layer="1"/>
+<wire x1="21.59" y1="37.465" x2="26.035" y2="41.91" width="0.8128" layer="1"/>
 </signal>
 <signal name="VA">

Commit message: 20180529
Parts:
- moved X1 0.63 mm to (29.2, -2.54)
Routing:
- net N$2: track 78.7 -> 78.1 mm
- net +9V: track 104.3 -> 104.9 mm
- net N$4: track 92.9 -> 93.5 mm
- net OUT: track 21.2 -> 21.8 mm
Changed lines of the file:
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@@
 <element name="R1" library="pedals-resistors" package="R0207/3" value="47" x="23.495" y="45.72" rot="R270"/>
 <element name="SPEED" library="pedals-potentiometers" package="16MM" value="500kC" x="10.795" y="44.196"/>
-<element name="X1" library="pedals-headers" package="PAK100/2500-10" value="2510-" x="29.845" y="-2.54" rot="R180">
-<attribute name="MF" value="3M" x="29.845" y="-2.54" size="1.778" layer="27" rot="R180" display="off"/>
-<attribute name="MPN" value="2510-6002UB" x="29.845" y="-2.54" size="1.778" layer="27" rot="R180" display="off"/>
-<attribute name="OC_FARNELL" value="9838244" x="29.845" y="-2.54" size="1.778" layer="27" rot="R180" display="off"/>
-<attribute name="OC_NEWARK" value="46F4725" x="29.845" y="-2.54" size="1.778" layer="27" rot="R180" display="off"/>
+<element name="X1" library="pedals-headers" package="PAK100/2500-10" value="2510-" x="29.21" y="-2.54" rot="R180">
+<attribute name="MF" value="3M" x="29.21" y="-2.54" size="1.778" layer="27" rot="R180" display="off"/>
+<attribute name="MPN" value="2510-6002UB" x="29.21" y="-2.54" size="1.778" layer="27" rot="R180" display="off"/>
+<attribute name="OC_FARNELL" value="9838244" x="29.21" y="-2.54" size="1.778" layer="27" rot="R180" display="off"/>
+<attribute name="OC_NEWARK" value="46F4725" x="29.21" y="-2.54" size="1.778" layer="27" rot="R180" display="off"/>
 </element>
 <element name="D1" library="pedals-diodes" package="DO41-2" value="1N4002" x="20.955" y="46.7995" rot="R270"/>
@@
 <wire x1="26.035" y1="62.23" x2="26.035" y2="52.07" width="0.8128" layer="16"/>
 <wire x1="26.035" y1="52.07" x2="23.495" y2="49.53" width="0.8128" layer="16"/>
-<wire x1="28.575" y1="-1.27" x2="28.575" y2="0.635" width="0.8128" layer="1"/>
-<wire x1="28.575" y1="0.635" x2="29.845" y2="1.905" width="0.8128" layer="1"/>
-<wire x1="29.845" y1="1.905" x2="40.64" y2="1.905" width="0.8128" layer="1"/>
+<wire x1="27.94" y1="-1.27" x2="27.94" y2="0.635" width="0.8128" layer="1"/>
+<wire x1="27.94" y1="0.635" x2="29.21" y2="1.905" width="0.8128" layer="1"/>
+<wire x1="29.21" y1="1.905" x2="40.64" y2="1.905" width="0.8128" layer="1"/>
 <wire x1="40.64" y1="1.905" x2="41.91" y2="3.175" width="0.8128" layer="1"/>
 <wire x1="41.91" y1="3.175" x2="41.91" y2="33.655" width="0.8128" layer="1"/>
@@
 <contactref element="INPUT" pad="S"/>
 <polygon width="0.3048" layer="16" isolate="0.254">
-<vertex x="0" y="72.39"/>
-<vertex x="58.42" y="72.39"/>
-<vertex x="59.055" y="-7.62"/>
-<vertex x="0.635" y="-7.62"/>
+<vertex x="-1.27" y="73.66"/>
+<vertex x="59.055" y="73.66"/>
+<vertex x="59.69" y="-7.62"/>
+<vertex x="-0.635" y="-7.62"/>
 </polygon>
 <contactref element="J1" pad="PWR"/>
@@
 <contactref element="D1" pad="A"/>
 <polygon width="0.3048" layer="1" isolate="0.254">
-<vertex x="-0.635" y="-7.62"/>
+<vertex x="-1.27" y="-7.62"/>
 <vertex x="59.055" y="-7.62"/>
 <vertex x="59.055" y="73.66"/>
-<vertex x="-0.635" y="73.66"/>
+<vertex x="-1.27" y="73.66"/>
 </polygon>
 <via x="57.5945" y="61.595" extent="1-16" drill="0.5" diameter="0.85"/>
@@
 <contactref element="IC1" pad="4"/>
 <via x="19.05" y="-2.54" extent="1-16" drill="0.5" diameter="0.85"/>
-<via x="9.525" y="-2.54" extent="1-16" drill="0.5" diameter="0.85"/>
+<via x="8.89" y="-2.54" extent="1-16" drill="0.5" diameter="0.85"/>
 <via x="39.37" y="-2.54" extent="1-16" drill="0.5" diameter="0.85"/>
 <via x="55.499" y="5.715" extent="1-16" drill="0.5" diameter="0.85"/>
@@
 <via x="13.335" y="33.655" extent="1-16" drill="0.5" diameter="0.85"/>
 <via x="10.795" y="33.655" extent="1-16" drill="0.5" diameter="0.85"/>
+<via x="13.335" y="41.91" extent="1-16" drill="0.5" diameter="0.85"/>
+<via x="8.255" y="44.45" extent="1-16" drill="0.5" diameter="0.85"/>
+<via x="25.5905" y="28.575" extent="1-16" drill="0.5" diameter="0.85"/>
+<via x="23.0505" y="31.115" extent="1-16" drill="0.5" diameter="0.85"/>
+<via x="40.4495" y="32.131" extent="1-16" drill="0.5" diameter="0.85"/>
+<via x="43.6245" y="40.005" extent="1-16" drill="0.5" diameter="0.85"/>
+<via x="52.324" y="40.005" extent="1-16" drill="0.5" diameter="0.85"/>
+<via x="43.6245" y="32.131" extent="1-16" drill="0.5" diameter="0.85"/>
+<via x="40.513" y="19.685" extent="1-16" drill="0.5" diameter="0.85"/>
+<via x="40.513" y="13.335" extent="1-16" drill="0.5" diameter="0.85"/>
+<via x="5.5245" y="5.715" extent="1-16" drill="0.5" diameter="0.85"/>
+<via x="10.795" y="31.115" extent="1-16" drill="0.5" diameter="0.85"/>
+<via x="13.335" y="31.115" extent="1-16" drill="0.5" diameter="0.85"/>
+<via x="29.4005" y="28.575" extent="1-16" drill="0.5" diameter="0.85"/>
+<via x="35.2425" y="31.6865" extent="1-16" drill="0.5" diameter="0.85"/>
+<via x="50.1015" y="17.78" extent="1-16" drill="0.5" diameter="0.85"/>
 </signal>
 <signal name="VR">
@@
 <contactref element="R22" pad="2"/>
 <wire x1="52.705" y1="1.27" x2="50.165" y2="1.27" width="0.254" layer="16"/>
-<wire x1="33.655" y1="-3.81" x2="45.085" y2="-3.81" width="0.254" layer="1"/>
+<wire x1="33.02" y1="-3.81" x2="45.085" y2="-3.81" width="0.254" layer="1"/>
 <wire x1="45.085" y1="-3.81" x2="50.165" y2="1.27" width="0.254" layer="1"/>
 </signal>
@@
 <contactref element="X1" pad="8"/>
 <contactref element="R4" pad="1"/>
-<wire x1="26.035" y1="-3.81" x2="9.525" y2="-3.81" width="0.254" layer="1"/>
-<wire x1="9.525" y1="-3.81" x2="4.445" y2="1.27" width="0.254" layer="1"/>
-<wire x1="4.445" y1="1.27" x2="4.445" y2="12.065" width="0.254" layer="1"/>
+<wire x1="25.4" y1="-3.81" x2="8.255" y2="-3.81" width="0.254" layer="1"/>
+<wire x1="8.255" y1="-3.81" x2="4.445" y2="0" width="0.254" layer="1"/>
+<wire x1="4.445" y1="0" x2="4.445" y2="12.065" width="0.254" layer="1"/>
 </signal>
 <signal name="N$4">
 <contactref element="OUTPUT" pad="T"/>
 <contactref element="X1" pad="1"/>
-<wire x1="33.655" y1="-1.27" x2="53.975" y2="-1.27" width="0.254" layer="16"/>
+<wire x1="33.02" y1="-1.27" x2="53.975" y2="-1.27" width="0.254" layer="16"/>
 <wire x1="53.975" y1="-1.27" x2="56.515" y2="1.27" width="0.254" layer="16"/>
 <wire x1="56.515" y1="1.27" x2="56.515" y2="44.45" width="0.254" layer="16"/>
@@
 <wire x1="1.905" y1="49.53" x2="1.905" y2="5.08" width="0.254" layer="16"/>
 <wire x1="1.905" y1="5.08" x2="8.255" y2="-1.27" width="0.254" layer="16"/>
-<wire x1="8.255" y1="-1.27" x2="26.035" y2="-1.27" width="0.254" layer="16"/>
+<wire x1="8.255" y1="-1.27" x2="25.4" y2="-1.27" width="0.254" layer="16"/>
 </signal>
 <signal name="VB">
