File: Paul C. Timmy/pcb/timmy.brd (EAGLE design)
At the start: 59 x 87.8 mm, 58 parts, among them IC1 TL072, J1 POWER_JACK, Q1 2N5457, Q2 2N5457, Q3 2N5457, Q4 2N5457, Q5 2N3906-, X1 2510-

Commit message: 20171106
Parts:
- removed C11, C6: 47n, pedals-capacitors-film:BOX_SMALL
- removed C13: 10n, pedals-capacitors-film:BOX_SMALL
- removed C4: 47u, pedals-capacitors-elec:050_020
- removed IC2: (no value), pedals-integrated circuits:DIL14
- removed Q1, Q2, Q3, Q4: 2N5457, pedals-transistors:TO92-
- removed Q5: 2N3906-, pedals-transistors:TO92-
- removed R12, R14, R15, R17: 10k, pedals-resistors:R0207/3
- removed R13, R16, R27, R7: 22k, pedals-resistors:R0207/3
- removed R18, R19, R20, R22, R24, R26: 150k, pedals-resistors:R0207/3
- removed R21: 56k, pedals-resistors:R0207/3
- removed R23: 3.9M, pedals-resistors:R0207/3
- removed R25: 470k, pedals-resistors:R0207/3
- removed TRIM1: 250k, pedals-potentiometers:RTRIM3296W
- removed U$2: (no value), pedals-pcb:125B_PCB_HUGE
- added BASS, TREBLE: 50kB, pedals-potentiometers:16MM
- added D3, D4, D5, D6, D7, D8: 1N4148, pedals-diodes:DO35-2
- added U$1: (no value), pedals-pcb:125B_PCB
- C10: value 47n -> 10n
- C12: value 15u -> 1u; device pedals-capacitors-elec:050_020_1 -> pedals-capacitors-film:BOX_BIG
- C2: value 100n -> 100u; device pedals-capacitors-film:050X030_025_2 -> pedals-capacitors-elec:050_020
- C3: value 100u -> 47u
- C5: value 10n -> 47n
- C7: value 47n -> 100p; device pedals-capacitors-film:BOX_SMALL -> pedals-capacitors-film:050X030_025_2
- C8: value 47n -> 39n
- C9: value 47n -> 1u; device pedals-capacitors-film:BOX_SMALL -> pedals-capacitors-film:BOX_BIG
- D2: value 5.1V -> 1N4148; device pedals-diodes:DO41-2 -> pedals-diodes:DO35-2
- GAIN: value 500kC -> 1MB
- IC1: value TL072 -> LM4558; device pedals-integrated circuits:DIL0 -> pedals-integrated circuits:DIL08
- R10: value 22k -> 3.3k
- R11, R6, R8: value 10k -> 3.3k
- R2: value 10k -> 8.2k
- R3: value 680 -> 10k
- R4: value 10k -> 2.2M
- R5: value 470k -> 510k
- R9: value 10k -> 1.5k
- SW1: device pedals-switches:1MS1T1B1C0M2QE -> pedals-switches:M9040P
- VOLUME: value 1MB -> 10kB
- moved R8 84.9 mm to (-46.4, 29.2)
- moved R6 79.0 mm to (-41.3, 41.3), turned to 90 degrees
- moved D2 73.2 mm to (-43.8, 41.9)
- moved C7 65.5 mm to (-33.7, 41.9), turned to 270 degrees
- moved R10 55.9 mm to (-8.89, 36.8), turned to 90 degrees
- moved C3 45.3 mm to (-20.0, 29.2), turned to 0 degrees
- moved C10 45.2 mm to (-8.89, 45.7)
- moved C5 41.3 mm to (-33.7, 30.5)
- moved R4 41.3 mm to (-36.2, 29.2), turned to 270 degrees
- moved R9 35.8 mm to (-6.35, 36.8), turned to 90 degrees
- moved R11 33.4 mm to (-10.2, 25.4), turned to 90 degrees
- moved C2 28.2 mm to (38.5, 30.5), turned to 0 degrees
- moved IC1 21.9 mm to (28.6, 23.5), turned to 270 degrees
- moved C12 19.7 mm to (-14.0, 45.7), turned to 270 degrees
- moved R5 19.7 mm to (28.6, 16.5), turned to 180 degrees
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- renumbered DEPTH to VOLUME, SPEED to GAIN
Connections:
- removed net N$18: C9.2, IC2.8, R14.2, R15.1
- removed net N$19: C13.1, GAIN.1, IC1.1, R25.1
- removed net N$20: IC2.13, R15.2, R17.1
- removed net N$21: C9.1, IC2.12, Q4.3, R16.2
- removed net N$22: IC2.14, R17.2, R18.1, R27.2
- removed net N$24: Q5.2, R18.2, R19.1, R20.1
- removed net N$25: C11.2, Q5.1, R20.2, R21.2
- removed net N$26: C13.2, IC1.2, R24.1
- removed net N$27: C12.+, GAIN.2, GAIN.3, R23.1, R24.2
- removed net VA: C10.2, Q1.1, Q2.1, Q3.1, Q4.1, R23.2, VOLUME.1, VOLUME.2
- net GND: now also C10.2, C2.-, R3.1, R4.1, VOLUME.1; no longer C12.-, C2.2, C4.-, D2.A, IC2.11, R21.1, R22.1, TRIM1.1
- net IN: now also C5.2, R4.2; no longer R4.1
- net N$1: now also D6.C, SW1.3; no longer R3.1, TRIM1.2
- net N$10: now also D7.A, D8.C, SW1.1; no longer C7.2, IC2.1, R8.2, R9.1
- net N$11: now also BASS.3, C8.1, R8.1; no longer R27.1, SW1.1
- net N$12: now also R9.1, TREBLE.3; no longer IC2.6, R11.1, R9.2, SW1.2
- net N$13: now also BASS.1, BASS.2, C9.1; no longer C7.1, IC2.5, Q2.3, R10.2
- net N$14: now also C10.1, IC1.5, R9.2; no longer C8.2, IC2.7, R11.2, R12.1
- net N$15: now also IC1.6, R10.1, R11.2; no longer IC1.3, R25.2, R26.1
- net N$16: now also C12.2, IC1.7, R10.2; no longer IC2.9, R12.2, R14.1
- net N$17: now also C12.1, VOLUME.3; no longer C8.1, IC2.10, Q3.3, R13.2
- net N$3: now also C5.1, IC1.3, R5.2; no longer R3.2, VOLUME.3
- net N$5: now also C7.2, D3.C, D4.A, IC1.2, R6.1, R8.2, SW1.2; no longer C5.2, R4.2
- net N$6: now also C7.1, D2.A, D5.C, D6.A, D7.C, D8.A, GAIN.2, GAIN.3, IC1.1, TREBLE.1, TREBLE.2; no longer C6.2, IC1.6, IC1.7, R19.2, R6.1
- net N$7: now also GAIN.1; no longer IC2.2, R8.1
- net N$8: now also D2.C, D3.A; no longer C5.1, IC1.5, R5.1
- net N$9: now also D4.C, D5.A; no longer C6.1, IC2.3, Q1.3, R7.2
- net OUT: now also VOLUME.2; no longer C11.1, R22.2
- net VB: now also C3.+, C8.2, C9.2, R11.1, R3.2, R5.1; no longer C10.1, C4.+, D2.C, Q1.2, Q2.2, Q3.2, Q4.2, Q5.3, R10.1, R13.1, R16.1, R26.2, R5.2, R7.1, TRIM1.3
- net VR: now also C2.+; no longer C2.1, C3.+, IC2.4
Routing:
- net VB: track 70.2 -> 0.00 mm
- net VA: track 64.9 -> 0.00 mm
- net OUT: track 0.00 -> 62.7 mm
- net VR: track 25.3 -> 0.00 mm
- net N$2: track 88.6 -> 71.8 mm
- net N$15: track 15.9 -> 0.00 mm
- net N$4: track 99.7 -> 84.3 mm
- net N$27: track 12.7 -> 0.00 mm
- net N$25: track 12.0 -> 0.00 mm
- net N$19: track 11.8 -> 0.00 mm
- net N$26: track 8.15 -> 0.00 mm
- net N$1: track 6.88 -> 0.00 mm
- net N$8: track 6.13 -> 0.00 mm
- net N$5: track 6.13 -> 0.00 mm
- net N$24: track 5.08 -> 0.00 mm
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Other:
- board size 59 x 87.8 mm -> 59 x 71.3 mm

Commit message: 20180529
Parts:
- moved D8 74.1 mm to (-26.7, 1.27)
- moved D7 64.6 mm to (-19.1, 6.35)
- moved D6 57.7 mm to (-17.8, 11.4)
Changed lines of the file:
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@@
 <?xml version="1.0" encoding="utf-8"?>
 <!DOCTYPE eagle SYSTEM "eagle.dtd">
-<eagle version="8.2.0">
+<eagle version="8.5.1">
 <drawing>
 <settings>
 <setting alwaysvectorfont="no"/>
+<setting keepoldvectorfont="yes"/>
 <setting verticaltext="up"/>
 </settings>
@@
 <param name="dpMaxLengthDifference" value="10mm"/>
 <param name="dpGapFactor" value="2.5"/>
-<param name="checkGrid" value="0"/>
 <param name="checkAngle" value="0"/>
 <param name="checkFont" value="1"/>
 <param name="checkRestrict" value="0"/>
+<param name="checkStop" value="0"/>
+<param name="checkValues" value="0"/>
 <param name="useDiameter" value="13"/>
 <param name="maxErrors" value="50"/>
@@
 <element name="C3" library="pedals-capacitors-elec" package="050_020" value="47u" x="-19.957415625" y="29.21"/>
 <element name="SW1" library="pedals-switches" package="M9040P" value="" x="29.21" y="34.29" rot="R180"/>
-<element name="D6" library="pedals-diodes" package="DO35-2" value="1N4148" x="5.715" y="-41.275"/>
-<element name="D7" library="pedals-diodes" package="DO35-2" value="1N4148" x="5.715" y="-53.34"/>
-<element name="D8" library="pedals-diodes" package="DO35-2" value="1N4148" x="5.715" y="-65.405"/>
+<element name="D6" library="pedals-diodes" package="DO35-2" value="1N4148" x="-17.78" y="11.43"/>
+<element name="D7" library="pedals-diodes" package="DO35-2" value="1N4148" x="-19.05" y="6.35"/>
+<element name="D8" library="pedals-diodes" package="DO35-2" value="1N4148" x="-26.67" y="1.27"/>
 </elements>
 <signals>
@@
 <wire x1="-38.735" y1="39.37" x2="-33.655" y2="44.45" width="0" layer="19" extent="1-1"/>
 <wire x1="-43.815" y1="44.45" x2="-38.735" y2="39.37" width="0" layer="19" extent="1-1"/>
-<wire x1="8.255" y1="-41.275" x2="47.625" y2="12.6525" width="0" layer="19" extent="1-1"/>
-<wire x1="3.175" y1="-53.34" x2="8.255" y2="-41.275" width="0" layer="19" extent="1-1"/>
-<wire x1="8.255" y1="-65.405" x2="3.175" y2="-53.34" width="0" layer="19" extent="1-1"/>
+<wire x1="-15.24" y1="11.43" x2="47.625" y2="12.6525" width="0" layer="19" extent="1-1"/>
+<wire x1="-21.59" y1="6.35" x2="-15.24" y2="11.43" width="0" layer="19" extent="1-1"/>
+<wire x1="-24.13" y1="1.27" x2="-21.59" y2="6.35" width="0" layer="19" extent="1-1"/>
 </signal>
 <signal name="N$7">
@@
 <contactref element="SW1" pad="3"/>
 <contactref element="D6" pad="C"/>
-<wire x1="3.175" y1="-41.275" x2="33.8201" y2="34.29" width="0" layer="19" extent="1-1"/>
+<wire x1="-20.32" y1="11.43" x2="33.8201" y2="34.29" width="0" layer="19" extent="1-1"/>
 </signal>
 <signal name="N$10">
@@
 <contactref element="D7" pad="A"/>
 <contactref element="D8" pad="C"/>
-<wire x1="8.255" y1="-53.34" x2="3.175" y2="-65.405" width="0" layer="19" extent="1-1"/>
-<wire x1="24.5745" y1="34.29" x2="8.255" y2="-53.34" width="0" layer="19" extent="1-1"/>
+<wire x1="-16.51" y1="6.35" x2="-29.21" y2="1.27" width="0" layer="19" extent="1-1"/>
+<wire x1="24.5745" y1="34.29" x2="-16.51" y2="6.35" width="0" layer="19" extent="1-1"/>
 </signal>
 </signals>
