File: EHX Big Muff/pcb/opamp.sch (EAGLE design)
At the start: 52 parts, among them IC1 JRC4558, IC2 LM741, J2 POWER_JACK, SW1 SPDT, X1 2510-

Commit message: 20180803
Parts:
- removed X1: 2510-, pedals-headers:2510-
- added C16: 10u, pedals-capacitors-elec:0500
- added C17: 100u, pedals-capacitors-elec:0500
- added C18: 100n, pedals-capacitors-film:CER/FILM2
- added D8: 1N4148, pedals-diodes:DO35.2
- added K1: NA, pedals-relays:NA
- added LED, SW: JST-XH-02-PIN-ROUND-PAD, pedals-headers:JST-XH-02-PIN-ROUND-PAD
- added OK1: LTV816, pedals-integrated circuits:LTV816
- added Q6: 2N3904, pedals-transistors:2N3904
- added R27: 22k, pedals-resistors:R_.3B
- added R28: 1k, pedals-resistors:R_.3B
- added REG1: LM78L05, pedals-regulators:LM78L05
- added U1: ATTINY85-20P, pedals-microcontrollers:ATTINY85-20P
Connections:
- removed net N$35: OUTPUT.T, X1-1.KL
- removed net N$36: INPUT.T, X1-7.KL
- new net +5V: C16.+, C18.1, D8.C, K11.+, R28.2, REG1.VO, U1.VCC
- new net N$1: D8.A, K11.-, LED-1.S, Q6.C
- new net N$2: Q6.B, R27.2
- new net N$27: LED-2.S, R28.1
- new net N$38: K12.O, K13.O
- new net PB0: OK1.A, U1.PB0
- new net PB1: U1.PB1
- new net PB2: U1.PB2
- new net PB3: SW-2.S, U1.PB3
- new net PB4: U1.PB4
- new net PB5: R27.1, U1.NRES/PB5
- new net RETURN: K12.S, R20.2, VOLUME.2
- new net SEND: C6.1, K13.S, R6.2
- net +18V: now also C17.+, REG1.VI; no longer X1-5.KL
- net GND: now also C16.-, C17.-, C18.2, OK1.C, OK1.EMIT, Q6.E, REG1.GND, SW-1.S, U1.GND; no longer X1-3.KL
- net IN: now also INPUT.T, K13.P; no longer C6.1, R6.2, X1-8.KL
- net OUT: now also K12.P, OK1.COL, OUTPUT.T; no longer R20.2, VOLUME.2, X1-2.KL
Other:
- moved on the sheet: D1

Commit message: 20180910
Parts:
- R13: value 47 -> 47R
- SW1: value SPDT -> (none); device pedals-switches:SPDT -> pedals-switches:DPDT
Connections:
- new net N$28: C12.1, C13.+, SW1_A.1
- new net N$29: C15.1, SW1_A.3
- net N$14: now also C11.2; no longer C11.1
- net N$19: now also C11.1, SW1_A.2; no longer C11.2, C12.1, C13.+, C15.1
- net N$24: now also SW1_B.3; no longer SW1.O
- net N$25: now also SW1_B.1; no longer SW1.S
- net N$26: now also SW1_B.2; no longer SW1.P
- net N$6: now also C8.2; no longer C8.1
- net N$8: now also C8.1; no longer C8.2
Other:
- moved on the sheet: C11, C12, C13, C14, C15, C6, C8, R16, R17, R18, R19, R20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
