File: Ross Compressor/pcb/rosscomp_th.sch (EAGLE design)
At the start: 58 parts, among them IC1 CA3080E, J1 POWER_JACK, Q1 2N5088, Q2 2N5088, Q3 2N5088, Q4 2N5088, Q5 2N5088, X1 2510-

Commit message: 20180803
Parts:
- removed X1: 2510-, pedals-headers:2510-
- added BLEND: 10kB, pedals-potentiometers:POTS16MM
- added C15: 10u, pedals-capacitors-elec:0500
- added C18, C23: 100n, pedals-capacitors-film:CER/FILM2
- added C19: 47u, pedals-capacitors-elec:0500
- added C20: 470n, pedals-capacitors-film:CER/FILMBOX.2
- added C21: 39p, pedals-capacitors-film:CER/FILM2
- added C22: 4.7u, pedals-capacitors-elec:0500
- added C24: 100u, pedals-capacitors-elec:0500
- added D4: 1N4148, pedals-diodes:DO35.2
- added IC2: TL072, pedals-integrated circuits:DUALTH
- added K1: NA, pedals-relays:NA
- added LED, SW: JST-XH-02-PIN-ROUND-PAD, pedals-headers:JST-XH-02-PIN-ROUND-PAD
- added OK1: LTV816, pedals-integrated circuits:LTV816
- added Q6: 2N3904, pedals-transistors:2N3904
- added R27: 22k, pedals-resistors:R_.3B
- added R28: 1k, pedals-resistors:R_.3B
- added R29, R30: 50k, pedals-resistors:R_.3B
- added R31: 1M, pedals-resistors:R_.3B
- added R32: 100k, pedals-resistors:R_.3B
- added R33: 220k, pedals-resistors:R_.3B
- added R34, R35, R36, R37: 15k, pedals-resistors:R_.3B
- added R38: 56k, pedals-resistors:R_.3B
- added REG1: LM78L05, pedals-regulators:LM78L05
- added U1: ATTINY85-20P, pedals-microcontrollers:ATTINY85-20P
- VOL: value 100kA -> 50kA
Connections:
- new net +5V: C15.+, C18.1, D4.C, K11.+, R28.2, REG1.VO, U1.VCC
- new net N$24: LED-2.S, R28.1
- new net N$28: C21.2, IC2_A.-IN, R32.2, R33.1
- new net N$29: C21.1, IC2_A.OUT, R33.2, R34.1
- new net N$30: BLEND.1, R34.2, R37.1
- new net N$31: BLEND.3, R35.2, R36.1
- new net N$33: BLEND.2, IC2_B.+IN
- new net N$34: R23.2, R35.1
- new net N$35: C22.+, IC2_B.OUT, R38.2
- new net N$36: C22.-, VOL.3
- new net N$37: IC2_B.-IN, R36.2, R37.2, R38.1
- new net N$38: K12.O, K13.O
- new net PB0: OK1.A, U1.PB0
- new net PB1: U1.PB1
- new net PB2: U1.PB2
- new net PB3: SW-2.S, U1.PB3
- new net PB4: U1.PB4
- new net PB5: R27.1, U1.NRES/PB5
- new net RETURN: K12.S, VOL.2
- new net SEND: C3.2, C5.1, K13.S, R7.2
- new net VC: C19.+, IC2_A.+IN, R29.2, R30.2
- net +9V: now also C24.+, REG1.VI; no longer X1-5.KL
- net GND: now also C15.-, C18.2, C19.-, C23.1, C24.-, IC2_PWR.V-, OK1.C, OK1.EMIT, Q6.E, R30.1, R31.1, REG1.GND, SW-1.S, U1.GND; no longer X1-3.KL
- net IN: now also INPUT.T, K13.P; no longer C3.2, C5.1, R7.2, X1-8.KL
- net N$1: now also D4.A, K11.-, LED-1.S, Q6.C; no longer INPUT.T, X1-7.KL
- net N$22: now also C20.1, R32.1; no longer R23.2, VOL.3
- net N$4: now also Q6.B, R27.2; no longer OUTPUT.T, X1-1.KL
- net N$9: now also C20.2, R31.2
- net OUT: now also K12.P, OK1.COL, OUTPUT.T; no longer VOL.2, X1-2.KL
- net VR: now also C23.2, IC2_PWR.V+, R29.1
Other:
- moved on the sheet: C1, C14, C2, D1, INPUT, J1, OUTPUT, R1, R16, R2, VOL

Commit message: 20180910
Connections:
- removed net N$33: BLEND.2, IC2_B.+IN
- removed net N$38: K12.O, K13.O
- new net N$27: K12.O, K13.S
- new net N$32: K13.P
- net GND: now also K13.O
- net IN: no longer K13.P
- net OUT: no longer K12.P
- net PB3: now also R27.1; no longer SW-2.S
- net PB4: now also SW-2.S
- net PB5: no longer R27.1
- net RETURN: no longer K12.S
- net SEND: no longer K13.S
- net VC: now also BLEND.2, IC2_B.+IN
Other:
- moved on the sheet: K1
Changed lines of the file:
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@@
 <?xml version="1.0" encoding="utf-8"?>
 <!DOCTYPE eagle SYSTEM "eagle.dtd">
-<eagle version="9.0.0">
+<eagle version="9.1.3">
 <drawing>
 <settings>
@@
 <part name="C24" library="pedals-capacitors-elec" deviceset="050" device="0" value="100u"/>
 <part name="GND41" library="gm-supply" deviceset="GND" device=""/>
+<part name="VC3" library="pedals-supply" deviceset="VC" device=""/>
+<part name="GND42" library="pedals-supply" deviceset="GND" device=""/>
 </parts>
 <sheets>
@@
 <instance part="GND39" gate="GND" x="363.22" y="12.7"/>
 <instance part="K1" gate="1" x="-73.66" y="81.28"/>
-<instance part="K1" gate="2" x="-45.72" y="91.44"/>
-<instance part="K1" gate="3" x="-45.72" y="73.66"/>
+<instance part="K1" gate="2" x="-35.56" y="88.9" rot="R90"/>
+<instance part="K1" gate="3" x="-55.88" y="88.9" rot="R270"/>
 <instance part="C23" gate="G$1" x="33.02" y="113.03" rot="MR270"/>
 <instance part="GND40" gate="GND" x="33.02" y="101.6"/>
 <instance part="C24" gate="1" x="5.08" y="114.3" rot="MR270"/>
 <instance part="GND41" gate="GND" x="5.08" y="101.6"/>
+<instance part="VC3" gate="G$1" x="353.06" y="0" rot="R180"/>
+<instance part="GND42" gate="GND" x="-50.8" y="78.74"/>
 </instances>
 <busses>
@@
 <wire x1="5.08" y1="109.22" x2="5.08" y2="104.14" width="0.1524" layer="91"/>
 </segment>
+<segment>
+<pinref part="K1" gate="3" pin="O"/>
+<pinref part="GND42" gate="GND" pin="GND"/>
+<wire x1="-50.8" y1="83.82" x2="-50.8" y2="81.28" width="0.1524" layer="91"/>
+</segment>
 </net>
 <net name="OUT" class="0">
@@
 <pinref part="OK1" gate="G$1" pin="COL"/>
 </segment>
-<segment>
-<pinref part="K1" gate="2" pin="P"/>
-<wire x1="-45.72" y1="88.9" x2="-45.72" y2="86.36" width="0.1524" layer="91"/>
-<label x="-45.72" y="86.36" size="1.778" layer="95" rot="R270"/>
-</segment>
 </net>
 <net name="IN" class="0">
@@
 <label x="2.54" y="43.18" size="1.778" layer="95"/>
 <pinref part="INPUT" gate="G$1" pin="T"/>
-</segment>
-<segment>
-<pinref part="K1" gate="3" pin="P"/>
-<wire x1="-45.72" y1="71.12" x2="-45.72" y2="68.58" width="0.1524" layer="91"/>
-<label x="-45.72" y="68.58" size="1.778" layer="95" rot="R270"/>
 </segment>
 </net>
@@
 </segment>
 <segment>
+<pinref part="R27" gate="G$1" pin="1"/>
+<wire x1="-91.44" y1="66.04" x2="-93.98" y2="66.04" width="0.1524" layer="91"/>
+<label x="-99.06" y="66.04" size="1.778" layer="95"/>
+</segment>
+</net>
+<net name="PB4" class="0">
+<segment>
+<pinref part="U1" gate="G$1" pin="PB4"/>
+<wire x1="-20.32" y1="35.56" x2="-17.78" y2="35.56" width="0.1524" layer="91"/>
+<label x="-17.78" y="35.56" size="1.778" layer="95"/>
+</segment>
+<segment>
 <pinref part="SW" gate="-2" pin="S"/>
 <wire x1="-53.34" y1="60.96" x2="-55.88" y2="60.96" width="0.1524" layer="91"/>
@@
 </segment>
 </net>
-<net name="PB4" class="0">
-<segment>
-<pinref part="U1" gate="G$1" pin="PB4"/>
-<wire x1="-20.32" y1="35.56" x2="-17.78" y2="35.56" width="0.1524" layer="91"/>
-<label x="-17.78" y="35.56" size="1.778" layer="95"/>
-</segment>
-</net>
 <net name="PB5" class="0">
 <segment>
@@
 <wire x1="-20.32" y1="38.1" x2="-17.78" y2="38.1" width="0.1524" layer="91"/>
 <label x="-17.78" y="38.1" size="1.778" layer="95"/>
-</segment>
-<segment>
-<pinref part="R27" gate="G$1" pin="1"/>
-<wire x1="-91.44" y1="66.04" x2="-93.98" y2="66.04" width="0.1524" layer="91"/>
-<label x="-99.06" y="66.04" size="1.778" layer="95"/>
 </segment>
 </net>
@@
 <label x="33.02" y="55.88" size="1.778" layer="95"/>
 </segment>
-<segment>
-<pinref part="K1" gate="3" pin="S"/>
-<wire x1="-50.8" y1="78.74" x2="-53.34" y2="78.74" width="0.1524" layer="91"/>
-<label x="-60.96" y="78.74" size="1.778" layer="95"/>
-</segment>
 </net>
 <net name="RETURN" class="0">
@@
 <wire x1="391.16" y1="12.7" x2="393.7" y2="12.7" width="0.1524" layer="91"/>
 <label x="393.7" y="12.7" size="1.778" layer="95"/>
-</segment>
-<segment>
-<pinref part="K1" gate="2" pin="S"/>
-<wire x1="-50.8" y1="96.52" x2="-53.34" y2="96.52" width="0.1524" layer="91"/>
-<label x="-63.5" y="96.52" size="1.778" layer="95"/>
 </segment>
 </net>
@@
 <pinref part="IC2" gate="_A" pin="+IN"/>
 <wire x1="297.18" y1="2.54" x2="299.72" y2="2.54" width="0.1524" layer="91"/>
+</segment>
+<segment>
+<pinref part="BLEND" gate="G$1" pin="2"/>
+<wire x1="340.36" y1="15.24" x2="353.06" y2="15.24" width="0.1524" layer="91"/>
+<wire x1="353.06" y1="15.24" x2="353.06" y2="20.32" width="0.1524" layer="91"/>
+<pinref part="IC2" gate="_B" pin="+IN"/>
+<wire x1="353.06" y1="20.32" x2="355.6" y2="20.32" width="0.1524" layer="91"/>
+<pinref part="VC3" gate="G$1" pin="VC"/>
+<wire x1="353.06" y1="15.24" x2="353.06" y2="2.54" width="0.1524" layer="91"/>
+<junction x="353.06" y="15.24"/>
 </segment>
 </net>
@@
 </segment>
 </net>
-<net name="N$33" class="0">
-<segment>
-<pinref part="BLEND" gate="G$1" pin="2"/>
-<wire x1="340.36" y1="15.24" x2="353.06" y2="15.24" width="0.1524" layer="91"/>
-<wire x1="353.06" y1="15.24" x2="353.06" y2="20.32" width="0.1524" layer="91"/>
-<pinref part="IC2" gate="_B" pin="+IN"/>
-<wire x1="353.06" y1="20.32" x2="355.6" y2="20.32" width="0.1524" layer="91"/>
-</segment>
-</net>
 <net name="N$36" class="0">
 <segment>
@@
 </segment>
 </net>
-<net name="N$38" class="0">
-<segment>
-<pinref part="K1" gate="3" pin="O"/>
-<wire x1="-40.64" y1="78.74" x2="-38.1" y2="78.74" width="0.1524" layer="91"/>
-<wire x1="-38.1" y1="78.74" x2="-38.1" y2="96.52" width="0.1524" layer="91"/>
+<net name="N$27" class="0">
+<segment>
+<pinref part="K1" gate="3" pin="S"/>
+<wire x1="-50.8" y1="93.98" x2="-50.8" y2="96.52" width="0.1524" layer="91"/>
+<wire x1="-50.8" y1="96.52" x2="-40.64" y2="96.52" width="0.1524" layer="91"/>
 <pinref part="K1" gate="2" pin="O"/>
-<wire x1="-38.1" y1="96.52" x2="-40.64" y2="96.52" width="0.1524" layer="91"/>
-</segment>
-</net>
+<wire x1="-40.64" y1="96.52" x2="-40.64" y2="93.98" width="0.1524" layer="91"/>
+</segment>
+</net>
+<net name="N$32" class="0">
+<segment>
+<pinref part="K1" gate="3" pin="P"/>
+<wire x1="-58.42" y1="88.9" x2="-60.96" y2="88.9" width="0.1524" layer="91"/>
+</segment>
+</net>
