File: Relay switching/pcb/relay_switch_opto.brd (EAGLE design)
At the start: 160 x 100 mm, 12 parts, among them K1 G5V-2, Q1 2N3904, SW1 MOMENTARY, U1 ATTINY85-20P

Commit message: 20181201
Parts:
- removed K1: G5V-2, pedals-relays:G5V-2
- added K2: NA, pedals-relays:NA
- moved D1 1.80 mm to (35.6, 3.81)
- moved D2 1.27 mm to (45.7, 3.81)
- moved C3 1.27 mm to (55.9, 16.5)
- moved Q1 1.27 mm to (47.0, 10.2)
- moved R1 1.27 mm to (50.8, 10.2), turned to 270 degrees
- moved R2 1.27 mm to (43.2, 10.2)
- moved REG1 1.27 mm to (44.5, 19.1)
- moved U1 1.27 mm to (57.1, 10.2)
- moved C2 1.09 mm to (49.1, 17.5)
Connections:
- net +5V: now also K2.1; no longer K1.1
- net GND: now also K2.10; no longer K1.11
- net IN: now also K2.3, K2.8; no longer K1.6, K1.9
- net N$2: now also K2.12; no longer K1.16
- net OUT: now also K2.4; no longer K1.4
- net RETURN: now also K2.5; no longer K1.8
- net SEND: now also K2.9; no longer K1.13
Changed lines of the file:
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@@
 </autorouter>
 <elements>
-<element name="C2" library="pedals-capacitors-elec" package="050_020" value="10u" x="49.53" y="16.51" rot="R90"/>
-<element name="C3" library="pedals-capacitors-film" package="050X030_025_2" value="100n" x="55.88" y="17.78"/>
-<element name="D1" library="pedals-diodes" package="DO35-2" value="1N4148" x="36.83" y="2.54" rot="R180"/>
-<element name="D2" library="pedals-diodes" package="3MM_D" value="LED" x="46.99" y="3.81"/>
-<element name="K1" library="pedals-relays" package="G5V-2" package3d_urn="urn:adsk.eagle:package:24545/1" value="G5V-2" x="34.29" y="13.97" rot="R90">
-<attribute name="MF" value="" x="34.29" y="13.97" size="1.778" layer="27" rot="R90" display="off"/>
-<attribute name="MPN" value="G5V-2 5DC" x="34.29" y="13.97" size="1.778" layer="27" rot="R90" display="off"/>
-<attribute name="OC_FARNELL" value="9949488" x="34.29" y="13.97" size="1.778" layer="27" rot="R90" display="off"/>
-<attribute name="OC_NEWARK" value="78K5703" x="34.29" y="13.97" size="1.778" layer="27" rot="R90" display="off"/>
-<attribute name="SPICEPREFIX" value="J" x="34.29" y="13.97" size="1.778" layer="27" rot="R90" display="off"/>
-</element>
+<element name="C2" library="pedals-capacitors-elec" package="050_020" value="10u" x="49.149" y="17.526" rot="R90"/>
+<element name="C3" library="pedals-capacitors-film" package="050X030_025_2" value="100n" x="55.88" y="16.51"/>
+<element name="D1" library="pedals-diodes" package="DO35-2" value="1N4148" x="35.56" y="3.81" rot="R180"/>
+<element name="D2" library="pedals-diodes" package="3MM_D" value="LED" x="45.72" y="3.81"/>
 <element name="OK1" library="pedals-integrated circuits" package="DIL04" package3d_urn="urn:adsk.eagle:package:21938/1" value="LTV816" x="55.88" y="25.4">
 <attribute name="MF" value="" x="55.88" y="25.4" size="1.778" layer="27" display="off"/>
@@
 <attribute name="OC_NEWARK" value="unknown" x="55.88" y="25.4" size="1.778" layer="27" display="off"/>
 </element>
-<element name="Q1" library="pedals-transistors" package="TO92-" value="2N3904" x="46.99" y="8.89" rot="R270"/>
-<element name="R1" library="pedals-resistors" package="R0207/3" value="22k" x="50.8" y="8.89" rot="R90"/>
-<element name="R2" library="pedals-resistors" package="R0207/3" value="1k" x="43.18" y="8.89" rot="R90"/>
-<element name="REG1" library="pedals-regulators" package="TO92-" value="LM78L05" x="44.45" y="17.78" rot="R270"/>
+<element name="Q1" library="pedals-transistors" package="TO92-" value="2N3904" x="46.99" y="10.16" rot="R270"/>
+<element name="R1" library="pedals-resistors" package="R0207/3" value="22k" x="50.8" y="10.16" rot="R270"/>
+<element name="R2" library="pedals-resistors" package="R0207/3" value="1k" x="43.18" y="10.16" rot="R90"/>
+<element name="REG1" library="pedals-regulators" package="TO92-" value="LM78L05" x="44.45" y="19.05" rot="R270"/>
 <element name="SW1" library="pedals-switches" package="SPST" value="MOMENTARY" x="59.69" y="2.54"/>
-<element name="U1" library="pedals-microcontrollers" package="PDIP08_300MIL" value="ATTINY85-20P" x="57.15" y="11.43"/>
+<element name="U1" library="pedals-microcontrollers" package="PDIP08_300MIL" value="ATTINY85-20P" x="57.15" y="10.16"/>
+<element name="K2" library="pedals-relays" package="NA" package3d_urn="urn:adsk.eagle:package:24348/1" value="NA" x="35.56" y="12.7" rot="R90">
+<attribute name="MF" value="" x="35.56" y="12.7" size="1.778" layer="27" rot="R90" display="off"/>
+<attribute name="MPN" value="" x="35.56" y="12.7" size="1.778" layer="27" rot="R90" display="off"/>
+<attribute name="OC_FARNELL" value="unknown" x="35.56" y="12.7" size="1.778" layer="27" rot="R90" display="off"/>
+<attribute name="OC_NEWARK" value="unknown" x="35.56" y="12.7" size="1.778" layer="27" rot="R90" display="off"/>
+</element>
 </elements>
 <signals>
@@
 <contactref element="OK1" pad="2"/>
 <contactref element="OK1" pad="3"/>
-<contactref element="K1" pad="11"/>
 <polygon width="0.1524" layer="1">
 <vertex x="0" y="43.18"/>
@@
 <vertex x="63.5" y="43.18"/>
 </polygon>
+<contactref element="K2" pad="10"/>
 </signal>
 <signal name="+9V">
@@
 <contactref element="U1" pad="5"/>
 <contactref element="OK1" pad="1"/>
-<wire x1="54.61" y1="21.59" x2="60.96" y2="15.24" width="0" layer="19" extent="1-1"/>
+<wire x1="54.61" y1="21.59" x2="60.96" y2="13.97" width="0" layer="19" extent="1-1"/>
 </signal>
 <signal name="PB1">
 <contactref element="U1" pad="6"/>
 <contactref element="R1" pad="1"/>
-<wire x1="50.8" y1="5.08" x2="58.42" y2="15.24" width="0" layer="19" extent="1-1"/>
+<wire x1="50.8" y1="13.97" x2="58.42" y2="13.97" width="0" layer="19" extent="1-1"/>
 </signal>
 <signal name="PB2">
@@
 <contactref element="U1" pad="3"/>
 <contactref element="SW1" pad="1"/>
-<wire x1="58.42" y1="2.54" x2="58.42" y2="7.62" width="0" layer="19" extent="1-1"/>
+<wire x1="58.42" y1="2.54" x2="58.42" y2="6.35" width="0" layer="19" extent="1-1"/>
 </signal>
 <signal name="PB5">
@@
 <contactref element="C3" pad="1"/>
 <contactref element="D1" pad="C"/>
-<contactref element="K1" pad="1"/>
 <contactref element="R2" pad="2"/>
-<wire x1="53.34" y1="15.24" x2="53.34" y2="17.78" width="0" layer="19" extent="1-1"/>
-<wire x1="49.528728125" y1="15.511778125" x2="53.34" y2="15.24" width="0" layer="19" extent="1-1"/>
-<wire x1="44.45" y1="15.24" x2="49.528728125" y2="15.511778125" width="0" layer="19" extent="1-1"/>
-<wire x1="43.18" y1="12.7" x2="44.45" y2="15.24" width="0" layer="19" extent="1-1"/>
-<wire x1="38.1" y1="5.08" x2="43.18" y2="12.7" width="0" layer="19" extent="1-1"/>
-<wire x1="39.37" y1="2.54" x2="38.1" y2="5.08" width="0" layer="19" extent="1-1"/>
+<contactref element="K2" pad="1"/>
+<wire x1="53.34" y1="13.97" x2="53.34" y2="16.51" width="0" layer="19" extent="1-1"/>
+<wire x1="49.147728125" y1="16.527778125" x2="53.34" y2="16.51" width="0" layer="19" extent="1-1"/>
+<wire x1="44.45" y1="16.51" x2="49.147728125" y2="16.527778125" width="0" layer="19" extent="1-1"/>
+<wire x1="43.18" y1="13.97" x2="44.45" y2="16.51" width="0" layer="19" extent="1-1"/>
+<wire x1="38.1" y1="6.35" x2="43.18" y2="13.97" width="0" layer="19" extent="1-1"/>
+<wire x1="38.1" y1="3.81" x2="38.1" y2="6.35" width="0" layer="19" extent="1-1"/>
 </signal>
 <signal name="N$2">
 <contactref element="D1" pad="A"/>
-<contactref element="K1" pad="16"/>
 <contactref element="Q1" pad="1"/>
 <contactref element="D2" pad="P$1"/>
-<wire x1="48.26" y1="3.81" x2="46.99" y2="6.35" width="0" layer="19" extent="1-1"/>
-<wire x1="34.29" y1="2.54" x2="46.99" y2="6.35" width="0" layer="19" extent="1-1"/>
-<wire x1="30.48" y1="5.08" x2="34.29" y2="2.54" width="0" layer="19" extent="1-1"/>
+<contactref element="K2" pad="12"/>
+<wire x1="46.99" y1="3.81" x2="46.99" y2="7.62" width="0" layer="19" extent="1-1"/>
+<wire x1="33.02" y1="3.81" x2="46.99" y2="3.81" width="0" layer="19" extent="1-1"/>
+<wire x1="33.02" y1="6.35" x2="33.02" y2="3.81" width="0" layer="19" extent="1-1"/>
 </signal>
 <signal name="N$3">
 <contactref element="R1" pad="2"/>
 <contactref element="Q1" pad="2"/>
-<wire x1="46.99" y1="8.89" x2="50.8" y2="12.7" width="0" layer="19" extent="1-1"/>
+<wire x1="46.99" y1="10.16" x2="50.8" y2="6.35" width="0" layer="19" extent="1-1"/>
 </signal>
 <signal name="N$4">
 <contactref element="R2" pad="1"/>
 <contactref element="D2" pad="ANODE"/>
-<wire x1="45.72" y1="3.81" x2="43.18" y2="5.08" width="0" layer="19" extent="1-1"/>
+<wire x1="44.45" y1="3.81" x2="43.18" y2="6.35" width="0" layer="19" extent="1-1"/>
 </signal>
 <signal name="RETURN">
 <contactref element="OK1" pad="4"/>
-<contactref element="K1" pad="8"/>
-<wire x1="38.1" y1="22.86" x2="54.61" y2="29.21" width="0" layer="19" extent="1-1"/>
+<contactref element="K2" pad="5"/>
+<wire x1="38.1" y1="16.51" x2="54.61" y2="29.21" width="0" layer="19" extent="1-1"/>
 </signal>
 <signal name="IN">
-<contactref element="K1" pad="9"/>
-<contactref element="K1" pad="6"/>
-<wire x1="30.48" y1="22.86" x2="38.1" y2="17.78" width="0" layer="19" extent="1-1"/>
+<contactref element="K2" pad="3"/>
+<contactref element="K2" pad="8"/>
+<wire x1="33.02" y1="16.51" x2="38.1" y2="11.43" width="0" layer="19" extent="1-1"/>
 </signal>
 <signal name="OUT">
-<contactref element="K1" pad="4"/>
+<contactref element="K2" pad="4"/>
 </signal>
 <signal name="SEND">
-<contactref element="K1" pad="13"/>
+<contactref element="K2" pad="9"/>
 </signal>
 </signals>
