File: #Misc/Ibanez TS808/ts808_redraw.sch (EAGLE design)
At the start: 73 parts, among them IC101 RC4558, Q101 2SC1815BL, Q102 1SK44SP, Q103 2SC1815BL, Q104 2SK44SP, Q105 2SC1815BL, Q106 2SC1815BL, Q107 2SC1815BL

Commit message: 20171230
Parts:
- removed BATTERY: BATTERY, pedals-jacks:BATTERY
- removed DC: DCJACK, pedals-jacks:DC_KOBICONN
- removed INPUT: (no value), pedals-jacks:STEREO3PADS
- removed OUTPUT: (no value), pedals-jacks:MONO
Connections:
- removed net N$1 (its old number): C101.2, INPUT.T
- removed net N$2 (its old number): BATTERY.P$2, INPUT.R
- removed net N$26: C109.-, OUTPUT.TIP, R115.2
- removed net N$28: BATTERY.P$1, DC.R
- new net IN: C101.2
- new net OUT: C109.-, R115.2
- net +9V: no longer DC.S
- net GND: no longer DC.T, INPUT.S, OUTPUT.SLEEVE
Other:
- note removed: "1"
- note removed: "10"
- note removed: "11"
- note removed: "12"
- note removed: "13"
- note removed: "15"
- note removed: "2"
- note removed: "3"
- note removed: "4"
- note removed: "5"
- note removed: "6"
- note removed: "7"
- note removed: "8"
- note removed: "9"
- moved on the sheet: C103, C104, C106, C107, C108, C109, C110, C111, C112, C113, C114, C115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

Commit message: 20200325/10:41
Connections:
- net GND: no longer LEVEL.1
- net VB: now also LEVEL.1
