File: #Misc/Boss OD-1/od1_redraw.sch (EAGLE design)
At the start: 67 parts, among them Q1 2N5457, Q2 2N5457

Commit message: 20200329/10:01
Parts:
- R9: value 100k -> 10k
Other:
- note removed: "DRIVE"
- note removed: "LEVEL"
Changed lines of the file:
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@@
 <setting verticaltext="up"/>
 </settings>
-<grid distance="0.1" unitdist="inch" unit="inch" style="lines" multiple="1" display="yes" altdistance="0.01" altunitdist="inch" altunit="inch"/>
+<grid distance="0.1" unitdist="inch" unit="inch" style="lines" multiple="1" display="no" altdistance="0.01" altunitdist="inch" altunit="inch"/>
 <layers>
 <layer number="1" name="Top" color="4" fill="1" visible="no" active="no"/>
@@
 <part name="V2" library="gm-supply" deviceset="+9V" device=""/>
 <part name="GND1" library="gm-supply" deviceset="GND" device=""/>
-<part name="R9" library="pedals-resistors" deviceset="R_" device=".3B" value="100k"/>
+<part name="R9" library="pedals-resistors" deviceset="R_" device=".3B" value="10k"/>
 <part name="D3" library="pedals-diodes" deviceset="DO35" device=".2"/>
 <part name="GND2" library="gm-supply" deviceset="GND" device=""/>
@@
 <sheet>
 <plain>
-<text x="93.98" y="86.36" size="1.778" layer="95">DRIVE</text>
-<text x="175.26" y="50.8" size="1.778" layer="95">LEVEL</text>
 </plain>
 <instances>
@@
 <attribute name="VALUE" x="25.273" y="-20.32" size="1.778" layer="96" rot="R90" align="center"/>
 </instance>
-<instance part="C17" gate="1" x="33.02" y="-17.78" smashed="yes" rot="R270">
-<attribute name="NAME" x="36.703" y="-17.78" size="1.778" layer="95" rot="MR270" align="center"/>
-<attribute name="VALUE" x="29.337" y="-17.78" size="1.778" layer="96" rot="MR270" align="center"/>
+<instance part="C17" gate="1" x="33.02" y="-17.78" smashed="yes" rot="MR270">
+<attribute name="NAME" x="29.337" y="-17.78" size="1.778" layer="95" rot="R270" align="center"/>
+<attribute name="VALUE" x="36.703" y="-17.78" size="1.778" layer="96" rot="R270" align="center"/>
 </instance>
 <instance part="GND102" gate="GND" x="22.86" y="-27.94" smashed="yes">
