File: #Misc/Boss OD-2R/od2r_redraw.sch (EAGLE design)
At the start: 160 parts, among them Q1 2SK117-GR, Q10 2SK118-Y, Q102 2SK30A-Y, Q13 2SK117-GR, Q14 2SK117-GR, Q15 2SA970-GR, Q17 2SC3378-GR, Q18 2SA1335-GR, Q19 2SK118-Y, Q20 2SC3378-GR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

Commit message: 20200329/10:01
Parts:
- R82: value R7k -> 47k
- renumbered SW102 to ON/OFF
Other:
- moved on the sheet: C21, C22, Q18, R45, R46, R47
