File: #Misc/Dunlop Crybaby GCB-95/gcb95_redraw.sch (EAGLE design)
At the start: 29 parts, among them Q101 MPSA18, Q102 MPSA18, Q103 MPSA18

Commit message: 20200329/10:01
Parts:
- removed R109: (no value), pedals-resistors:R_.3B
Connections:
- removed net N$8: C108.2, R105.1, R109.1, R111.1
- net N$9: now also C108.2, R105.1, R111.1; no longer R109.2
