File: #Misc/Fulltone Fulldrive 2/fulldrive2.sch (EAGLE design)
At the start: 50 parts, among them IC1 JRC4558, Q1 2N5088, Q2 2N5088, Q3 2N7000, Q4 2N7000

Commit message: 20200329/10:01
Parts:
- C1: value 10p -> 22n
- C2: value 22n -> 10p
Connections:
- net GND: now also C2.2; no longer C1.2, VOL.1
- net IN: now also C1.2, C2.1; no longer C1.1, C2.2
- net N$16: now also R5.2; no longer R5.1
- net N$2: now also C1.1; no longer C2.1
- net VB: now also R5.1, VOL.1; no longer R5.2
Other:
- moved on the sheet: BOOST, C1, C10, C11, C12, C13, C14, C2, C4, C5, C6, C7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
