File: #Misc/Fulltone OCD/ocd_redraw.sch (EAGLE design)
At the start: 33 parts, among them IC1 TL082CP, Q1 2N7000, Q2 2N7000

Commit message: 20200329/10:01
Other:
- moved on the sheet: C1, C2, C3, R1, R2, R3
