File: #Misc/Nobels ODR-B/odrb.sch (EAGLE design)
At the start: 126 parts, among them J1 INPUT, J2 OUTPUT, J4 POWER, P1 50kB, P11 500kA, P21 50kB, P22 50kB, P31 10kC, Q1 K222E, Q2 C2362G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

Commit message: 20200329/10:32
Parts:
- renumbered C4 to C28
Connections:
- net N$66: now also JP4 -1.S; no longer JP4 -3.S
- net N$67: now also JP4 -3.S; no longer JP4 -1.S
- net N$68: now also JP5 -3.S; no longer JP5 -1.S
- net VB: now also JP5 -1.S; no longer JP5 -3.S
Other:
- moved on the sheet: C106, C41, D7, JP4 -1, JP4 -3, JP5 -1, JP5 -3, JP5-1, JP5-2, JP5-3, Q7, R109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
